Commit message: tinkering till drone flies...

File: models/copterPIX/ardupilot_plugin.xacro (robot description, xacro)
@@ -1,4 +1,6 @@
 <?xml version="1.0" ?>
 <robot name="copterPIX" xmlns:xacro="http://www.ros.org/wiki/xacro">
+    <xacro:property name="multiplier" value="1000"/>
+    <xacro:property name="multiplier_negative" value="${-1 * multiplier}"/>
     <gazebo>
         <plugin name="arducopter_plugin" filename="libArduPilotPlugin.so">
@@ -22,5 +24,5 @@
                 <cmd_min>-2.5</cmd_min>
                 <jointName>rotor_joint_0</jointName>
-                <multiplier>-838</multiplier>
+                <multiplier>${multiplier_negative}</multiplier>
                 <controlVelocitySlowdownSim>1</controlVelocitySlowdownSim>
             </control>
@@ -36,5 +38,5 @@
                 <cmd_min>-2.5</cmd_min>
                 <jointName>rotor_joint_1</jointName>
-                <multiplier>838</multiplier>
+                <multiplier>${multiplier}</multiplier>
                 <controlVelocitySlowdownSim>1</controlVelocitySlowdownSim>
             </control>
@@ -50,5 +52,5 @@
                 <cmd_min>-2.5</cmd_min>
                 <jointName>rotor_joint_2</jointName>
-                <multiplier>-838</multiplier>
+                <multiplier>${multiplier_negative}</multiplier>
                 <controlVelocitySlowdownSim>1</controlVelocitySlowdownSim>
             </control>
@@ -64,5 +66,5 @@
                 <cmd_min>-2.5</cmd_min>
                 <jointName>rotor_joint_3</jointName>
-                <multiplier>838</multiplier>
+                <multiplier>${multiplier}</multiplier>
                 <controlVelocitySlowdownSim>1</controlVelocitySlowdownSim>
             </control>
@@ -78,5 +80,5 @@
                 <cmd_min>-2.5</cmd_min>
                 <jointName>rotor_joint_4</jointName>
-                <multiplier>838</multiplier>
+                <multiplier>${multiplier}</multiplier>
                 <controlVelocitySlowdownSim>1</controlVelocitySlowdownSim>
             </control>
@@ -92,5 +94,5 @@
                 <cmd_min>-2.5</cmd_min>
                 <jointName>rotor_joint_5</jointName>
-                <multiplier>-838</multiplier>
+                <multiplier>${multiplier_negative}</multiplier>
                 <controlVelocitySlowdownSim>1</controlVelocitySlowdownSim>
             </control>

File: models/copterPIX/robot.urdf.xacro (robot description, xacro)
@@ -7,14 +7,14 @@
   <xacro:property name="prop_ccw_mesh" value="$(find drone)/STLs/iris_prop_ccw.dae"/>
   <!-- Base link -->
-  <!-- <link name="base_link"> -->
+  <link name="base_link">
     <!-- You can leave this link empty if you don't need a specific geometry or inertial properties for the base -->
-  <!-- </link> -->
+  </link>
   <!-- Joint (fixed) -->
-  <!-- <joint name="fixed_joint" type="fixed">
+  <joint name="fixed_joint" type="fixed">
     <parent link="base_link"/>
     <child link="core_link"/>
     <origin xyz="0 0 0.6" rpy="0 0 0"/>
-  </joint> -->
-  <xacro:property name="g_mms_to_kg_ms" value="1000000000" />
+  </joint>
+  <xacro:property name="g_mms_to_kg_ms" value="1000000000"/>
   <!-- <xacro:property name="mass" value="26.0" />
   <xacro:property name="ixx" value="${373162267137.9 / g_mms_to_kg_ms}"/>
@@ -24,12 +24,41 @@
   <xacro:property name="iyz" value="${50504029566.32 / g_mms_to_kg_ms}"/>
   <xacro:property name="izz" value="${574188826210.05 / g_mms_to_kg_ms}"/> -->
-  <xacro:property name="mass" value="2.0" />
-  <xacro:property name="ixx" value="${0.1}"/>
+  <!-- <xacro:property name="mass" value="4" />
+  <xacro:property name="s" value="50" />
+  <xacro:property name="ixx" value="${1 * s}"/>
+  <xacro:property name="ixy" value="${0 * s}"/>
+  <xacro:property name="ixz" value="${0 * s}"/>
+  <xacro:property name="iyy" value="${1 * s}"/>
+  <xacro:property name="iyz" value="${0 * s}"/>
+  <xacro:property name="izz" value="${1.6 * s}"/> -->
+  <xacro:property name="mass" value="26" />
+  <xacro:property name="s" value="50" />
+  <xacro:property name="ixx" value="${1}"/>
   <xacro:property name="ixy" value="${0}"/>
   <xacro:property name="ixz" value="${0}"/>
-  <xacro:property name="iyy" value="${0.1}"/>
+  <xacro:property name="iyy" value="${1}"/>
   <xacro:property name="iyz" value="${0}"/>
-  <xacro:property name="izz" value="${0.15}"/>
-  <xacro:link_creator_i link_name="core_link" pose_xyz="0 0 0" pose_rpy="0 0 0" mesh_path="${hex_mesh}" scale_xyz="0.4 0.4 0.04" center_mass_xyz="0 0 -0.25" mass="${mass}" ixx="${ixx}" ixy="${ixy}" ixz="${ixz}" iyy="${iyy}" iyz="${iyz}" izz="${izz}"/>
+  <xacro:property name="izz" value="${1.6}"/>
+  <xacro:link_creator_i_foundation link_name="core_link" pose_xyz="0 0 0" pose_rpy="0 0 0" mesh_path="${hex_mesh}" scale_xyz="0.4 0.4 0.04" center_mass_xyz="0 0 -0.15" mass="${mass}" ixx="${ixx}" ixy="${ixy}" ixz="${ixz}" iyy="${iyy}" iyz="${iyz}" izz="${izz}">
+    <extra_collision>
+      <surface>
+        <contact>
+          <ode>
+            <max_vel>100.0</max_vel>
+            <min_depth>0.001</min_depth>
+          </ode>
+        </contact>
+        <friction>
+          <ode>
+            <mu>100000.0</mu>
+            <mu2>100000.0</mu2>
+          </ode>
+        </friction>
+      </surface>
+    </extra_collision>
+    <seperate_collider><box filename="${hex_mesh}" scale="0.4 0.4 0.04"/></seperate_collider>
+    <extra_visual/>
+    <extra_settings/>
+  </xacro:link_creator_i_foundation>
   <!-- <xacro:link_creator link_name="core_link" pose_xyz="0 0 0" pose_rpy="0 0 0" mesh_path="${hex_mesh}" scale_xyz="0.4 0.4 0.04"/> -->
   <joint name="leg_0_link_joint" type="fixed">
@@ -71,11 +100,48 @@
   <xacro:drone_arm num="4" parent_link="core_link" dis_from_center="0.175" length="0.56" diameter="0.025" arm_incline_angle="${4 * deg_to_rad}" arm_mesh="${hex_mesh}" prop_mesh="${prop_ccw_mesh}" cw="false" prop_size_multiplier="2.04" rmass="0.2" rixx="0.000312" rixy="0" rixz="0" riyy="0.0053345" riyz="0" rizz="0.005363328" angle="${60 * deg_to_rad}"/>
   <xacro:drone_arm num="5" parent_link="core_link" dis_from_center="0.175" length="0.56" diameter="0.025" arm_incline_angle="${4 * deg_to_rad}" arm_mesh="${hex_mesh}" prop_mesh="${prop_cw_mesh}" cw="true" prop_size_multiplier="2.04" rmass="0.2" rixx="0.000312" rixy="0" rixz="0" riyy="0.0053345" riyz="0" rizz="0.005363328" angle="${240 * deg_to_rad}"/> -->
-  <xacro:drone_arm num="0" parent_link="core_link" dis_from_center="0.175" length="0.56" diameter="0.025" arm_incline_angle="${4 * deg_to_rad}" arm_mesh="${hex_mesh}" prop_mesh="${prop_cw_mesh}"  cw="true"  prop_size_multiplier="2.04" rmass="0.025" rixx="0.00000975" rixy="0" rixz="0" riyy="0.000166704" riyz="0" rizz="0.000167604" angle="${0 * deg_to_rad}"/>
-  <xacro:drone_arm num="1" parent_link="core_link" dis_from_center="0.175" length="0.56" diameter="0.025" arm_incline_angle="${4 * deg_to_rad}" arm_mesh="${hex_mesh}" prop_mesh="${prop_ccw_mesh}" cw="false" prop_size_multiplier="2.04" rmass="0.025" rixx="0.00000975" rixy="0" rixz="0" riyy="0.000166704" riyz="0" rizz="0.000167604" angle="${180 * deg_to_rad}"/>
-  <xacro:drone_arm num="2" parent_link="core_link" dis_from_center="0.175" length="0.56" diameter="0.025" arm_incline_angle="${4 * deg_to_rad}" arm_mesh="${hex_mesh}" prop_mesh="${prop_cw_mesh}"  cw="true"  prop_size_multiplier="2.04" rmass="0.025" rixx="0.00000975" rixy="0" rixz="0" riyy="0.000166704" riyz="0" rizz="0.000167604" angle="${120 * deg_to_rad}"/>
-  <xacro:drone_arm num="3" parent_link="core_link" dis_from_center="0.175" length="0.56" diameter="0.025" arm_incline_angle="${4 * deg_to_rad}" arm_mesh="${hex_mesh}" prop_mesh="${prop_ccw_mesh}" cw="false" prop_size_multiplier="2.04" rmass="0.025" rixx="0.00000975" rixy="0" rixz="0" riyy="0.000166704" riyz="0" rizz="0.000167604" angle="${300 * deg_to_rad}"/>
-  <xacro:drone_arm num="4" parent_link="core_link" dis_from_center="0.175" length="0.56" diameter="0.025" arm_incline_angle="${4 * deg_to_rad}" arm_mesh="${hex_mesh}" prop_mesh="${prop_ccw_mesh}" cw="false" prop_size_multiplier="2.04" rmass="0.025" rixx="0.00000975" rixy="0" rixz="0" riyy="0.000166704" riyz="0" rizz="0.000167604" angle="${60 * deg_to_rad}"/>
-  <xacro:drone_arm num="5" parent_link="core_link" dis_from_center="0.175" length="0.56" diameter="0.025" arm_incline_angle="${4 * deg_to_rad}" arm_mesh="${hex_mesh}" prop_mesh="${prop_cw_mesh}"  cw="true"  prop_size_multiplier="2.04" rmass="0.025" rixx="0.00000975" rixy="0" rixz="0" riyy="0.000166704" riyz="0" rizz="0.000167604" angle="${240 * deg_to_rad}"/>
+  <xacro:drone_arm num="0" parent_link="core_link" dis_from_center="0.175" length="0.56" diameter="0.025" arm_incline_angle="${6 * deg_to_rad}" arm_mesh="${hex_mesh}" prop_mesh="${prop_cw_mesh}"  cw="true"  prop_size_multiplier="2.04" rmass="0.025" rixx="0.00000975" rixy="0" rixz="0" riyy="0.000166704" riyz="0" rizz="0.000167604" angle="${0 * deg_to_rad}"/>
+  <xacro:drone_arm num="1" parent_link="core_link" dis_from_center="0.175" length="0.56" diameter="0.025" arm_incline_angle="${6 * deg_to_rad}" arm_mesh="${hex_mesh}" prop_mesh="${prop_ccw_mesh}" cw="false" prop_size_multiplier="2.04" rmass="0.025" rixx="0.00000975" rixy="0" rixz="0" riyy="0.000166704" riyz="0" rizz="0.000167604" angle="${180 * deg_to_rad}"/>
+  <xacro:drone_arm num="2" parent_link="core_link" dis_from_center="0.175" length="0.56" diameter="0.025" arm_incline_angle="${6 * deg_to_rad}" arm_mesh="${hex_mesh}" prop_mesh="${prop_cw_mesh}"  cw="true"  prop_size_multiplier="2.04" rmass="0.025" rixx="0.00000975" rixy="0" rixz="0" riyy="0.000166704" riyz="0" rizz="0.000167604" angle="${120 * deg_to_rad}"/>
+  <xacro:drone_arm num="3" parent_link="core_link" dis_from_center="0.175" length="0.56" diameter="0.025" arm_incline_angle="${6 * deg_to_rad}" arm_mesh="${hex_mesh}" prop_mesh="${prop_ccw_mesh}" cw="false" prop_size_multiplier="2.04" rmass="0.025" rixx="0.00000975" rixy="0" rixz="0" riyy="0.000166704" riyz="0" rizz="0.000167604" angle="${300 * deg_to_rad}"/>
+  <xacro:drone_arm num="4" parent_link="core_link" dis_from_center="0.175" length="0.56" diameter="0.025" arm_incline_angle="${6 * deg_to_rad}" arm_mesh="${hex_mesh}" prop_mesh="${prop_ccw_mesh}" cw="false" prop_size_multiplier="2.04" rmass="0.025" rixx="0.00000975" rixy="0" rixz="0" riyy="0.000166704" riyz="0" rizz="0.000167604" angle="${60 * deg_to_rad}"/>
+  <xacro:drone_arm num="5" parent_link="core_link" dis_from_center="0.175" length="0.56" diameter="0.025" arm_incline_angle="${6 * deg_to_rad}" arm_mesh="${hex_mesh}" prop_mesh="${prop_cw_mesh}"  cw="true"  prop_size_multiplier="2.04" rmass="0.025" rixx="0.00000975" rixy="0" rixz="0" riyy="0.000166704" riyz="0" rizz="0.000167604" angle="${240 * deg_to_rad}"/>
   <gazebo>
+    <!-- <link name='odometry_sensorgt_link'>
+      <pose>0 0 0 0 -0 0</pose>
+      <inertial>
+        <pose>0 0 0 0 -0 0</pose>
+        <mass>0.15</mass>
+        <inertia>
+          <ixx>0.0001</ixx>
+          <ixy>0</ixy>
+          <ixz>0</ixz>
+          <iyy>0.0002</iyy>
+          <iyz>0</iyz>
+          <izz>0.0002</izz>
+        </inertia>
+      </inertial>
+    </link>
+    <joint name='odometry_sensorgt_joint' type='revolute'>
+      <child>odometry_sensorgt_link</child>
+      <parent>core_link</parent>
+      <axis>
+        <xyz>0 0 1</xyz>
+        <limit>
+          <lower>0</lower>
+          <upper>0</upper>
+          <effort>0</effort>
+          <velocity>0</velocity>
+        </limit>
+        <dynamics>
+          <damping>1.0</damping>
+        </dynamics>
+        <use_parent_model_frame>1</use_parent_model_frame>
+      </axis>
+      <physics>
+        <ode>
+          <implicit_spring_damper>1</implicit_spring_damper>
+        </ode>
+      </physics>
+    </joint> -->
     <link name='imu_link'>
       <inertial>

File: xacros/macro.xacro (robot description, xacro)
@@ -30,5 +30,5 @@
         </gazebo>
         <xacro:prop_link_creator link_name="${prop_link}" pose_xyz="0 0 0.03" pose_rpy="0 -0 0" mesh_path="${prop_mesh}" scale_xyz="${prop_size_multiplier} ${prop_size_multiplier} ${prop_size_multiplier}" mass="${rmass}" ixx="${rixx}" ixy="${rixy}" ixz="${rixz}" iyy="${riyy}" iyz="${riyz}" izz="${rizz}"/>
-        <xacro:property name="cp" value="0.008"/>
+        <xacro:property name="cp" value="0.13"/>
         <xacro:property name="cp_negative" value="${-1 * cp}"/>
         <xacro:property name="area" value="0.002"/> <!--used to be 0.002-->
