Commit message: added inertial_macros.xacro, made the lift of the props larger(increased area) and made the macros of links smarter(automatic inertia calculation). also added servo channel in ardupilot_plugin.xacro and made a knob so later it will trigger the gun(ros topic will apply the force hopefully) so todo is to make python script for that and somehow apply force for the gun shot kickback

File: models/copterPIX/ardupilot_plugin.xacro (robot description, xacro)
@@ -1,5 +1,5 @@
 <?xml version="1.0" ?>
-<robot name="copterPIX" xmlns:xacro="http://www.ros.org/wiki/xacro">
-    <xacro:property name="multiplier" value="1200"/>
+<robot xmlns:xacro="http://www.ros.org/wiki/xacro">
+    <xacro:property name="multiplier" value="800"/>
     <xacro:property name="multiplier_negative" value="${-1 * multiplier}"/>
     <gazebo>
@@ -97,5 +97,36 @@
                 <controlVelocitySlowdownSim>1</controlVelocitySlowdownSim>
             </control>
+            <control channel="6">
+                <type>POSITION</type>
+                <jointName>fire_trigger_servo_joint</jointName>
+                <multiplier>1.5708</multiplier> <!-- Maps PWM range to -90 to 90 degrees -->
+                <controlVelocitySlowdownSim>1</controlVelocitySlowdownSim>
+            </control>
         </plugin>
     </gazebo>
 </robot>
+  <!-- /// \brief Interface ArduPilot from ardupilot stack
+  /// modeled after SITL/SIM_*
+  ///
+  /// The plugin requires the following parameters:
+  /// <control>             control description block
+  ///    <!- inputs from Ardupilot ->
+  ///    channel            attribute, ardupilot control channel
+  ///    multiplier         command multiplier
+  ///    <!- output to Gazebo ->
+  ///    type               type of control, VELOCITY, POSITION or EFFORT
+  ///    <p_gain>           velocity pid p gain
+  ///    <i_gain>           velocity pid i gain
+  ///    <d_gain>           velocity pid d gain
+  ///    <i_max>            velocity pid max integral correction
+  ///    <i_min>            velocity pid min integral correction
+  ///    <cmd_max>          velocity pid max command torque
+  ///    <cmd_min>          velocity pid min command torque
+  ///    <jointName>        motor joint, torque applied here
+  ///    <turningDirection> rotor turning direction, 'cw' or 'ccw'
+  ///    frequencyCutoff    filter incoming joint state
+  ///    samplingRate       sampling rate for filtering incoming joint state
+  ///    <rotorVelocitySlowdownSim> for rotor aliasing problem, experimental
+  /// <imuName>     scoped name for the imu sensor
+  /// <connectionTimeoutMaxCount> timeout before giving up on
+  ///                             controller synchronization -->

File: models/copterPIX/robot.urdf.xacro (robot description, xacro)
@@ -8,36 +8,21 @@
   <xacro:property name="prop_ccw_mesh" value="$(find drone)/STLs/iris_prop_ccw.dae"/>
   <xacro:property name="g_mms_to_kg_ms" value="1000000000"/>
-  <xacro:property name="mass" value="17.0" />
-  <!-- <xacro:property name="ixx" value="${373162267137.9 / g_mms_to_kg_ms}"/>
-  <xacro:property name="ixy" value="${19971359238.18 / g_mms_to_kg_ms}"/>
-  <xacro:property name="ixz" value="${-71155586006.28 / g_mms_to_kg_ms}"/>
-  <xacro:property name="iyy" value="${595713038514.03 / g_mms_to_kg_ms}"/>
-  <xacro:property name="iyz" value="${50504029566.32 / g_mms_to_kg_ms}"/>
-  <xacro:property name="izz" value="${574188826210.05 / g_mms_to_kg_ms}"/> -->
-  <xacro:property name="ixx" value="${1000000000 / g_mms_to_kg_ms}"/>
+  <xacro:property name="mass" value="19" />
+  <!-- <xacro:property name="ixx" value="${373162267137.9 / g_mms_to_kg_ms}"/>  these values are not valid, they are stupid wrong
+    <xacro:property name="ixy" value="${19971359238.18 / g_mms_to_kg_ms}"/>
+    <xacro:property name="ixz" value="${-71155586006.28 / g_mms_to_kg_ms}"/>
+    <xacro:property name="iyy" value="${595713038514.03 / g_mms_to_kg_ms}"/>
+    <xacro:property name="iyz" value="${50504029566.32 / g_mms_to_kg_ms}"/>
+    <xacro:property name="izz" value="${574188826210.05 / g_mms_to_kg_ms}"/>
+  -->
+  <xacro:property name="center_of_mass" value="0 0 0"/>
+  <!-- <xacro:property name="ixx" value="${10000000000 / g_mms_to_kg_ms}"/>
   <xacro:property name="ixy" value="${0 / g_mms_to_kg_ms}"/>
   <xacro:property name="ixz" value="${0 / g_mms_to_kg_ms}"/>
-  <xacro:property name="iyy" value="${1000000000 / g_mms_to_kg_ms}"/>
+  <xacro:property name="iyy" value="${10000000000 / g_mms_to_kg_ms}"/>
   <xacro:property name="iyz" value="${0 / g_mms_to_kg_ms}"/>
-  <xacro:property name="izz" value="${1200000000 / g_mms_to_kg_ms}"/>
-  <!-- <xacro:property name="mass" value="4" />
-    <xacro:property name="s" value="50" />
-    <xacro:property name="ixx" value="${1 * s}"/>
-    <xacro:property name="ixy" value="${0 * s}"/>
-    <xacro:property name="ixz" value="${0 * s}"/>
-    <xacro:property name="iyy" value="${1 * s}"/>
-    <xacro:property name="iyz" value="${0 * s}"/>
-    <xacro:property name="izz" value="${1.6 * s}"/>
-  -->
-  <!-- <xacro:property name="mass" value="4" />
-    <xacro:property name="s" value="1"/>
-    <xacro:property name="ixx" value="${0.08 * s}"/>
-    <xacro:property name="ixy" value="${0 * s}"/>
-    <xacro:property name="ixz" value="${0 * s}"/>
-    <xacro:property name="iyy" value="${0.08 * s}"/>
-    <xacro:property name="iyz" value="${0 * s}"/>
-    <xacro:property name="izz" value="${0.1 * s}"/>
-  -->
-  <xacro:link_creator_i link_name="base_link" pose_xyz="0 0 0" pose_rpy="0 0 0" mesh_path="${hex_mesh}" scale_xyz="0.4 0.4 0.04" center_mass_xyz="0 0 -0.5" mass="${mass}" ixx="${ixx}" ixy="${ixy}" ixz="${ixz}" iyy="${iyy}" iyz="${iyz}" izz="${izz}"/>
+  <xacro:property name="izz" value="${16000000000 / g_mms_to_kg_ms}"/> -->
+  <!-- <xacro:link_creator_i link_name="base_link" pose_xyz="0 0 0" pose_rpy="0 0 0" mesh_path="${hex_mesh}" scale_xyz="0.4 0.4 0.04" center_mass_xyz="${center_of_mass}" mass="${mass}" ixx="${ixx}" ixy="${ixy}" ixz="${ixz}" iyy="${iyy}" iyz="${iyz}" izz="${izz}"/> -->
+  <xacro:link_creator_i link_name="base_link" pose_xyz="0 0 0" pose_rpy="0 0 0" mesh_path="${hex_mesh}" scale_xyz="0.4 0.4 0.04" center_mass_xyz="${center_of_mass}" mass="${mass}"/>
   <!-- <xacro:link_creator_i_foundation link_name="base_link" pose_xyz="0 0 0" pose_rpy="0 0 0" mesh_path="${hex_mesh}" scale_xyz="0.4 0.4 0.04" seperate_collider_xyzrpy="0 0 -0.3 0 0 0" center_mass_xyz="0 0 -0.5" mass="${mass}" ixx="${ixx}" ixy="${ixy}" ixz="${ixz}" iyy="${iyy}" iyz="${iyz}" izz="${izz}">
     <extra_collision>
@@ -66,34 +51,37 @@
     <child link="leg_0_link"/>
   </joint>
-  <xacro:link_creator_i link_name="leg_0_link" pose_xyz="0 0.198 -0.305" pose_rpy="0.305 0 0" mesh_path="$(find drone)/STLs/hexagonal_prism_height_1_outer_diameter_1.stl" scale_xyz="0.024 0.024 0.61" mass="0.2" ixx="0.0" ixy="0.0" ixz="0.0" iyy="0.0" iyz="0.0" izz="0.0"/>
-  <!-- <xacro:link_creator link_name="leg_0_link" pose_xyz="0 0.198 -0.305" pose_rpy="0.305 0 0" mesh_path="${hex_mesh}" scale_xyz="0.024 0.024 0.61"/> -->
+  <!-- <xacro:link_creator_i link_name="leg_0_link" pose_xyz="0 0.198 -0.305" pose_rpy="0.305 0 0" mesh_path="$(find drone)/STLs/hexagonal_prism_height_1_outer_diameter_1.stl" scale_xyz="0.024 0.024 0.61" mass="0.2" ixx="0.0" ixy="0.0" ixz="0.0" iyy="0.0" iyz="0.0" izz="0.0"/> -->
+  <xacro:link_creator_i link_name="leg_0_link" pose_xyz="0 0.198 -0.305" pose_rpy="0.305 0 0" mesh_path="$(find drone)/STLs/hexagonal_prism_height_1_outer_diameter_1.stl" scale_xyz="0.024 0.024 0.61" mass="0.5"/>
   <joint name="leg_1_link_joint" type="fixed">
     <parent link="base_link"/>
     <child link="leg_1_link"/>
   </joint>
-  <xacro:link_creator_i link_name="leg_1_link" pose_xyz="0 -0.198 -0.305" pose_rpy="-0.305 0 0" mesh_path="$(find drone)/STLs/hexagonal_prism_height_1_outer_diameter_1.stl" scale_xyz="0.024 0.024 0.61" mass="0.2" ixx="0.0" ixy="0.0" ixz="0.0" iyy="0.0" iyz="0.0" izz="0.0"/>
-  <!-- <xacro:link_creator link_name="leg_1_link" pose_xyz="0 -0.198 -0.305" pose_rpy="-0.305 0 0" mesh_path="${hex_mesh}" scale_xyz="0.024 0.024 0.61"/> -->
+  <!-- <xacro:link_creator_i link_name="leg_1_link" pose_xyz="0 -0.198 -0.305" pose_rpy="-0.305 0 0" mesh_path="$(find drone)/STLs/hexagonal_prism_height_1_outer_diameter_1.stl" scale_xyz="0.024 0.024 0.61" mass="0.2" ixx="0.0" ixy="0.0" ixz="0.0" iyy="0.0" iyz="0.0" izz="0.0"/> -->
+  <xacro:link_creator_i link_name="leg_1_link" pose_xyz="0 -0.198 -0.305" pose_rpy="-0.305 0 0" mesh_path="$(find drone)/STLs/hexagonal_prism_height_1_outer_diameter_1.stl" scale_xyz="0.024 0.024 0.61" mass="0.5"/>
   <joint name="feet_0_link_joint" type="fixed">
     <parent link="base_link"/>
     <child link="feet_0_link"/>
   </joint>
-  <xacro:link_creator_i link_name="feet_0_link" pose_xyz="0 0.29 -0.6" pose_rpy="0 1.57079633 0" mesh_path="$(find drone)/STLs/hexagonal_prism_height_1_outer_diameter_1.stl" scale_xyz="0.024 0.024 0.58" mass="0.2" ixx="0.0" ixy="0.0" ixz="0.0" iyy="0.0" iyz="0.0" izz="0.0"/>
-  <!-- <xacro:link_creator link_name="feet_0_link" pose_xyz="0 0.29 -0.6" pose_rpy="0 1.57079633 0" mesh_path="${hex_mesh}" scale_xyz="0.024 0.024 0.58"/> -->
+  <!-- <xacro:link_creator_i link_name="feet_0_link" pose_xyz="0 0.29 -0.6" pose_rpy="0 1.57079633 0" mesh_path="$(find drone)/STLs/hexagonal_prism_height_1_outer_diameter_1.stl" scale_xyz="0.024 0.024 0.58" mass="0.2" ixx="0.0" ixy="0.0" ixz="0.0" iyy="0.0" iyz="0.0" izz="0.0"/> -->
+  <xacro:link_creator_i link_name="feet_0_link" pose_xyz="0 0.29 -0.6" pose_rpy="0 1.57079633 0" mesh_path="$(find drone)/STLs/hexagonal_prism_height_1_outer_diameter_1.stl" scale_xyz="0.024 0.024 0.58" mass="0.5"/>
   <joint name="feet_1_link_joint" type="fixed">
     <parent link="base_link"/>
     <child link="feet_1_link"/>
   </joint>
-  <xacro:link_creator_i link_name="feet_1_link" pose_xyz="0 -0.29 -0.6" pose_rpy="0 1.57079633 0" mesh_path="$(find drone)/STLs/hexagonal_prism_height_1_outer_diameter_1.stl" scale_xyz="0.024 0.024 0.58" mass="0.2" ixx="0.0" ixy="0.0" ixz="0.0" iyy="0.0" iyz="0.0" izz="0.0"/>
-  <!-- <xacro:link_creator link_name="feet_1_link" pose_xyz="0 -0.29 -0.6" pose_rpy="0 1.57079633 0" mesh_path="${hex_mesh}" scale_xyz="0.024 0.024 0.58"/> -->
+  <!-- <xacro:link_creator_i link_name="feet_1_link" pose_xyz="0 -0.29 -0.6" pose_rpy="0 1.57079633 0" mesh_path="$(find drone)/STLs/hexagonal_prism_height_1_outer_diameter_1.stl" scale_xyz="0.024 0.024 0.58" mass="0.2" ixx="0.0" ixy="0.0" ixz="0.0" iyy="0.0" iyz="0.0" izz="0.0"/> -->
+  <xacro:link_creator_i link_name="feet_1_link" pose_xyz="0 -0.29 -0.6" pose_rpy="0 1.57079633 0" mesh_path="$(find drone)/STLs/hexagonal_prism_height_1_outer_diameter_1.stl" scale_xyz="0.024 0.024 0.58" mass="0.5"/>
   <!-- Define the drone arms using the macro -->
   <xacro:property name="deg_to_rad" value="0.0174533"/>
-  <xacro:property name="dfc" value = "0.175"/>
   <xacro:property name="dfc" value = "0.175"/>
   <xacro:property name="leng" value="0.56"/>
   <xacro:property name="dia" value="0.025"/>
   <xacro:property name="aia" value="5"/>
-  <xacro:property name="cla" value="4.5"/>
-  <xacro:property name="cp" value="0.124"/>
-  <xacro:property name="area" value="0.012"/>
+  <xacro:property name="psm" value="2.04"/>
+  <xacro:property name="cylinder_r" value="0.25"/>
+  <xacro:property name="cylinder_l" value="0.02"/>
+  <xacro:property name="cla" value="4.3"/>
+  <xacro:property name="cp" value="0.2"/>
+  <xacro:property name="area" value="0.01"/>
+  <xacro:property name="amass" value="0.5"/>
   <xacro:property name="rmass" value="0.2"/>
   <xacro:property name="rixx" value="0.000312"/>
@@ -103,10 +91,10 @@
   <xacro:property name="riyz" value="0"/>
   <xacro:property name="rizz" value="0.005363328"/>
-  <xacro:drone_arm num="0" parent_link="base_link" dis_from_center="${dfc}" length="${leng}" diameter="${dia}" arm_incline_angle="${aia * deg_to_rad}" arm_mesh="${hex_mesh}" prop_mesh="${prop_cw_mesh}"  cw="true"  prop_size_multiplier="2.04" cla="4.5" cp="0.084" area="0.002" rmass="0.025" rixx="0.00000975" rixy="0" rixz="0" riyy="0.000166704" riyz="0" rizz="0.000167604" angle="${0 * deg_to_rad}"/>
-  <xacro:drone_arm num="1" parent_link="base_link" dis_from_center="${dfc}" length="${leng}" diameter="${dia}" arm_incline_angle="${aia * deg_to_rad}" arm_mesh="${hex_mesh}" prop_mesh="${prop_ccw_mesh}" cw="false" prop_size_multiplier="2.04" cla="4.5" cp="0.084" area="0.002" rmass="0.025" rixx="0.00000975" rixy="0" rixz="0" riyy="0.000166704" riyz="0" rizz="0.000167604" angle="${180 * deg_to_rad}"/>
-  <xacro:drone_arm num="2" parent_link="base_link" dis_from_center="${dfc}" length="${leng}" diameter="${dia}" arm_incline_angle="${aia * deg_to_rad}" arm_mesh="${hex_mesh}" prop_mesh="${prop_cw_mesh}"  cw="true"  prop_size_multiplier="2.04" cla="4.5" cp="0.084" area="0.002" rmass="0.025" rixx="0.00000975" rixy="0" rixz="0" riyy="0.000166704" riyz="0" rizz="0.000167604" angle="${120 * deg_to_rad}"/>
-  <xacro:drone_arm num="3" parent_link="base_link" dis_from_center="${dfc}" length="${leng}" diameter="${dia}" arm_incline_angle="${aia * deg_to_rad}" arm_mesh="${hex_mesh}" prop_mesh="${prop_ccw_mesh}" cw="false" prop_size_multiplier="2.04" cla="4.5" cp="0.084" area="0.002" rmass="0.025" rixx="0.00000975" rixy="0" rixz="0" riyy="0.000166704" riyz="0" rizz="0.000167604" angle="${300 * deg_to_rad}"/>
-  <xacro:drone_arm num="4" parent_link="base_link" dis_from_center="${dfc}" length="${leng}" diameter="${dia}" arm_incline_angle="${aia * deg_to_rad}" arm_mesh="${hex_mesh}" prop_mesh="${prop_ccw_mesh}" cw="false" prop_size_multiplier="2.04" cla="4.5" cp="0.084" area="0.002" rmass="0.025" rixx="0.00000975" rixy="0" rixz="0" riyy="0.000166704" riyz="0" rizz="0.000167604" angle="${60 * deg_to_rad}"/>
-  <xacro:drone_arm num="5" parent_link="base_link" dis_from_center="${dfc}" length="${leng}" diameter="${dia}" arm_incline_angle="${aia * deg_to_rad}" arm_mesh="${hex_mesh}" prop_mesh="${prop_cw_mesh}"  cw="true"  prop_size_multiplier="2.04" cla="4.5" cp="0.084" area="0.002" rmass="0.025" rixx="0.00000975" rixy="0" rixz="0" riyy="0.000166704" riyz="0" rizz="0.000167604" angle="${240 * deg_to_rad}"/>
+  <xacro:drone_arm num="0" parent_link="base_link" dis_from_center="${dfc}" length="${leng}" diameter="${dia}" arm_incline_angle="${aia * deg_to_rad}" arm_mesh="${hex_mesh}" prop_mesh="${prop_cw_mesh}"  cw="true"  prop_size_multiplier="${psm}" cylinder_r="${cylinder_r}" cylinder_l="${cylinder_l}" amass="${amass}"  cla="${cla}" cp="${cp}" area="${area}" rmass="${rmass}" rixx="${rixx}" rixy="${rixy}" rixz="${rixz}" riyy="${riyy}" riyz="${riyz}" rizz="${rizz}" angle="${0 * deg_to_rad}"/>
+  <xacro:drone_arm num="1" parent_link="base_link" dis_from_center="${dfc}" length="${leng}" diameter="${dia}" arm_incline_angle="${aia * deg_to_rad}" arm_mesh="${hex_mesh}" prop_mesh="${prop_ccw_mesh}" cw="false" prop_size_multiplier="${psm}" cylinder_r="${cylinder_r}" cylinder_l="${cylinder_l}" amass="${amass}"  cla="${cla}" cp="${cp}" area="${area}" rmass="${rmass}" rixx="${rixx}" rixy="${rixy}" rixz="${rixz}" riyy="${riyy}" riyz="${riyz}" rizz="${rizz}" angle="${180 * deg_to_rad}"/>
+  <xacro:drone_arm num="2" parent_link="base_link" dis_from_center="${dfc}" length="${leng}" diameter="${dia}" arm_incline_angle="${aia * deg_to_rad}" arm_mesh="${hex_mesh}" prop_mesh="${prop_cw_mesh}"  cw="true"  prop_size_multiplier="${psm}" cylinder_r="${cylinder_r}" cylinder_l="${cylinder_l}" amass="${amass}"  cla="${cla}" cp="${cp}" area="${area}" rmass="${rmass}" rixx="${rixx}" rixy="${rixy}" rixz="${rixz}" riyy="${riyy}" riyz="${riyz}" rizz="${rizz}" angle="${120 * deg_to_rad}"/>
+  <xacro:drone_arm num="3" parent_link="base_link" dis_from_center="${dfc}" length="${leng}" diameter="${dia}" arm_incline_angle="${aia * deg_to_rad}" arm_mesh="${hex_mesh}" prop_mesh="${prop_ccw_mesh}" cw="false" prop_size_multiplier="${psm}" cylinder_r="${cylinder_r}" cylinder_l="${cylinder_l}" amass="${amass}"  cla="${cla}" cp="${cp}" area="${area}" rmass="${rmass}" rixx="${rixx}" rixy="${rixy}" rixz="${rixz}" riyy="${riyy}" riyz="${riyz}" rizz="${rizz}" angle="${300 * deg_to_rad}"/>
+  <xacro:drone_arm num="4" parent_link="base_link" dis_from_center="${dfc}" length="${leng}" diameter="${dia}" arm_incline_angle="${aia * deg_to_rad}" arm_mesh="${hex_mesh}" prop_mesh="${prop_ccw_mesh}" cw="false" prop_size_multiplier="${psm}" cylinder_r="${cylinder_r}" cylinder_l="${cylinder_l}" amass="${amass}"  cla="${cla}" cp="${cp}" area="${area}" rmass="${rmass}" rixx="${rixx}" rixy="${rixy}" rixz="${rixz}" riyy="${riyy}" riyz="${riyz}" rizz="${rizz}" angle="${60 * deg_to_rad}"/>
+  <xacro:drone_arm num="5" parent_link="base_link" dis_from_center="${dfc}" length="${leng}" diameter="${dia}" arm_incline_angle="${aia * deg_to_rad}" arm_mesh="${hex_mesh}" prop_mesh="${prop_cw_mesh}"  cw="true"  prop_size_multiplier="${psm}" cylinder_r="${cylinder_r}" cylinder_l="${cylinder_l}" amass="${amass}"  cla="${cla}" cp="${cp}" area="${area}" rmass="${rmass}" rixx="${rixx}" rixy="${rixy}" rixz="${rixz}" riyy="${riyy}" riyz="${riyz}" rizz="${rizz}" angle="${240 * deg_to_rad}"/>
   <gazebo>
     <link name='imu_link'>
@@ -123,4 +111,16 @@
         </inertia>
       </inertial>
+      <visual name='imu_vis'>
+        <geometry>
+          <box>
+            <size>0.1 0.1 0.1</size>
+          </box>
+        </geometry>
+        <material>
+          <script>
+            <name>Gazebo/DarkGrey</name>
+          </script>
+        </material>
+      </visual>
       <sensor name="imu_sensor" type="imu">
         <pose>0 0 0 3.141593 0 0</pose>
@@ -152,16 +152,25 @@
     </joint>
   </gazebo>
+  <joint name="fire_trigger_servo_joint" type="continuous">
+    <parent link="base_link"/>
+    <child link="fire_trigger_servo_link"/>
+    <origin xyz="0 0 -0.45" rpy="0 0 0"/>
+    <axis xyz="0 0 1"/>
+    <limit effort="1.0" velocity="1.0" lower="-1.5708" upper="1.5708"/>
+    <dynamics damping="0.1" friction="0.1"/>
+  </joint>
+  <xacro:link_creator_i link_name="fire_trigger_servo_link" pose_xyz="0 0 0" pose_rpy="0 0 0" scale_xyz="0.04 0.009 0.009" mass="0.02" ixx="100000000" ixy="0" ixz="0" iyy="0" iyz="0" izz="0"/>
 </robot>
 <!--
 https://ardupilot.org/copter/docs/connect-escs-and-motors.html
-                      X
-                      ^
-                      |
-                      |
-                      | z
-          Y <~~~~~~~~~o~~~~~~~~~~
-                      |
-                      |
-                      |
+            X
+            ^
+            |
+            |
+            | z
+  Y <~~~~~~~o~~~~~~~~
+            |
+            |
+            |
                         (front)
                   120deg            60deg
