Commit message: automated ardupilot plugin component! working!

File: models/copterPIX/ardupilot_plugin.xacro (robot description, xacro)
@@ -1,116 +1,71 @@
 <?xml version="1.0" ?>
 <robot xmlns:xacro="http://www.ros.org/wiki/xacro">
-    <xacro:property name="multiplier" value="800"/>
-    <xacro:property name="multiplier_negative" value="${-1 * multiplier}"/>
-    <gazebo>
-        <plugin name="arducopter_plugin" filename="libArduPilotPlugin.so">
-            <fdm_addr>127.0.0.1</fdm_addr>
-            <fdm_port_in>9002</fdm_port_in>
-            <fdm_port_out>9003</fdm_port_out>
-            <modelXYZToAirplaneXForwardZDown>0 0 0 3.141593 0 0</modelXYZToAirplaneXForwardZDown>
-            <gazeboXYZToNED>0 0 0 3.141593 0 0</gazeboXYZToNED>
-            <imuName>imu_link::imu_sensor</imuName>
-            <connectionTimeoutMaxCount>5</connectionTimeoutMaxCount>
-            <!-- Control channels -->
-            <control channel="0">
-                <type>VELOCITY</type>
-                <offset>0</offset>
-                <p_gain>0.20</p_gain>
-                <i_gain>0</i_gain>
-                <d_gain>0</d_gain>
-                <i_max>0</i_max>
-                <i_min>0</i_min>
-                <cmd_max>2.5</cmd_max>
-                <cmd_min>-2.5</cmd_min>
-                <jointName>rotor_joint_0</jointName>
-                <multiplier>${multiplier_negative}</multiplier>
-                <controlVelocitySlowdownSim>1</controlVelocitySlowdownSim>
-            </control>
-            <control channel="1">
-                <type>VELOCITY</type>
-                <offset>0</offset>
-                <p_gain>0.20</p_gain>
-                <i_gain>0</i_gain>
-                <d_gain>0</d_gain>
-                <i_max>0</i_max>
-                <i_min>0</i_min>
-                <cmd_max>2.5</cmd_max>
-                <cmd_min>-2.5</cmd_min>
-                <jointName>rotor_joint_1</jointName>
-                <multiplier>${multiplier}</multiplier>
-                <controlVelocitySlowdownSim>1</controlVelocitySlowdownSim>
-            </control>
-            <control channel="2">
-                <type>VELOCITY</type>
-                <offset>0</offset>
-                <p_gain>0.20</p_gain>
-                <i_gain>0</i_gain>
-                <d_gain>0</d_gain>
-                <i_max>0</i_max>
-                <i_min>0</i_min>
-                <cmd_max>2.5</cmd_max>
-                <cmd_min>-2.5</cmd_min>
-                <jointName>rotor_joint_2</jointName>
-                <multiplier>${multiplier_negative}</multiplier>
-                <controlVelocitySlowdownSim>1</controlVelocitySlowdownSim>
-            </control>
-            <control channel="3">
-                <type>VELOCITY</type>
-                <offset>0</offset>
-                <p_gain>0.20</p_gain>
-                <i_gain>0</i_gain>
-                <d_gain>0</d_gain>
-                <i_max>0</i_max>
-                <i_min>0</i_min>
-                <cmd_max>2.5</cmd_max>
-                <cmd_min>-2.5</cmd_min>
-                <jointName>rotor_joint_3</jointName>
-                <multiplier>${multiplier}</multiplier>
-                <controlVelocitySlowdownSim>1</controlVelocitySlowdownSim>
-            </control>
-            <control channel="4">
-                <type>VELOCITY</type>
-                <offset>0</offset>
-                <p_gain>0.20</p_gain>
-                <i_gain>0</i_gain>
-                <d_gain>0</d_gain>
-                <i_max>0</i_max>
-                <i_min>0</i_min>
-                <cmd_max>2.5</cmd_max>
-                <cmd_min>-2.5</cmd_min>
-                <jointName>rotor_joint_4</jointName>
-                <multiplier>${multiplier}</multiplier>
-                <controlVelocitySlowdownSim>1</controlVelocitySlowdownSim>
-            </control>
-            <control channel="5">
-                <type>VELOCITY</type>
-                <offset>0</offset>
-                <p_gain>0.20</p_gain>
-                <i_gain>0</i_gain>
-                <d_gain>0</d_gain>
-                <i_max>0</i_max>
-                <i_min>0</i_min>
-                <cmd_max>2.5</cmd_max>
-                <cmd_min>-2.5</cmd_min>
-                <jointName>rotor_joint_5</jointName>
-                <multiplier>${multiplier_negative}</multiplier>
-                <controlVelocitySlowdownSim>1</controlVelocitySlowdownSim>
-            </control>
-            <control channel="6">
-                <jointName>fire_trigger_servo_joint</jointName>
-                <multiplier>1</multiplier>
-                <offset>0</offset>
-                <type>POSITION</type>
-                <p_gain>1.0</p_gain>
-                <i_gain>0</i_gain>
-                <d_gain>0</d_gain>
-                <i_max>0</i_max>
-                <i_min>0</i_min>
-                <cmd_max>2.5</cmd_max>
-                <cmd_min>-2.5</cmd_min>
-                <!-- <controlVelocitySlowdownSim>1</controlVelocitySlowdownSim> -->
-            </control>
-        </plugin>
-    </gazebo>
+    <xacro:macro name="ardupilot_plugin" params="number_of_arms
+                                                type multiplier jointName offset p_gain i_gain d_gain i_max i_min cmd_max cmd_min
+                                                controlVelocitySlowdownSim **extra_ardupilot_plugin_settings">
+        <!-- Define arms! -->
+        <xacro:property name="type_list" value="${type.split(' ')}" />
+        <xacro:property name="multiplier_list" value="${cws.split(' ')}" />
+        <xacro:property name="jointName_list" value="${prop_meshs.split(' ')}" />
+        <gazebo>
+            <plugin name="arducopter_plugin" filename="libArduPilotPlugin.so">
+                <fdm_addr>127.0.0.1</fdm_addr>
+                <fdm_port_in>9002</fdm_port_in>
+                <fdm_port_out>9003</fdm_port_out>
+                <modelXYZToAirplaneXForwardZDown>0 0 0 3.141593 0 0</modelXYZToAirplaneXForwardZDown>
+                <gazeboXYZToNED>0 0 0 3.141593 0 0</gazeboXYZToNED>
+                <imuName>imu_link::imu_sensor</imuName>
+                <connectionTimeoutMaxCount>5</connectionTimeoutMaxCount>
+                <!-- Recursive macro definition -->
+                <xacro:macro name="create_arms" params="i">
+                    <xacro:if value="${i > 0}">
+                        <!-- Here define the arm -->
+                        <xacro:property name="counter" value="${number_of_arms - i}" />
+                        <control channel="${counter}">
+                            <type>${type_list[counter]}</type>
+                            <multiplier>${multiplier_list[counter]}</multiplier>
+                            <jointName>${jointName_list[counter]}</jointName>
+                            <offset>${offset}</offset>
+                            <p_gain>${p_gain}</p_gain>
+                            <i_gain>${i_gain}</i_gain>
+                            <d_gain>${d_gain}</d_gain>
+                            <i_max>${i_max}</i_max>
+                            <i_min>${i_min}</i_min>
+                            <cmd_max>${cmd_max}</cmd_max>
+                            <cmd_min>${cmd_min}</cmd_min>
+                            <controlVelocitySlowdownSim>1</controlVelocitySlowdownSim>
+                            <!-- <controlVelocitySlowdownSim>1</controlVelocitySlowdownSim> -->
+                        </control>
+                        <!-- Recursively call the macro with a decremented count -->
+                        <xacro:create_arms i="${i - 1}"/>
+                    </xacro:if>
+                </xacro:macro>
+                <!-- Initial call to the macro with the desired number of joints -->
+                <xacro:create_arms i="${number_of_arms}"/>
+                <!-- end Define arms! -->
+                <xacro:macro name="extra_channels" params="channel _type _multiplier _jointName _offset _p_gain _i_gain _d_gain
+                                                _i_max _i_min _cmd_max _cmd_min">
+                    <control channel="${channel}">
+                        <type>${_type}</type>
+                        <multiplier>${_multiplier}</multiplier>
+                        <jointName>${_jointName}</jointName>
+                        <offset>${_offset}</offset>
+                        <p_gain>${_p_gain}</p_gain>
+                        <i_gain>${_i_gain}</i_gain>
+                        <d_gain>${_d_gain}</d_gain>
+                        <i_max>${_i_max}</i_max>
+                        <i_min>${_i_min}</i_min>
+                        <cmd_max>${_cmd_max}</cmd_max>
+                        <cmd_min>${_cmd_min}</cmd_min>
+                        <controlVelocitySlowdownSim>1</controlVelocitySlowdownSim>
+                        <!-- <controlVelocitySlowdownSim>1</controlVelocitySlowdownSim> -->
+                    </control>
+                </xacro:macro>
+                <extra_ardupilot_plugin_settings>
+                    <xacro:insert_block name="extra_ardupilot_plugin_settings"/>
+                </extra_ardupilot_plugin_settings>
+            </plugin>
+        </gazebo>
+    </xacro:macro>
 </robot>
   <!-- /// \brief Interface ArduPilot from ardupilot stack
@@ -139,2 +94,102 @@
   /// <connectionTimeoutMaxCount> timeout before giving up on
   ///                             controller synchronization -->
+<!-- <control channel="6">
+    <jointName>fire_trigger_servo_joint</jointName>
+    <multiplier>1</multiplier>
+    <offset>0</offset>
+    <type>POSITION</type>
+    <p_gain>1.0</p_gain>
+    <i_gain>0</i_gain>
+    <d_gain>0</d_gain>
+    <i_max>0</i_max>
+    <i_min>0</i_min>
+    <cmd_max>2.5</cmd_max>
+    <cmd_min>-2.5</cmd_min>
+        <controlVelocitySlowdownSim>1</controlVelocitySlowdownSim>
+</control> -->
+                <!-- Control channels -->
+                <!-- <control channel="0">
+                    <type>VELOCITY</type>
+                    <offset>0</offset>
+                    <p_gain>0.20</p_gain>
+                    <i_gain>0</i_gain>
+                    <d_gain>0</d_gain>
+                    <i_max>0</i_max>
+                    <i_min>0</i_min>
+                    <cmd_max>2.5</cmd_max>
+                    <cmd_min>-2.5</cmd_min>
+                    <jointName>rotor_joint_0</jointName>
+                    <multiplier>${multiplier_negative}</multiplier>
+                    <controlVelocitySlowdownSim>1</controlVelocitySlowdownSim>
+                </control>
+                <control channel="1">
+                    <type>VELOCITY</type>
+                    <offset>0</offset>
+                    <p_gain>0.20</p_gain>
+                    <i_gain>0</i_gain>
+                    <d_gain>0</d_gain>
+                    <i_max>0</i_max>
+                    <i_min>0</i_min>
+                    <cmd_max>2.5</cmd_max>
+                    <cmd_min>-2.5</cmd_min>
+                    <jointName>rotor_joint_1</jointName>
+                    <multiplier>${multiplier}</multiplier>
+                    <controlVelocitySlowdownSim>1</controlVelocitySlowdownSim>
+                </control>
+                <control channel="2">
+                    <type>VELOCITY</type>
+                    <offset>0</offset>
+                    <p_gain>0.20</p_gain>
+                    <i_gain>0</i_gain>
+                    <d_gain>0</d_gain>
+                    <i_max>0</i_max>
+                    <i_min>0</i_min>
+                    <cmd_max>2.5</cmd_max>
+                    <cmd_min>-2.5</cmd_min>
+                    <jointName>rotor_joint_2</jointName>
+                    <multiplier>${multiplier_negative}</multiplier>
+                    <controlVelocitySlowdownSim>1</controlVelocitySlowdownSim>
+                </control>
+                <control channel="3">
+                    <type>VELOCITY</type>
+                    <offset>0</offset>
+                    <p_gain>0.20</p_gain>
+                    <i_gain>0</i_gain>
+                    <d_gain>0</d_gain>
+                    <i_max>0</i_max>
+                    <i_min>0</i_min>
+                    <cmd_max>2.5</cmd_max>
+                    <cmd_min>-2.5</cmd_min>
+                    <jointName>rotor_joint_3</jointName>
+                    <multiplier>${multiplier}</multiplier>
+                    <controlVelocitySlowdownSim>1</controlVelocitySlowdownSim>
+                </control>
+                <control channel="4">
+                    <type>VELOCITY</type>
+                    <offset>0</offset>
+                    <p_gain>0.20</p_gain>
+                    <i_gain>0</i_gain>
+                    <d_gain>0</d_gain>
+                    <i_max>0</i_max>
+                    <i_min>0</i_min>
+                    <cmd_max>2.5</cmd_max>
+                    <cmd_min>-2.5</cmd_min>
+                    <jointName>rotor_joint_4</jointName>
+                    <multiplier>${multiplier}</multiplier>
+                    <controlVelocitySlowdownSim>1</controlVelocitySlowdownSim>
+                </control>
+                <control channel="5">
+                    <type>VELOCITY</type>
+                    <multiplier>${multiplier_negative}</multiplier>
+                    <jointName>rotor_joint_5</jointName>
+                    <offset>0</offset>
+                    <p_gain>0.20</p_gain>
+                    <i_gain>0</i_gain>
+                    <d_gain>0</d_gain>
+                    <i_max>0</i_max>
+                    <i_min>0</i_min>
+                    <cmd_max>2.5</cmd_max>
+                    <cmd_min>-2.5</cmd_min>
+                    <controlVelocitySlowdownSim>1</controlVelocitySlowdownSim>
+                </control>
+                -->

File: models/copterPIX/robot.urdf.xacro (robot description, xacro)
@@ -2,5 +2,4 @@
 <robot name="copterPIX" xmlns:xacro="http://www.ros.org/wiki/xacro">
   <xacro:include filename="$(find drone)/xacros/drone_maker.xacro"/>
-  <xacro:include filename="ardupilot_plugin.xacro"/>
   <xacro:property name="hex_mesh" value="$(find drone)/meshes/hexagonal_prism_height_1_outer_diameter_1.stl"/>
   <xacro:property name="prop_cw_mesh" value="$(find drone)/meshes/iris_prop_cw.dae"/>
@@ -41,4 +40,13 @@
   <xacro:property name="r_mass" value="0.2"/>
   <xacro:property name="r_iner" value="0.000312 0 0 0.0053345 0 0.005363328"/>
+  <xacro:property name="ardu_multiplier" value="800"/>
+  <xacro:property name="ardu_offset" value="0"/>
+  <xacro:property name="ardu_p_gain" value="0.2"/>
+  <xacro:property name="ardu_i_gain" value="0"/>
+  <xacro:property name="ardu_d_gain" value="0"/>
+  <xacro:property name="ardu_i_max" value="0"/>
+  <xacro:property name="ardu_i_min" value="0"/>
+  <xacro:property name="ardu_cmd_max" value="2.5"/>
+  <xacro:property name="ardu_cmd_min" value="-2.5"/>
   <xacro:drone_maker base_mesh="${base_mesh}" base_pose_xyz ="${base_pose_xyz}" base_pose_rpy="${base_pose_rpy}" base_scale_xyz="${base_scale_xyz}"
                      base_center_of_mass="${base_center_of_mass}" base_mass="${base_mass}" base_iner="${base_iner}"
@@ -47,5 +55,13 @@
                      arm_incline_angle="${arm_incline_angle}" arm_mesh="${arm_mesh}" prop_size_multiplier="${prop_size_multiplier}"
                      cylinder_d="${cylinder_d}" cylinder_l="${cylinder_l}" a_mass="${a_mass}" a_iner="${a_iner}"
-                     cla="${cla}" cp="${cp}" area="${area}" r_mass="${r_mass}"  r_iner="${r_iner}">
+                     cla="${cla}" cp="${cp}" area="${area}" r_mass="${r_mass}"  r_iner="${r_iner}"
+                     ardu_multiplier="${ardu_multiplier}" ardu_offset="${ardu_offset}"
+                     ardu_p_gain="${ardu_p_gain}" ardu_i_gain="${ardu_i_gain}" ardu_d_gain="${ardu_d_gain}"
+                     ardu_i_max="${ardu_i_max}" ardu_i_min="${ardu_i_min}" ardu_cmd_max="${ardu_cmd_max}" ardu_cmd_min="${ardu_cmd_min}">
+    <extra_ardupilot_plugin_settings>
+      <xacro:extra_channel channel="6" _type="POSITION" _multiplier="1" _jointName="fire_trigger_servo_joint"
+                                          _offset="0" _p_gain="1" _i_gain="0" _d_gain="0"
+                                          _i_max="0" _i_min="0" _cmd_max="2.5" _cmd_min="-2.5"/>
+    </extra_ardupilot_plugin_settings>
   </xacro:drone_maker>
   <joint name="leg_0_link_joint" type="fixed">

File: models/iris/robot.urdf.xacro (robot description, xacro)
@@ -2,5 +2,4 @@
 <robot name="copterPIX" xmlns:xacro="http://www.ros.org/wiki/xacro">
   <xacro:include filename="$(find drone)/xacros/drone_maker.xacro"/>
-  <xacro:include filename="ardupilot_plugin.xacro"/>
   <xacro:property name="hex_mesh" value="$(find drone)/meshes/hexagonal_prism_height_1_outer_diameter_1.stl"/>
   <xacro:property name="prop_cw_mesh" value="$(find drone)/meshes/iris_prop_cw.dae"/>
@@ -15,5 +14,5 @@
   <xacro:property name="number_of_arms" value="4"/>
   <xacro:property name="arm_angles" value="45 225 135 315"/>
-  <xacro:property name="cws" value="false false true true"/>
+  <xacro:property name="cws" value="0 0 1 1"/>
   <xacro:property name="prop_meshs" value="${prop_ccw_mesh} ${prop_ccw_mesh} ${prop_cw_mesh} ${prop_cw_mesh}"/>
   <xacro:property name="dis_from_center" value="0.08"/>
@@ -32,4 +31,13 @@
   <xacro:property name="r_mass" value="0.025"/>
   <xacro:property name="r_iner" value="9.75e-06 0 0 0.000166704 0 0.000167604"/>
+  <xacro:property name="ardu_multiplier" value="800"/>
+  <xacro:property name="ardu_offset" value="0"/>
+  <xacro:property name="ardu_p_gain" value="0.2"/>
+  <xacro:property name="ardu_i_gain" value="0"/>
+  <xacro:property name="ardu_d_gain" value="0"/>
+  <xacro:property name="ardu_i_max" value="0"/>
+  <xacro:property name="ardu_i_min" value="0"/>
+  <xacro:property name="ardu_cmd_max" value="2.5"/>
+  <xacro:property name="ardu_cmd_min" value="-2.5"/>
   <xacro:drone_maker base_mesh="${base_mesh}" base_pose_xyz ="${base_pose_xyz}" base_pose_rpy="${base_pose_rpy}" base_scale_xyz="${base_scale_xyz}"
                      base_center_of_mass="${base_center_of_mass}" base_mass="${base_mass}" base_iner="${base_iner}"
@@ -38,5 +46,10 @@
                      arm_incline_angle="${arm_incline_angle}" arm_mesh="${arm_mesh}" prop_size_multiplier="${prop_size_multiplier}"
                      cylinder_d="${cylinder_d}" cylinder_l="${cylinder_l}" a_mass="${a_mass}" a_iner="${a_iner}"
-                     cla="${cla}" cp="${cp}" area="${area}" r_mass="${r_mass}"  r_iner="${r_iner}">
+                     cla="${cla}" cp="${cp}" area="${area}" r_mass="${r_mass}"  r_iner="${r_iner}"
+                     ardu_multiplier="${ardu_multiplier}" ardu_offset="${ardu_offset}"
+                     ardu_p_gain="${ardu_p_gain}" ardu_i_gain="${ardu_i_gain}" ardu_d_gain="${ardu_d_gain}"
+                     ardu_i_max="${ardu_i_max}" ardu_i_min="${ardu_i_min}" ardu_cmd_max="${ardu_cmd_max}" ardu_cmd_min="${ardu_cmd_min}">
+    <extra_ardupilot_plugin_settings>
+    </extra_ardupilot_plugin_settings>
   </xacro:drone_maker>
 </robot>

File: xacros/drone_maker.xacro (robot description, xacro)
@@ -2,9 +2,13 @@
 <robot xmlns:xacro="http://www.ros.org/wiki/xacro">
     <xacro:include filename="macro.xacro"/>
+    <xacro:include filename="ardupilot_plugin.xacro"/>
     <xacro:property name="deg_to_rad" value="0.0174533"/>
     <xacro:macro name="drone_maker" params="base_mesh:='Box' base_pose_xyz:='0 0 0' base_pose_rpy:='0 0 0' base_scale_xyz:='0.4 0.4 0.04' base_center_of_mass:='0 0 0' base_mass base_iner:='None'
                                             number_of_arms arm_angles cws prop_meshs
                                             dis_from_center length diameter arm_incline_angle:='0' arm_mesh prop_size_multiplier
-                                            cylinder_d cylinder_l a_mass a_iner:='None' cla cp area r_mass r_iner">
+                                            cylinder_d cylinder_l a_mass a_iner:='None' cla cp area r_mass r_iner
+                                            ardu_multiplier ardu_offset ardu_p_gain ardu_i_gain ardu_d_gain
+                                            ardu_i_max ardu_i_min ardu_cmd_max ardu_cmd_min
+                                            **extra_ardupilot_plugin_settings">
         <xacro:property name="base_pose_rpy_list" value="${base_pose_rpy.split(' ')}" />
         <xacro:property name="base_pose_rpy_converted" value="${float(base_pose_rpy_list[0]) * deg_to_rad} ${float(base_pose_rpy_list[1]) * deg_to_rad} ${float(base_pose_rpy_list[2]) * deg_to_rad}" />
@@ -12,5 +16,4 @@
         <xacro:link_creator_i link_name="base_link" pose_xyz="${base_pose_xyz}" pose_rpy="${base_pose_rpy_converted}" mesh_path="${base_mesh}"
                                 scale_xyz="${base_scale_xyz}" center_mass_xyz="${base_center_of_mass}" mass="${base_mass}" iner="${base_iner}"/>
-        <!-- Define arms! -->
         <xacro:property name="arm_angle_list" value="${arm_angles.split(' ')}" />
         <xacro:property name="cw_list" value="${cws.split(' ')}" />
@@ -65,4 +68,12 @@
         </gazebo>
         <!-- end Define IMU! -->
+        <!-- Define ardupilot_plugin! -->
+        <xacro:ardupilot_plugin number_of_arms="${number_of_arms}" multiplier="${ardu_multiplier}" cws="${cws}"
+                                offset="${ardu_offset}" p_gain="${ardu_p_gain}" i_gain="${ardu_i_gain}" d_gain="${ardu_d_gain}"
+                                i_max="${ardu_i_max}" i_min="${ardu_i_min}" cmd_max="${ardu_cmd_max}" cmd_min="${ardu_cmd_min}">
+            <extra_ardupilot_plugin_settings>
+                <xacro:insert_block name="extra_ardupilot_plugin_settings"/>
+            </extra_ardupilot_plugin_settings>
+        </xacro:ardupilot_plugin>
     </xacro:macro>
 </robot>
