Commit message: edited robot.urdf.xacro

File: models/copterPIX/robot.urdf.xacro (robot description, xacro)
@@ -1,9 +1,6 @@
-<?xml version="1.0"?>
+<!-- <?xml version="1.0"?>
 <robot name="copterPIX" xmlns:xacro="http://www.ros.org/wiki/xacro">
-  <!-- Base link -->
   <link name="base_link">
-    <!-- You can leave this link empty if you don't need a specific geometry or inertial properties for the base -->
   </link>
-  <!-- Drone Core link -->
   <link name="core_link">
     <visual>
@@ -25,5 +22,4 @@
     </inertial>
   </link>
-  <!-- Joint (fixed) -->
   <joint name="fixed_joint" type="fixed">
     <parent link="base_link"/>
@@ -35,4 +31,94 @@
   </gazebo>
 </robot>
+ -->
+<!--
+<?xml version="1.0"?>
+<robot xmlns:xacro="http://www.ros.org/wiki/xacro"  name="robot">
+    <gazebo>
+        <plugin name="diff_drive" filename="libgazebo_ros_diff_drive.so">
+            <left_joint>left_wheel_joint</left_joint>
+            <right_joint>right_wheel_joint</right_joint>
+            <wheel_separation>0.35</wheel_separation>
+            <wheel_diameter>0.1</wheel_diameter>
+            <max_wheel_torque>200</max_wheel_torque>
+            <max_wheel_acceleration>10.0</max_wheel_acceleration>
+            <odometry_frame>odom</odometry_frame>
+            <robot_base_frame>base_link</robot_base_frame>
+            <publish_odom>true</publish_odom>
+            <publish_odom_tf>true</publish_odom_tf>
+            <publish_wheel_tf>true</publish_wheel_tf>
+        </plugin>
+    </gazebo>
+</robot> -->
+<?xml version="1.0" ?>
+<robot name="copterPIX" xmlns:xacro="http://www.ros.org/wiki/xacro">
+   <!-- Base link -->
+  <link name="base_link">
+    <!-- You can leave this link empty if you don't need a specific geometry or inertial properties for the base -->
+  </link>
+  <!-- Joint (fixed) -->
+  <joint name="fixed_joint" type="fixed">
+    <parent link="base_link"/>
+    <child link="core_link"/>
+    <origin xyz="0 0 0" rpy="0 0 0"/>
+  </joint>
+  <!-- Other definitions like base link, sensors, etc. -->
+  <!-- Define the drone arms using the macro -->
+  <xacro:drone_arm name="arm_1" joint_name="rotor_0_joint" propeller_link="prop_0_link" control_channel="0" multiplier="838" />
+  <xacro:drone_arm name="arm_2" joint_name="rotor_1_joint" propeller_link="prop_1_link" control_channel="1" multiplier="838" />
+  <xacro:drone_arm name="arm_3" joint_name="rotor_2_joint" propeller_link="prop_2_link" control_channel="2" multiplier="-838" />
+  <xacro:drone_arm name="arm_4" joint_name="rotor_3_joint" propeller_link="prop_3_link" control_channel="3" multiplier="-838" />
+  <!-- Plugin encapsulating all control channels -->
+  <gazebo>
+    <plugin name="arducopter_plugin" filename="libArduPilotPlugin.so">
+        <fdm_addr>127.0.0.1</fdm_addr>
+        <fdm_port_in>9002</fdm_port_in>
+        <fdm_port_out>9003</fdm_port_out>
+        <modelXYZToAirplaneXForwardZDown>0 0 0 3.141593 0 0</modelXYZToAirplaneXForwardZDown>
+        <gazeboXYZToNED>0 0 0 3.141593 0 0</gazeboXYZToNED>
+        <imuName>iris_demo::iris::iris/imu_link::imu_sensor</imuName>
+        <connectionTimeoutMaxCount>5</connectionTimeoutMaxCount>
+        <!-- Control channels -->
+        <xacro:control_channel channel="0" joint_name="rotor_0_joint" multiplier="-838" />         <!--cw-->
+        <xacro:control_channel channel="1" joint_name="rotor_1_joint" multiplier="838" />         <!--cw-->
+        <xacro:control_channel channel="2" joint_name="rotor_2_joint" multiplier="-838" />         <!--cw-->
+        <xacro:control_channel channel="3" joint_name="rotor_3_joint" multiplier="838" />         <!--cw-->
+        <xacro:control_channel channel="4" joint_name="rotor_4_joint" multiplier="-838" />
+        <xacro:control_channel channel="5" joint_name="rotor_5_joint" multiplier="838" />
+    </plugin>
+  </gazebo>
+  <xacro:macro name="control_channel" params="channel joint_name multiplier">
+    <control channel="${channel}">
+      <type>VELOCITY</type>
+      <offset>0</offset>
+      <p_gain>0.20</p_gain>
+      <i_gain>0</i_gain>
+      <d_gain>0</d_gain>
+      <i_max>0</i_max>
+      <i_min>0</i_min>
+      <cmd_max>2.5</cmd_max>
+      <cmd_min>-2.5</cmd_min>
+      <jointName>${joint_name}</jointName>
+      <multiplier>${multiplier}</multiplier>
+      <controlVelocitySlowdownSim>1</controlVelocitySlowdownSim>
+    </control>
+  </xacro:macro>
+</robot>
+<!--
+https://ardupilot.org/copter/docs/connect-escs-and-motors.html
+              cw (3)           ccw (5)
+                \               /
+                 \             /
+                   \         /
+                    \       /
+                      \   /
+      ccw(2) ~~~~~~~~~~~~~~~~~~~~~~~~ cw(1)
+                      /   \
+                    /       \
+                   /         \
+                 /             \
+                /               \
+              cw (6)           ccw (4)
+ -->
 <!-- <?xml version="1.0"?>
 <robot name="drone" xmlns:xacro="http://www.ros.org/wiki/xacro">

Commit message: arm.xacro progress and little bit more

File: models/copterPIX/robot.urdf.xacro (robot description, xacro)
@@ -34,5 +34,5 @@
 <!--
 <?xml version="1.0"?>
-<robot xmlns:xacro="http://www.ros.org/wiki/xacro"  name="robot">
+<robot xmlns:xacro="http://www.ros.org/wiki/xacro" name="robot">
     <gazebo>
         <plugin name="diff_drive" filename="libgazebo_ros_diff_drive.so">
@@ -53,5 +53,6 @@
 <?xml version="1.0" ?>
 <robot name="copterPIX" xmlns:xacro="http://www.ros.org/wiki/xacro">
-   <!-- Base link -->
+  <xacro:include filename="inertial_macros.xacro"/>
+  <!-- Base link -->
   <link name="base_link">
     <!-- You can leave this link empty if you don't need a specific geometry or inertial properties for the base -->
@@ -63,30 +64,52 @@
     <origin xyz="0 0 0" rpy="0 0 0"/>
   </joint>
+  <link name="core_link">
+    <visual>
+      <geometry>
+        <box size="1 1 1"/>
+      </geometry>
+      <material name="red">
+        <color rgba="0.8 0.1 0.1 1.0"/>
+      </material>
+    </visual>
+    <collision>
+      <geometry>
+        <box size="1 1 1"/>
+      </geometry>
+    </collision>
+    <inertial>
+      <mass value="1.0"/>
+      <inertia ixx="0.1" ixy="0.0" ixz="0.0" iyy="0.1" iyz="0.0" izz="0.1"/>
+    </inertial>
+  </link>
   <!-- Other definitions like base link, sensors, etc. -->
   <!-- Define the drone arms using the macro -->
-  <xacro:drone_arm name="arm_1" joint_name="rotor_0_joint" propeller_link="prop_0_link" control_channel="0" multiplier="838" />
-  <xacro:drone_arm name="arm_2" joint_name="rotor_1_joint" propeller_link="prop_1_link" control_channel="1" multiplier="838" />
-  <xacro:drone_arm name="arm_3" joint_name="rotor_2_joint" propeller_link="prop_2_link" control_channel="2" multiplier="-838" />
-  <xacro:drone_arm name="arm_4" joint_name="rotor_3_joint" propeller_link="prop_3_link" control_channel="3" multiplier="-838" />
+  <xacro:property name="angle_in_radians" value="0.628319" />   <!--60 degrees in radians-->
+  <xacro:drone_arm arm_link="arm_link_0" rotor_joint="rotor_joint_0" propeller_link="prop_link_0" parent_link="core_link" angle="${angle_in_radians * 3 + angle_in_radians / 2}"/>
+  <xacro:drone_arm arm_link="arm_link_1" rotor_joint="rotor_joint_1" propeller_link="prop_link_1" parent_link="core_link" angle="${angle_in_radians * 3 + angle_in_radians / 2}"/>
+  <xacro:drone_arm arm_link="arm_link_2" rotor_joint="rotor_joint_2" propeller_link="prop_link_2" parent_link="core_link" angle="${angle_in_radians * 3 + angle_in_radians / 2}"/>
+  <xacro:drone_arm arm_link="arm_link_3" rotor_joint="rotor_joint_3" propeller_link="prop_link_3" parent_link="core_link" angle="${angle_in_radians * 3 + angle_in_radians / 2}"/>
+  <xacro:drone_arm arm_link="arm_link_4" rotor_joint="rotor_joint_4" propeller_link="prop_link_4" parent_link="core_link" angle="${angle_in_radians * 3 + angle_in_radians / 2}"/>
+  <xacro:drone_arm arm_link="arm_link_5" rotor_joint="rotor_joint_5" propeller_link="prop_link_5" parent_link="core_link" angle="${angle_in_radians * 3 + angle_in_radians / 2}"/>
   <!-- Plugin encapsulating all control channels -->
   <gazebo>
     <plugin name="arducopter_plugin" filename="libArduPilotPlugin.so">
-        <fdm_addr>127.0.0.1</fdm_addr>
-        <fdm_port_in>9002</fdm_port_in>
-        <fdm_port_out>9003</fdm_port_out>
-        <modelXYZToAirplaneXForwardZDown>0 0 0 3.141593 0 0</modelXYZToAirplaneXForwardZDown>
-        <gazeboXYZToNED>0 0 0 3.141593 0 0</gazeboXYZToNED>
-        <imuName>iris_demo::iris::iris/imu_link::imu_sensor</imuName>
-        <connectionTimeoutMaxCount>5</connectionTimeoutMaxCount>
-        <!-- Control channels -->
-        <xacro:control_channel channel="0" joint_name="rotor_0_joint" multiplier="-838" />         <!--cw-->
-        <xacro:control_channel channel="1" joint_name="rotor_1_joint" multiplier="838" />         <!--cw-->
-        <xacro:control_channel channel="2" joint_name="rotor_2_joint" multiplier="-838" />         <!--cw-->
-        <xacro:control_channel channel="3" joint_name="rotor_3_joint" multiplier="838" />         <!--cw-->
-        <xacro:control_channel channel="4" joint_name="rotor_4_joint" multiplier="-838" />
-        <xacro:control_channel channel="5" joint_name="rotor_5_joint" multiplier="838" />
+      <fdm_addr>127.0.0.1</fdm_addr>
+      <fdm_port_in>9002</fdm_port_in>
+      <fdm_port_out>9003</fdm_port_out>
+      <modelXYZToAirplaneXForwardZDown>0 0 0 3.141593 0 0</modelXYZToAirplaneXForwardZDown>
+      <gazeboXYZToNED>0 0 0 3.141593 0 0</gazeboXYZToNED>
+      <imuName>iris_demo::iris::iris/imu_link::imu_sensor</imuName>
+      <connectionTimeoutMaxCount>5</connectionTimeoutMaxCount>
+      <!-- Control channels -->
+      <xacro:control_channel channel="0" rotor_joint="rotor_joint_0" multiplier="-838" /> <!--cw-->
+      <xacro:control_channel channel="1" rotor_joint="rotor_joint_1" multiplier="838" /> <!--ccw-->
+      <xacro:control_channel channel="2" rotor_joint="rotor_joint_2" multiplier="-838" /> <!--cw-->
+      <xacro:control_channel channel="3" rotor_joint="rotor_joint_3" multiplier="838" /> <!--ccw-->
+      <xacro:control_channel channel="4" rotor_joint="rotor_joint_4" multiplier="-838" /> <!--cw-->
+      <xacro:control_channel channel="5" rotor_joint="rotor_joint_5" multiplier="838" /> <!--ccw-->
     </plugin>
   </gazebo>
-  <xacro:macro name="control_channel" params="channel joint_name multiplier">
+  <xacro:macro name="control_channel" params="channel rotor_joint multiplier">
     <control channel="${channel}">
       <type>VELOCITY</type>
@@ -99,5 +122,5 @@
       <cmd_max>2.5</cmd_max>
       <cmd_min>-2.5</cmd_min>
-      <jointName>${joint_name}</jointName>
+      <jointName>${rotor_joint}</jointName>
       <multiplier>${multiplier}</multiplier>
       <controlVelocitySlowdownSim>1</controlVelocitySlowdownSim>
@@ -107,5 +130,6 @@
 <!--
 https://ardupilot.org/copter/docs/connect-escs-and-motors.html
-              cw (3)           ccw (5)
+                     (front)
+              cw (2)           ccw (4)
                 \               /
                  \             /
@@ -113,5 +137,5 @@
                     \       /
                       \   /
-      ccw(2) ~~~~~~~~~~~~~~~~~~~~~~~~ cw(1)
+      ccw(1) ~~~~~~~~~~~~~~~~~~~~~~~~ cw(0)
                       /   \
                     /       \
@@ -119,5 +143,5 @@
                  /             \
                 /               \
-              cw (6)           ccw (4)
+              cw (5)           ccw (3)
  -->
 <!-- <?xml version="1.0"?>

File: xacros/arms.xacro (robot description, xacro)
@@ -1,4 +1,23 @@
 <?xml version="1.0"?>
-<robot xmlns:xacro="http://www.ros.org/wiki/xacro" >
+<robot xmlns:xacro="http://www.ros.org/wiki/xacro">
+    <xacro:macro name="drone_arm" params="arm_link rotor_joint propeller_link parent_link angle">
+        <joint name="fixed_joint" type="fixed">
+            <parent link="${parent_link}"/>
+            <child link="${arm_link}"/>
+            <origin xyz="0 0 0" rpy="0 0 ${angle}"/>
+        </joint>
+        <link name="${arm_link}">
+            <!-- Define the link properties here -->
+        </link>
+        <joint name="${rotor_joint}" type="fixed">
+            <!-- Define the joint properties here -->
+        </joint>
+        <link name="${propeller_link}">
+            <!-- Define the propeller properties here -->
+        </link>
+        <plugin name="lift_drag_plugin" filename="libLiftDragPlugin.so">
+            <!-- Define the lift drag plugin properties here -->
+        </plugin>
+    </xacro:macro>
     <!-- Specify some standard inertial calculations https://en.wikipedia.org/wiki/List_of_moments_of_inertia -->
     <!-- These make use of xacro's mathematical functionality -->
@@ -7,7 +26,5 @@
             <xacro:insert_block name="origin"/>
             <mass value="${mass}" />
-            <inertia ixx="${(2/5) * mass * (radius*radius)}" ixy="0.0" ixz="0.0"
-                    iyy="${(2/5) * mass * (radius*radius)}" iyz="0.0"
-                    izz="${(2/5) * mass * (radius*radius)}" />
+            <inertia ixx="${(2/5) * mass * (radius*radius)}" ixy="0.0" ixz="0.0" iyy="${(2/5) * mass * (radius*radius)}" iyz="0.0" izz="${(2/5) * mass * (radius*radius)}" />
         </inertial>
     </xacro:macro>
@@ -16,7 +33,5 @@
             <xacro:insert_block name="origin"/>
             <mass value="${mass}" />
-            <inertia ixx="${(1/12) * mass * (y*y+z*z)}" ixy="0.0" ixz="0.0"
-                    iyy="${(1/12) * mass * (x*x+z*z)}" iyz="0.0"
-                    izz="${(1/12) * mass * (x*x+y*y)}" />
+            <inertia ixx="${(1/12) * mass * (y*y+z*z)}" ixy="0.0" ixz="0.0" iyy="${(1/12) * mass * (x*x+z*z)}" iyz="0.0" izz="${(1/12) * mass * (x*x+y*y)}" />
         </inertial>
     </xacro:macro>
@@ -25,7 +40,5 @@
             <xacro:insert_block name="origin"/>
             <mass value="${mass}" />
-            <inertia ixx="${(1/12) * mass * (3*radius*radius + length*length)}" ixy="0.0" ixz="0.0"
-                    iyy="${(1/12) * mass * (3*radius*radius + length*length)}" iyz="0.0"
-                    izz="${(1/2) * mass * (radius*radius)}" />
+            <inertia ixx="${(1/12) * mass * (3*radius*radius + length*length)}" ixy="0.0" ixz="0.0" iyy="${(1/12) * mass * (3*radius*radius + length*length)}" iyz="0.0" izz="${(1/2) * mass * (radius*radius)}" />
         </inertial>
     </xacro:macro> -->

Commit message: big changes in copterPIX

File: models/copterPIX/robot.urdf.xacro (robot description, xacro)
@@ -53,5 +53,5 @@
 <?xml version="1.0" ?>
 <robot name="copterPIX" xmlns:xacro="http://www.ros.org/wiki/xacro">
-  <xacro:include filename="inertial_macros.xacro"/>
+  <xacro:include filename="./../../STLs/macro.xacro"/>
   <!-- Base link -->
   <link name="base_link">
@@ -64,5 +64,5 @@
     <origin xyz="0 0 0" rpy="0 0 0"/>
   </joint>
-  <link name="core_link">
+  <!-- <link name="core_link">
     <visual>
       <geometry>
@@ -82,5 +82,6 @@
       <inertia ixx="0.1" ixy="0.0" ixz="0.0" iyy="0.1" iyz="0.0" izz="0.1"/>
     </inertial>
-  </link>
+  </link> -->
+  <xacro:link_creator name="core_link" pose_xyz="0 0 60" pose_rpy="0 0 0" mesh_path="./../../STLs/hexagonal_prism_height_1_outer_diameter_1.stl" scale_xyz="0.4 0.4 0.04" mass="1.0" ixx="0.1" ixy="0.0" ixz="0.0" iyy="0.1" iyz="0.0" izz="0.1"/>
   <!-- Other definitions like base link, sensors, etc. -->
   <!-- Define the drone arms using the macro -->

File: models/simple_box/robot.urdf.xacro (robot description, xacro)
@@ -3,8 +3,54 @@
   <!-- Base link -->
   <link name="base_link">
+  </link>
+  <link name="base_linkaa">
+    <visual>
+      <geometry>
+        <box size="1 1 1"/>
+      </geometry>
+      <material name="red">
+        <color rgba="0.8 0.1 0.1 1.0"/>
+      </material>
+      <origin xyz="30 0 0" rpy="0 0 0"/>
+    </visual>
+    <collision>
+      <geometry>
+        <box size="1 1 1"/>
+      </geometry>
+    </collision>
+    <inertial>
+      <mass value="1.0"/>
+      <inertia ixx="0.1" ixy="0.0" ixz="0.0" iyy="0.1" iyz="0.0" izz="0.1"/>
+    </inertial>
+  </link>
+  <joint name="fixed_joint" type="fixed">
+    <parent link="base_link"/>
+    <child link="base_linkaa"/>
+  </joint>
+  <!-- <link name="base_linkaaa"> -->
+    <!-- <pose>30 0 0 0 0 0</pose> -->
+    <!-- <origin xyz="30 0 0 0" rpy="0 0 0 0"/> -->
     <!-- You can leave this link empty if you don't need a specific geometry or inertial properties for the base -->
-  </link>
+<!--
+     <visual>
+      <geometry>
+        <box size="1 1 1"/>
+      </geometry>
+      <material name="red">
+        <color rgba="0.8 0.1 0.1 1.0"/>
+      </material>
+    </visual>
+    <collision>
+      <geometry>
+        <box size="1 1 1"/>
+      </geometry>
+    </collision>
+    <inertial>
+      <mass value="1.0"/>
+      <inertia ixx="0.1" ixy="0.0" ixz="0.0" iyy="0.1" iyz="0.0" izz="0.1"/>
+    </inertial>
+  </link> -->
   <!-- Box link -->
-  <link name="box_link">
+  <!-- <link name="box_link">
     <visual>
       <geometry>
@@ -24,12 +70,12 @@
       <inertia ixx="0.1" ixy="0.0" ixz="0.0" iyy="0.1" iyz="0.0" izz="0.1"/>
     </inertial>
-  </link>
+  </link> -->
   <!-- Joint (fixed) -->
-  <joint name="fixed_joint" type="fixed">
+  <!-- <joint name="fixed_joint" type="fixed">
     <parent link="base_link"/>
     <child link="box_link"/>
     <origin xyz="0 0 0" rpy="0 0 0"/>
-  </joint>
-  <!-- <gazebo reference="box_link">
+  </joint> -->
+  <!-- <gazebo reference="base_linka">
     <material> Gazebo/Red</material>
   </gazebo> -->

File: xacros/macro.xacro (robot description, xacro)
@@ -20,4 +20,52 @@
         </plugin>
     </xacro:macro>
+    <xacro:macro name="link_creator" params="link_name pose_xyz pose_rpy mesh_path scale_xyz mass ixx ixy ixz iyy iyz izz">
+        <link name="${link_name}">
+            <visual>
+                <geometry>
+                    <mesh filename="${mesh_path}" scale="${scale_xyz}"/>
+                </geometry>
+                <material name="red">
+                    <color rgba="0.8 0.1 0.1 1.0"/>
+                </material>
+                <origin xyz="${pose_xyz }" rpy="${pose_rpy}"/>
+            </visual>
+            <collision>
+                <geometry>
+                    <mesh filename="${mesh_path}" scale="${scale_xyz}"/>
+                </geometry>
+                <origin xyz="${pose_xyz }" rpy="${pose_rpy}"/>
+            </collision>
+            <inertial>
+                <mass value="${mass}"/>
+                <inertia ixx="${ixx}" ixy="${ixy}" ixz="${ixz}" iyy="${iyy}" iyz="${iyz}" izz="${izz}"/>
+            </inertial>
+        </link>
+    </xacro:macro>
+    <xacro:macro name="temp" params="link_name">
+        <link name="${link_name}">
+            <visual>
+                <geometry>
+                    <box size="1 1 1"/>
+                </geometry>
+                <material name="red">
+                    <color rgba="0.8 0.1 0.1 1.0"/>
+                </material>
+            </visual>
+            <collision>
+                <geometry>
+                    <box size="1 1 1"/>
+                </geometry>
+            </collision>
+            <inertial>
+                <mass value="1.0"/>
+                <inertia ixx="0.1" ixy="0.0" ixz="0.0" iyy="0.1" iyz="0.0" izz="0.1"/>
+            </inertial>
+        </link>
+        <gazebo reference="${link_name}">
+            <material> Gazebo/Red</material>
+        </gazebo>
+    </xacro:macro>
+</robot>
     <!-- Specify some standard inertial calculations https://en.wikipedia.org/wiki/List_of_moments_of_inertia -->
     <!-- These make use of xacro's mathematical functionality -->
@@ -43,3 +91,2 @@
         </inertial>
     </xacro:macro> -->
-</robot>
