Commit message: plugins added both lift and ardu, fixed the legs

File: models/copterPIX/robot.urdf.xacro (robot description, xacro)
@@ -2,4 +2,5 @@
 <robot name="copterPIX" xmlns:xacro="http://www.ros.org/wiki/xacro">
   <xacro:include filename="$(find drone)/xacros/macro.xacro"/>
+  <xacro:include filename="ardupilot_plugin.xacro"/>
   <!-- Base link -->
   <link name="base_link">
@@ -17,38 +18,71 @@
     <child link="leg_0_link"/>
   </joint>
-  <xacro:link_creator link_name="leg_0_link" pose_xyz="0.1 0.145 -0.3" pose_rpy="0.185 0 0" mesh_path="$(find drone)/STLs/hexagonal_prism_height_1_outer_diameter_1.stl" scale_xyz="0.024 0.024 0.6" mass="1.0" ixx="0.1" ixy="0.0" ixz="0.0" iyy="0.1" iyz="0.0" izz="0.1"/>
+  <xacro:link_creator link_name="leg_0_link" pose_xyz="0 0.198 -0.305" pose_rpy="0.305 0 0" mesh_path="$(find drone)/STLs/hexagonal_prism_height_1_outer_diameter_1.stl" scale_xyz="0.024 0.024 0.61" mass="1.0" ixx="0.1" ixy="0.0" ixz="0.0" iyy="0.1" iyz="0.0" izz="0.1"/>
   <joint name="leg_1_link_joint" type="fixed">
     <parent link="core_link"/>
     <child link="leg_1_link"/>
   </joint>
-  <xacro:link_creator link_name="leg_1_link" pose_xyz="0.1 -0.145 -0.3" pose_rpy="-0.185 0 0" mesh_path="$(find drone)/STLs/hexagonal_prism_height_1_outer_diameter_1.stl" scale_xyz="0.024 0.024 0.6" mass="1.0" ixx="0.1" ixy="0.0" ixz="0.0" iyy="0.1" iyz="0.0" izz="0.1"/>
-  <joint name="leg_2_link_joint" type="fixed">
-    <parent link="core_link"/>
-    <child link="leg_2_link"/>
-  </joint>
-  <xacro:link_creator link_name="leg_2_link" pose_xyz="-0.1 -0.145 -0.3" pose_rpy="-0.185 0 0" mesh_path="$(find drone)/STLs/hexagonal_prism_height_1_outer_diameter_1.stl" scale_xyz="0.024 0.024 0.6" mass="1.0" ixx="0.1" ixy="0.0" ixz="0.0" iyy="0.1" iyz="0.0" izz="0.1"/>
-  <joint name="leg_3_link_joint" type="fixed">
-    <parent link="core_link"/>
-    <child link="leg_3_link"/>
-  </joint>
-  <xacro:link_creator link_name="leg_3_link" pose_xyz="-0.1 0.145 -0.3" pose_rpy="0.185 0 0" mesh_path="$(find drone)/STLs/hexagonal_prism_height_1_outer_diameter_1.stl" scale_xyz="0.024 0.024 0.6" mass="1.0" ixx="0.1" ixy="0.0" ixz="0.0" iyy="0.1" iyz="0.0" izz="0.1"/>
+  <xacro:link_creator link_name="leg_1_link" pose_xyz="0 -0.198 -0.305" pose_rpy="-0.305 0 0" mesh_path="$(find drone)/STLs/hexagonal_prism_height_1_outer_diameter_1.stl" scale_xyz="0.024 0.024 0.61" mass="1.0" ixx="0.1" ixy="0.0" ixz="0.0" iyy="0.1" iyz="0.0" izz="0.1"/>
   <joint name="feet_0_link_joint" type="fixed">
     <parent link="core_link"/>
     <child link="feet_0_link"/>
   </joint>
-  <xacro:link_creator link_name="feet_0_link" pose_xyz="0 0.2 -0.6" pose_rpy="0 1.57079633 0" mesh_path="$(find drone)/STLs/hexagonal_prism_height_1_outer_diameter_1.stl" scale_xyz="0.024 0.024 0.6" mass="1.0" ixx="0.1" ixy="0.0" ixz="0.0" iyy="0.1" iyz="0.0" izz="0.1"/>
+  <xacro:link_creator link_name="feet_0_link" pose_xyz="0 0.29 -0.6" pose_rpy="0 1.57079633 0" mesh_path="$(find drone)/STLs/hexagonal_prism_height_1_outer_diameter_1.stl" scale_xyz="0.024 0.024 0.58" mass="1.0" ixx="0.1" ixy="0.0" ixz="0.0" iyy="0.1" iyz="0.0" izz="0.1"/>
   <joint name="feet_1_link_joint" type="fixed">
     <parent link="core_link"/>
     <child link="feet_1_link"/>
   </joint>
-  <xacro:link_creator link_name="feet_1_link" pose_xyz="0 -0.2 -0.6" pose_rpy="0 1.57079633 0" mesh_path="$(find drone)/STLs/hexagonal_prism_height_1_outer_diameter_1.stl" scale_xyz="0.024 0.024 0.6" mass="1.0" ixx="0.1" ixy="0.0" ixz="0.0" iyy="0.1" iyz="0.0" izz="0.1"/>
+  <xacro:link_creator link_name="feet_1_link" pose_xyz="0 -0.29 -0.6" pose_rpy="0 1.57079633 0" mesh_path="$(find drone)/STLs/hexagonal_prism_height_1_outer_diameter_1.stl" scale_xyz="0.024 0.024 0.58" mass="1.0" ixx="0.1" ixy="0.0" ixz="0.0" iyy="0.1" iyz="0.0" izz="0.1"/>
   <!-- Define the drone arms using the macro -->
   <xacro:property name="deg_to_rad" value="0.0174533" />   <!--60 degrees in radians-->
-  <xacro:drone_arm arm_link_name="arm_link_0" rotor_joint_name="rotor_joint_0" propeller_link_name="prop_link_0" parent_link="core_link" dis_from_center="17.5" length="56" angle="${0 * deg_to_rad}"/>
-  <xacro:drone_arm arm_link_name="arm_link_1" rotor_joint_name="rotor_joint_1" propeller_link_name="prop_link_1" parent_link="core_link" dis_from_center="17.5" length="56" angle="${180 * deg_to_rad}"/>
-  <xacro:drone_arm arm_link_name="arm_link_2" rotor_joint_name="rotor_joint_2" propeller_link_name="prop_link_2" parent_link="core_link" dis_from_center="17.5" length="56" angle="${120 * deg_to_rad}"/>
-  <xacro:drone_arm arm_link_name="arm_link_3" rotor_joint_name="rotor_joint_3" propeller_link_name="prop_link_3" parent_link="core_link" dis_from_center="17.5" length="56" angle="${300 * deg_to_rad}"/>
-  <xacro:drone_arm arm_link_name="arm_link_4" rotor_joint_name="rotor_joint_4" propeller_link_name="prop_link_4" parent_link="core_link" dis_from_center="17.5" length="56" angle="${90 * deg_to_rad}"/>
-  <xacro:drone_arm arm_link_name="arm_link_5" rotor_joint_name="rotor_joint_5" propeller_link_name="prop_link_5" parent_link="core_link" dis_from_center="17.5" length="56" angle="${240 * deg_to_rad}"/>
+  <xacro:drone_arm num="0" parent_link="core_link" dis_from_center="0.175" length="0.56" diameter="0.025" arm_incline_angle="${10 * deg_to_rad}" prop_size_multiplier="2.04" cw="true" angle="${0}"/>
+  <xacro:drone_arm num="1" parent_link="core_link" dis_from_center="0.175" length="0.56" diameter="0.025" arm_incline_angle="${10 * deg_to_rad}" prop_size_multiplier="2.04" cw="false" angle="${180 * deg_to_rad}"/>
+  <xacro:drone_arm num="2" parent_link="core_link" dis_from_center="0.175" length="0.56" diameter="0.025" arm_incline_angle="${10 * deg_to_rad}" prop_size_multiplier="2.04" cw="true" angle="${120 * deg_to_rad}"/>
+  <xacro:drone_arm num="3" parent_link="core_link" dis_from_center="0.175" length="0.56" diameter="0.025" arm_incline_angle="${10 * deg_to_rad}" prop_size_multiplier="2.04" cw="false" angle="${300 * deg_to_rad}"/>
+  <xacro:drone_arm num="4" parent_link="core_link" dis_from_center="0.175" length="0.56" diameter="0.025" arm_incline_angle="${10 * deg_to_rad}" prop_size_multiplier="2.04" cw="true" angle="${60 * deg_to_rad}"/>
+  <xacro:drone_arm num="5" parent_link="core_link" dis_from_center="0.175" length="0.56" diameter="0.025" arm_incline_angle="${10 * deg_to_rad}" prop_size_multiplier="2.04" cw="false" angle="${240 * deg_to_rad}"/>
+  <gazebo>
+    <link name='imu_link'>
+      <inertial>
+        <pose>0 0 0 0 0 0</pose>
+        <mass>0.15</mass>
+        <inertia>
+          <ixx>0.00001</ixx>
+          <ixy>0</ixy>
+          <ixz>0</ixz>
+          <iyy>0.00002</iyy>
+          <iyz>0</iyz>
+          <izz>0.00002</izz>
+        </inertia>
+      </inertial>
+      <sensor name="imu_sensor" type="imu">
+        <pose>0 0 0 3.141593 0 0</pose>
+        <always_on>1</always_on>
+        <update_rate>1000.0</update_rate>
+      </sensor>
+    </link>
+    <joint name='imu_joint' type='fixed'>
+      <child>imu_link</child>
+      <parent>core_link</parent>
+      <axis>
+        <xyz>0 0 1</xyz>
+        <limit>
+          <lower>0</lower>
+          <upper>0</upper>
+          <effort>0</effort>
+          <velocity>0</velocity>
+        </limit>
+        <dynamics>
+          <damping>1.0</damping>
+        </dynamics>
+        <use_parent_model_frame>1</use_parent_model_frame>
+      </axis>
+      <physics>
+        <ode>
+          <implicit_spring_damper>1</implicit_spring_damper>
+        </ode>
+      </physics>
+    </joint>
+  </gazebo>
 </robot>
 <!--

File: xacros/ardupilot_plugin.xacro (robot description, xacro)
@@ -1,3 +1,2 @@
-  <!-- Plugin encapsulating all control channels -->
   <gazebo>
     <plugin name="arducopter_plugin" filename="libArduPilotPlugin.so">
@@ -34,2 +33,18 @@
     </control>
   </xacro:macro>
+      <plugin name="arducopter_plugin" filename="libArduPilotPlugin.so">
+      <fdm_addr>127.0.0.1</fdm_addr>
+      <fdm_port_in>9002</fdm_port_in>
+      <fdm_port_out>9003</fdm_port_out>
+      <modelXYZToAirplaneXForwardZDown>0 0 0 3.141593 0 0</modelXYZToAirplaneXForwardZDown>
+      <gazeboXYZToNED>0 0 0 3.141593 0 0</gazeboXYZToNED>
+      <imuName>copterPIX::base_link::core_link::imu_link::imu_sensor</imuName>
+      <connectionTimeoutMaxCount>5</connectionTimeoutMaxCount>
+      <!-- Control channels -->
+      <xacro:control_channel channel="0" rotor_joint="rotor_joint_0" multiplier="-838" /> <!--cw-->
+      <xacro:control_channel channel="1" rotor_joint="rotor_joint_1" multiplier="838" /> <!--ccw-->
+      <xacro:control_channel channel="2" rotor_joint="rotor_joint_2" multiplier="-838" /> <!--cw-->
+      <xacro:control_channel channel="3" rotor_joint="rotor_joint_3" multiplier="838" /> <!--ccw-->
+      <xacro:control_channel channel="4" rotor_joint="rotor_joint_4" multiplier="-838" /> <!--cw-->
+      <xacro:control_channel channel="5" rotor_joint="rotor_joint_5" multiplier="838" /> <!--ccw-->
+    </plugin>

File: xacros/macro.xacro (robot description, xacro)
@@ -1,49 +1,69 @@
 <?xml version="1.0"?>
 <robot xmlns:xacro="http://www.ros.org/wiki/xacro">
-    <xacro:macro name="drone_arm" params="arm_link_name rotor_joint_name propeller_link_name parent_link dis_from_center length diameter angle arm_incline_angle">
-        <joint name="fixed_joint" type="fixed">
+    <xacro:macro name="drone_arm" params="num parent_link dis_from_center length diameter arm_incline_angle prop_size_multiplier cw angle">
+        <xacro:property name="core_arm_joint" value="core_arm_joint_${num}" />
+        <xacro:property name="arm_link" value="arm_link_${num}" />
+        <xacro:property name="rotor_joint" value="rotor_joint_${num}" />
+        <xacro:property name="prop_link" value="prop_link_${num}" />
+        <xacro:property name="rotor_blade_0" value="rotor_${num}_blade_0" />
+        <xacro:property name="rotor_blade_1" value="rotor_${num}_blade_1" />
+        <joint name="${core_arm_joint}" type="fixed">
             <parent link="${parent_link}"/>
-            <child link="${arm_link_name}"/>
+            <child link="${arm_link}"/>
             <origin xyz="0 0 0" rpy="0 0 ${angle}"/>
         </joint>
-        <xacro:link_creator link_name="${arm_link_name}" pose_xyz="0 ${length / 2 + dis_from_center} 0" pose_rpy="${arm_incline_angle} 0 0" mesh_path="$(find drone)/STLs/hexagonal_prism_height_1_outer_diameter_1.stl" scale_xyz="${diameter} ${diameter} ${length}" mass="1.0" ixx="0.1" ixy="0.0" ixz="0.0" iyy="0.1" iyz="0.0" izz="0.1"/>
-        <joint name="${rotor_joint_name}" type="fixed">
-            <!-- Define the joint properties here -->
+        <xacro:link_creator link_name="${arm_link}" pose_xyz="0 ${cos(arm_incline_angle) * (length / 2.0) + dis_from_center} ${sin(arm_incline_angle) * (length / 2.0)}" pose_rpy="${arm_incline_angle + 1.57079632679} 0 0" mesh_path="$(find drone)/STLs/hexagonal_prism_height_1_outer_diameter_1.stl" scale_xyz="${diameter} ${diameter} ${length}" mass="1.0" ixx="0.1" ixy="0.0" ixz="0.0" iyy="0.1" iyz="0.0" izz="0.1"/>
+        <joint name="${rotor_joint}" type="continuous">
+            <parent link="${arm_link}"/>
+            <child link="${prop_link}"/>
+            <origin xyz="0 ${cos(arm_incline_angle) * length + dis_from_center} ${sin(arm_incline_angle) * length}" rpy="0 0 0"/>
+            <axis xyz="0 0 1"/>
+            <dynamics damping="0.004"/>
         </joint>
-        <link name="${propeller_link_name}">
-            <!-- Define the propeller properties here -->
-        </link>
-        <plugin name="rotor_3_blade_1" filename="libLiftDragPlugin.so"> change name later
-        <a0>0.3</a0>
-        <alpha_stall>1.4</alpha_stall>
-        <cla>4.2500</cla>
-        <cda>0.10</cda>
-        <cma>0.00</cma>
-        <cla_stall>-0.025</cla_stall>
-        <cda_stall>0.0</cda_stall>
-        <cma_stall>0.0</cma_stall>
-        <area>0.002</area>
-        <air_density>1.2041</air_density>
-        <cp>0.084 0 0</cp>
-        <forward>0 -1 0</forward>
-        <upward>0 0 1</upward>
-        <link_name>iris::rotor_3</link_name>
-        </plugin>
-        <plugin name="rotor_3_blade_2" filename="libLiftDragPlugin.so"> change name later
-        <a0>0.3</a0>
-        <alpha_stall>1.4</alpha_stall>
-        <cla>4.2500</cla>
-        <cda>0.10</cda>
-        <cma>0.00</cma>
-        <cla_stall>-0.025</cla_stall>
-        <cda_stall>0.0</cda_stall>
-        <cma_stall>0.0</cma_stall>
-        <area>0.002</area>
-        <air_density>1.2041</air_density>
-        <cp>-0.084 0 0</cp>
-        <forward>0 1 0</forward>
-        <upward>0 0 1</upward>
-        <link_name>iris::rotor_3</link_name>
-        </plugin>
+        <gazebo reference="${rotor_joint}">
+            <ode>
+                <implicit_spring_damper>1</implicit_spring_damper>
+            </ode>
+        </gazebo>
+        <xacro:if value="${cw}">
+            <xacro:link_creator link_name="${prop_link}" pose_xyz="0 0 0.03" pose_rpy="0 0 0" mesh_path="$(find drone)/STLs/iris_prop_cw.dae" scale_xyz="${prop_size_multiplier} ${prop_size_multiplier} ${prop_size_multiplier}" mass="1.0" ixx="0.1" ixy="0.0" ixz="0.0" iyy="0.1" iyz="0.0" izz="0.1"/>
+        </xacro:if>
+        <xacro:unless value="${cw}">
+            <xacro:link_creator link_name="${prop_link}" pose_xyz="0 0 0.03" pose_rpy="0 0 0" mesh_path="$(find drone)/STLs/iris_prop_ccw.dae" scale_xyz="${prop_size_multiplier} ${prop_size_multiplier} ${prop_size_multiplier}" mass="1.0" ixx="0.1" ixy="0.0" ixz="0.0" iyy="0.1" iyz="0.0" izz="0.1"/>
+        </xacro:unless>
+        <gazebo>
+            <plugin name="${rotor_blade_0}" filename="libLiftDragPlugin.so">
+                <a0>0.3</a0>
+                <alpha_stall>1.4</alpha_stall>
+                <cla>4.2500</cla>
+                <cda>0.10</cda>
+                <cma>0.00</cma>
+                <cla_stall>-0.025</cla_stall>
+                <cda_stall>0.0</cda_stall>
+                <cma_stall>0.0</cma_stall>
+                <area>0.002</area>
+                <air_density>1.2041</air_density>
+                <cp>0.084 0 0</cp>
+                <forward>0 -1 0</forward>
+                <upward>0 0 1</upward>
+                <link_name>${prop_link}</link_name>
+            </plugin>
+            <plugin name="${rotor_blade_1}" filename="libLiftDragPlugin.so">
+                <a0>0.3</a0>
+                <alpha_stall>1.4</alpha_stall>
+                <cla>4.2500</cla>
+                <cda>0.10</cda>
+                <cma>0.00</cma>
+                <cla_stall>-0.025</cla_stall>
+                <cda_stall>0.0</cda_stall>
+                <cma_stall>0.0</cma_stall>
+                <area>0.002</area>
+                <air_density>1.2041</air_density>
+                <cp>-0.084 0 0</cp>
+                <forward>0 1 0</forward>
+                <upward>0 0 1</upward>
+                <link_name>${prop_link}</link_name>
+            </plugin>
+        </gazebo>
     </xacro:macro>
     <xacro:macro name="link_creator" params="link_name pose_xyz pose_rpy mesh_path scale_xyz mass ixx ixy ixz iyy iyz izz">
@@ -69,28 +89,4 @@
             </inertial>
         </link>
-    </xacro:macro>
-    <xacro:macro name="temp" params="link_name">
-        <link name="${link_name}">
-            <visual>
-                <geometry>
-                    <box size="1 1 1"/>
-                </geometry>
-                <material name="red">
-                    <color rgba="0.8 0.1 0.1 1.0"/>
-                </material>
-            </visual>
-            <collision>
-                <geometry>
-                    <box size="1 1 1"/>
-                </geometry>
-            </collision>
-            <inertial>
-                <mass value="1.0"/>
-                <inertia ixx="0.1" ixy="0.0" ixz="0.0" iyy="0.1" iyz="0.0" izz="0.1"/>
-            </inertial>
-        </link>
-        <gazebo reference="${link_name}">
-            <material> Gazebo/Red</material>
-        </gazebo>
     </xacro:macro>
 </robot>
