Commit message: big big changesgit stage -A!

File: models/copterPIX/robot.urdf.xacro (robot description, xacro)
@@ -18,28 +18,28 @@
     <child link="leg_0_link"/>
   </joint>
-  <xacro:link_creator link_name="leg_0_link" pose_xyz="0 0.198 -0.305" pose_rpy="0.305 0 0" mesh_path="$(find drone)/STLs/hexagonal_prism_height_1_outer_diameter_1.stl" scale_xyz="0.024 0.024 0.61" mass="1.0" ixx="0.1" ixy="0.0" ixz="0.0" iyy="0.1" iyz="0.0" izz="0.1"/>
+  <xacro:link_creator link_name="leg_0_link" pose_xyz="0 0.198 -0.305" pose_rpy="0.305 0 0" mesh_path="$(find drone)/STLs/hexagonal_prism_height_1_outer_diameter_1.stl" scale_xyz="0.024 0.024 0.61" mass="0.2" ixx="0.0" ixy="0.0" ixz="0.0" iyy="0.0" iyz="0.0" izz="0.0"/>
   <joint name="leg_1_link_joint" type="fixed">
     <parent link="core_link"/>
     <child link="leg_1_link"/>
   </joint>
-  <xacro:link_creator link_name="leg_1_link" pose_xyz="0 -0.198 -0.305" pose_rpy="-0.305 0 0" mesh_path="$(find drone)/STLs/hexagonal_prism_height_1_outer_diameter_1.stl" scale_xyz="0.024 0.024 0.61" mass="1.0" ixx="0.1" ixy="0.0" ixz="0.0" iyy="0.1" iyz="0.0" izz="0.1"/>
+  <xacro:link_creator link_name="leg_1_link" pose_xyz="0 -0.198 -0.305" pose_rpy="-0.305 0 0" mesh_path="$(find drone)/STLs/hexagonal_prism_height_1_outer_diameter_1.stl" scale_xyz="0.024 0.024 0.61" mass="0.2" ixx="0.0" ixy="0.0" ixz="0.0" iyy="0.0" iyz="0.0" izz="0.0"/>
   <joint name="feet_0_link_joint" type="fixed">
     <parent link="core_link"/>
     <child link="feet_0_link"/>
   </joint>
-  <xacro:link_creator link_name="feet_0_link" pose_xyz="0 0.29 -0.6" pose_rpy="0 1.57079633 0" mesh_path="$(find drone)/STLs/hexagonal_prism_height_1_outer_diameter_1.stl" scale_xyz="0.024 0.024 0.58" mass="1.0" ixx="0.1" ixy="0.0" ixz="0.0" iyy="0.1" iyz="0.0" izz="0.1"/>
+  <xacro:link_creator link_name="feet_0_link" pose_xyz="0 0.29 -0.6" pose_rpy="0 1.57079633 0" mesh_path="$(find drone)/STLs/hexagonal_prism_height_1_outer_diameter_1.stl" scale_xyz="0.024 0.024 0.58" mass="0.2" ixx="0.0" ixy="0.0" ixz="0.0" iyy="0.0" iyz="0.0" izz="0.0"/>
   <joint name="feet_1_link_joint" type="fixed">
     <parent link="core_link"/>
     <child link="feet_1_link"/>
   </joint>
-  <xacro:link_creator link_name="feet_1_link" pose_xyz="0 -0.29 -0.6" pose_rpy="0 1.57079633 0" mesh_path="$(find drone)/STLs/hexagonal_prism_height_1_outer_diameter_1.stl" scale_xyz="0.024 0.024 0.58" mass="1.0" ixx="0.1" ixy="0.0" ixz="0.0" iyy="0.1" iyz="0.0" izz="0.1"/>
+  <xacro:link_creator link_name="feet_1_link" pose_xyz="0 -0.29 -0.6" pose_rpy="0 1.57079633 0" mesh_path="$(find drone)/STLs/hexagonal_prism_height_1_outer_diameter_1.stl" scale_xyz="0.024 0.024 0.58" mass="0.2" ixx="0.0" ixy="0.0" ixz="0.0" iyy="0.0" iyz="0.0" izz="0.0"/>
   <!-- Define the drone arms using the macro -->
   <xacro:property name="deg_to_rad" value="0.0174533" />   <!--60 degrees in radians-->
-  <xacro:drone_arm num="0" parent_link="core_link" dis_from_center="0.175" length="0.56" diameter="0.025" arm_incline_angle="${10 * deg_to_rad}" prop_size_multiplier="2.04" cw="true" angle="${0}"/>
-  <xacro:drone_arm num="1" parent_link="core_link" dis_from_center="0.175" length="0.56" diameter="0.025" arm_incline_angle="${10 * deg_to_rad}" prop_size_multiplier="2.04" cw="false" angle="${180 * deg_to_rad}"/>
-  <xacro:drone_arm num="2" parent_link="core_link" dis_from_center="0.175" length="0.56" diameter="0.025" arm_incline_angle="${10 * deg_to_rad}" prop_size_multiplier="2.04" cw="true" angle="${120 * deg_to_rad}"/>
-  <xacro:drone_arm num="3" parent_link="core_link" dis_from_center="0.175" length="0.56" diameter="0.025" arm_incline_angle="${10 * deg_to_rad}" prop_size_multiplier="2.04" cw="false" angle="${300 * deg_to_rad}"/>
-  <xacro:drone_arm num="4" parent_link="core_link" dis_from_center="0.175" length="0.56" diameter="0.025" arm_incline_angle="${10 * deg_to_rad}" prop_size_multiplier="2.04" cw="true" angle="${60 * deg_to_rad}"/>
-  <xacro:drone_arm num="5" parent_link="core_link" dis_from_center="0.175" length="0.56" diameter="0.025" arm_incline_angle="${10 * deg_to_rad}" prop_size_multiplier="2.04" cw="false" angle="${240 * deg_to_rad}"/>
+  <xacro:drone_arm num="0" parent_link="core_link" dis_from_center="0.175" length="0.56" diameter="0.025" arm_incline_angle="${4 * deg_to_rad}" prop_size_multiplier="2.04" amass="0.2" aixx="0" aixy="0" aixz="0" aiyy="0" aiyz="0" aizz="0" rmass="0.2" rixx="0.000312" rixy="0" rixz="0" riyy="0.0053345" riyz="0" rizz="0.005363328" cw="true" angle="${0}"/>
+  <xacro:drone_arm num="1" parent_link="core_link" dis_from_center="0.175" length="0.56" diameter="0.025" arm_incline_angle="${4 * deg_to_rad}" prop_size_multiplier="2.04" amass="0.2" aixx="0" aixy="0" aixz="0" aiyy="0" aiyz="0" aizz="0" rmass="0.2" rixx="0.000312" rixy="0" rixz="0" riyy="0.0053345" riyz="0" rizz="0.005363328" cw="false" angle="${180 * deg_to_rad}"/>
+  <xacro:drone_arm num="2" parent_link="core_link" dis_from_center="0.175" length="0.56" diameter="0.025" arm_incline_angle="${4 * deg_to_rad}" prop_size_multiplier="2.04" amass="0.2" aixx="0" aixy="0" aixz="0" aiyy="0" aiyz="0" aizz="0" rmass="0.2" rixx="0.000312" rixy="0" rixz="0" riyy="0.0053345" riyz="0" rizz="0.005363328" cw="true" angle="${120 * deg_to_rad}"/>
+  <xacro:drone_arm num="3" parent_link="core_link" dis_from_center="0.175" length="0.56" diameter="0.025" arm_incline_angle="${4 * deg_to_rad}" prop_size_multiplier="2.04" amass="0.2" aixx="0" aixy="0" aixz="0" aiyy="0" aiyz="0" aizz="0" rmass="0.2" rixx="0.000312" rixy="0" rixz="0" riyy="0.0053345" riyz="0" rizz="0.005363328" cw="false" angle="${300 * deg_to_rad}"/>
+  <xacro:drone_arm num="4" parent_link="core_link" dis_from_center="0.175" length="0.56" diameter="0.025" arm_incline_angle="${4 * deg_to_rad}" prop_size_multiplier="2.04" amass="0.2" aixx="0" aixy="0" aixz="0" aiyy="0" aiyz="0" aizz="0" rmass="0.2" rixx="0.000312" rixy="0" rixz="0" riyy="0.0053345" riyz="0" rizz="0.005363328" cw="true" angle="${60 * deg_to_rad}"/>
+  <xacro:drone_arm num="5" parent_link="core_link" dis_from_center="0.175" length="0.56" diameter="0.025" arm_incline_angle="${4 * deg_to_rad}" prop_size_multiplier="2.04" amass="0.2" aixx="0" aixy="0" aixz="0" aiyy="0" aiyz="0" aizz="0" rmass="0.2" rixx="0.000312" rixy="0" rixz="0" riyy="0.0053345" riyz="0" rizz="0.005363328" cw="false" angle="${240 * deg_to_rad}"/>
   <gazebo>
     <link name='imu_link'>

File: xacros/macro.xacro (robot description, xacro)
@@ -1,5 +1,5 @@
 <?xml version="1.0"?>
 <robot xmlns:xacro="http://www.ros.org/wiki/xacro">
-    <xacro:macro name="drone_arm" params="num parent_link dis_from_center length diameter arm_incline_angle prop_size_multiplier cw angle">
+    <xacro:macro name="drone_arm" params="num parent_link dis_from_center length diameter arm_incline_angle prop_size_multiplier amass aixx aixy aixz aiyy aiyz aizz rmass rixx rixy rixz riyy riyz rizz cw angle">
         <xacro:property name="core_arm_joint" value="core_arm_joint_${num}" />
         <xacro:property name="arm_link" value="arm_link_${num}" />
@@ -13,9 +13,9 @@
             <origin xyz="0 0 0" rpy="0 0 ${angle}"/>
         </joint>
-        <xacro:link_creator link_name="${arm_link}" pose_xyz="0 ${cos(arm_incline_angle) * (length / 2.0) + dis_from_center} ${sin(arm_incline_angle) * (length / 2.0)}" pose_rpy="${arm_incline_angle + 1.57079632679} 0 0" mesh_path="$(find drone)/STLs/hexagonal_prism_height_1_outer_diameter_1.stl" scale_xyz="${diameter} ${diameter} ${length}" mass="1.0" ixx="0.1" ixy="0.0" ixz="0.0" iyy="0.1" iyz="0.0" izz="0.1"/>
+        <xacro:link_creator link_name="${arm_link}" pose_xyz="0 ${cos(arm_incline_angle) * (length / 2.0) + dis_from_center} ${sin(arm_incline_angle) * (length / 2.0)}" pose_rpy="${arm_incline_angle + 1.57079632679} 0 0" mesh_path="$(find drone)/STLs/hexagonal_prism_height_1_outer_diameter_1.stl" scale_xyz="${diameter} ${diameter} ${length}" mass="${amass}" ixx="${aixx}" ixy="${aixy}" ixz="${aixz}" iyy="${aiyy}" iyz="${aiyz}" izz="${aizz}"/>
         <joint name="${rotor_joint}" type="continuous">
             <parent link="${arm_link}"/>
             <child link="${prop_link}"/>
-            <origin xyz="0 ${cos(arm_incline_angle) * length + dis_from_center} ${sin(arm_incline_angle) * length}" rpy="0 0 0"/>
+            <origin xyz="0 ${cos(arm_incline_angle) * length + dis_from_center} ${sin(arm_incline_angle) * length}" rpy="${arm_incline_angle} 0 0"/>
             <axis xyz="0 0 1"/>
             <dynamics damping="0.004"/>
@@ -27,8 +27,8 @@
         </gazebo>
         <xacro:if value="${cw}">
-            <xacro:link_creator link_name="${prop_link}" pose_xyz="0 0 0.03" pose_rpy="0 0 0" mesh_path="$(find drone)/STLs/iris_prop_cw.dae" scale_xyz="${prop_size_multiplier} ${prop_size_multiplier} ${prop_size_multiplier}" mass="1.0" ixx="0.1" ixy="0.0" ixz="0.0" iyy="0.1" iyz="0.0" izz="0.1"/>
+            <xacro:link_creator link_name="${prop_link}" pose_xyz="0 0 0.03" pose_rpy="0 0 0" mesh_path="$(find drone)/STLs/iris_prop_cw.dae" scale_xyz="${prop_size_multiplier} ${prop_size_multiplier} ${prop_size_multiplier}" mass="${rmass}" ixx="${rixx}" ixy="${rixy}" ixz="${rixz}" iyy="${riyy}" iyz="${riyz}" izz="${rizz}"/>
         </xacro:if>
         <xacro:unless value="${cw}">
-            <xacro:link_creator link_name="${prop_link}" pose_xyz="0 0 0.03" pose_rpy="0 0 0" mesh_path="$(find drone)/STLs/iris_prop_ccw.dae" scale_xyz="${prop_size_multiplier} ${prop_size_multiplier} ${prop_size_multiplier}" mass="1.0" ixx="0.1" ixy="0.0" ixz="0.0" iyy="0.1" iyz="0.0" izz="0.1"/>
+            <xacro:link_creator link_name="${prop_link}" pose_xyz="0 0 0.03" pose_rpy="0 0 0" mesh_path="$(find drone)/STLs/iris_prop_ccw.dae" scale_xyz="${prop_size_multiplier} ${prop_size_multiplier} ${prop_size_multiplier}" mass="${rmass}" ixx="${rixx}" ixy="${rixy}" ixz="${rixz}" iyy="${riyy}" iyz="${riyz}" izz="${rizz}"/>
         </xacro:unless>
         <gazebo>

Commit message: README.md changed

File: models/copterPIX/robot.urdf.xacro (robot description, xacro)
@@ -13,5 +13,5 @@
     <origin xyz="0 0 0.6" rpy="0 0 0"/>
   </joint>
-  <xacro:link_creator link_name="core_link" pose_xyz="0 0 0" pose_rpy="0 0 0" mesh_path="$(find drone)/STLs/hexagonal_prism_height_1_outer_diameter_1.stl" scale_xyz="0.4 0.4 0.04" mass="1.0" ixx="0.1" ixy="0.0" ixz="0.0" iyy="0.1" iyz="0.0" izz="0.1"/>
+  <xacro:link_creator link_name="core_link" pose_xyz="0 0 0" pose_rpy="0 0 0" mesh_path="$(find drone)/STLs/hexagonal_prism_height_1_outer_diameter_1.stl" scale_xyz="0.4 0.4 0.04" mass="20.0" ixx="0.1" ixy="0.0" ixz="0.0" iyy="0.1" iyz="0.0" izz="0.1"/>
   <joint name="leg_0_link_joint" type="fixed">
     <parent link="core_link"/>
@@ -35,5 +35,5 @@
   <xacro:link_creator link_name="feet_1_link" pose_xyz="0 -0.29 -0.6" pose_rpy="0 1.57079633 0" mesh_path="$(find drone)/STLs/hexagonal_prism_height_1_outer_diameter_1.stl" scale_xyz="0.024 0.024 0.58" mass="0.2" ixx="0.0" ixy="0.0" ixz="0.0" iyy="0.0" iyz="0.0" izz="0.0"/>
   <!-- Define the drone arms using the macro -->
-  <xacro:property name="deg_to_rad" value="0.0174533" />   <!--60 degrees in radians-->
+  <xacro:property name="deg_to_rad" value="0.0174533" />
   <xacro:drone_arm num="0" parent_link="core_link" dis_from_center="0.175" length="0.56" diameter="0.025" arm_incline_angle="${4 * deg_to_rad}" prop_size_multiplier="2.04" amass="0.2" aixx="0" aixy="0" aixz="0" aiyy="0" aiyz="0" aizz="0" rmass="0.2" rixx="0.000312" rixy="0" rixz="0" riyy="0.0053345" riyz="0" rizz="0.005363328" cw="true" angle="${0}"/>
   <xacro:drone_arm num="1" parent_link="core_link" dis_from_center="0.175" length="0.56" diameter="0.025" arm_incline_angle="${4 * deg_to_rad}" prop_size_multiplier="2.04" amass="0.2" aixx="0" aixy="0" aixz="0" aiyy="0" aiyz="0" aizz="0" rmass="0.2" rixx="0.000312" rixy="0" rixz="0" riyy="0.0053345" riyz="0" rizz="0.005363328" cw="false" angle="${180 * deg_to_rad}"/>
