Commit message: made the macros better!

File: models/copterPIX/robot.urdf.xacro (robot description, xacro)
@@ -6,4 +6,7 @@
   <xacro:property name="prop_cw_mesh" value="$(find drone)/STLs/iris_prop_cw.dae"/>
   <xacro:property name="prop_ccw_mesh" value="$(find drone)/STLs/iris_prop_ccw.dae"/>
+    <!-- <xacro:property name="hex_mesh" value="hexagonal_prism_height_1_outer_diameter_1.stl"/>
+  <xacro:property name="prop_cw_mesh" value="iris_prop_cw.dae"/>
+  <xacro:property name="prop_ccw_mesh" value="iris_prop_ccw.dae"/> -->
   <!-- Base link -->
   <link name="base_link">
@@ -24,5 +27,5 @@
   <xacro:property name="iyz" value="${50504029566.32 / g_mms_to_kg_ms}"/>
   <xacro:property name="izz" value="${574188826210.05 / g_mms_to_kg_ms}"/>
-  <xacro:link_creator_center_mass link_name="core_link" pose_xyz="0 0 0" pose_rpy="0 0 0" mesh_path="${hex_mesh}" scale_xyz="0.4 0.4 0.04" mass_xyz="0 0 -0.18" mass_rpy="0 0 0" mass="${mass}" ixx="${ixx}" ixy="${ixy}" ixz="${ixz}" iyy="${iyy}" iyz="${iyz}" izz="${izz}"/>
+  <xacro:link_creator_i link_name="core_link" pose_xyz="0 0 0" pose_rpy="0 0 0" mesh_path="${hex_mesh}" scale_xyz="0.4 0.4 0.04" center_mass_xyz="0 0 -0.18" mass="${mass}" ixx="${ixx}" ixy="${ixy}" ixz="${ixz}" iyy="${iyy}" iyz="${iyz}" izz="${izz}"/>
   <joint name="leg_0_link_joint" type="fixed">
     <parent link="core_link"/>
@@ -30,5 +33,5 @@
   </joint>
   <!-- <xacro:link_creator link_name="leg_0_link" pose_xyz="0 0.198 -0.305" pose_rpy="0.305 0 0" mesh_path="$(find drone)/STLs/hexagonal_prism_height_1_outer_diameter_1.stl" scale_xyz="0.024 0.024 0.61" mass="0.0" ixx="0.0" ixy="0.0" ixz="0.0" iyy="0.0" iyz="0.0" izz="0.0"/> -->
-  <xacro:link_creator_no_mass link_name="leg_0_link" pose_xyz="0 0.198 -0.305" pose_rpy="0.305 0 0" mesh_path="${hex_mesh}" scale_xyz="0.024 0.024 0.61"/>
+  <xacro:link_creator link_name="leg_0_link" pose_xyz="0 0.198 -0.305" pose_rpy="0.305 0 0" mesh_path="${hex_mesh}" scale_xyz="0.024 0.024 0.61"/>
   <joint name="leg_1_link_joint" type="fixed">
     <parent link="core_link"/>
@@ -36,5 +39,5 @@
   </joint>
   <!-- <xacro:link_creator link_name="leg_1_link" pose_xyz="0 -0.198 -0.305" pose_rpy="-0.305 0 0" mesh_path="$(find drone)/STLs/hexagonal_prism_height_1_outer_diameter_1.stl" scale_xyz="0.024 0.024 0.61" mass="0.0" ixx="0.0" ixy="0.0" ixz="0.0" iyy="0.0" iyz="0.0" izz="0.0"/> -->
-  <xacro:link_creator_no_mass link_name="leg_1_link" pose_xyz="0 -0.198 -0.305" pose_rpy="-0.305 0 0" mesh_path="${hex_mesh}" scale_xyz="0.024 0.024 0.61"/>
+  <xacro:link_creator link_name="leg_1_link" pose_xyz="0 -0.198 -0.305" pose_rpy="-0.305 0 0" mesh_path="${hex_mesh}" scale_xyz="0.024 0.024 0.61"/>
   <joint name="feet_0_link_joint" type="fixed">
     <parent link="core_link"/>
@@ -42,5 +45,5 @@
   </joint>
   <!-- <xacro:link_creator link_name="feet_0_link" pose_xyz="0 0.29 -0.6" pose_rpy="0 1.57079633 0" mesh_path="$(find drone)/STLs/hexagonal_prism_height_1_outer_diameter_1.stl" scale_xyz="0.024 0.024 0.58" mass="0.0" ixx="0.0" ixy="0.0" ixz="0.0" iyy="0.0" iyz="0.0" izz="0.0"/> -->
-  <xacro:link_creator_no_mass link_name="feet_0_link" pose_xyz="0 0.29 -0.6" pose_rpy="0 1.57079633 0" mesh_path="${hex_mesh}" scale_xyz="0.024 0.024 0.58"/>
+  <xacro:link_creator link_name="feet_0_link" pose_xyz="0 0.29 -0.6" pose_rpy="0 1.57079633 0" mesh_path="${hex_mesh}" scale_xyz="0.024 0.024 0.58"/>
   <joint name="feet_1_link_joint" type="fixed">
     <parent link="core_link"/>
@@ -48,5 +51,5 @@
   </joint>
   <!-- <xacro:link_creator link_name="feet_1_link" pose_xyz="0 -0.29 -0.6" pose_rpy="0 1.57079633 0" mesh_path="$(find drone)/STLs/hexagonal_prism_height_1_outer_diameter_1.stl" scale_xyz="0.024 0.024 0.58" mass="0.0" ixx="0.0" ixy="0.0" ixz="0.0" iyy="0.0" iyz="0.0" izz="0.0"/> -->
-  <xacro:link_creator_no_mass link_name="feet_1_link" pose_xyz="0 -0.29 -0.6" pose_rpy="0 1.57079633 0" mesh_path="${hex_mesh}" scale_xyz="0.024 0.024 0.58"/>
+  <xacro:link_creator link_name="feet_1_link" pose_xyz="0 -0.29 -0.6" pose_rpy="0 1.57079633 0" mesh_path="${hex_mesh}" scale_xyz="0.024 0.024 0.58"/>
   <!-- Define the drone arms using the macro -->
   <xacro:property name="deg_to_rad" value="0.0174533" />

File: models/simple_box/robot.urdf.xacro (robot description, xacro)
@@ -1,82 +1,36 @@
 <?xml version="1.0"?>
 <robot name="simple_box" xmlns:xacro="http://www.ros.org/wiki/xacro">
-  <!-- Base link -->
-  <link name="base_link">
-  </link>
-  <link name="base_linkaa">
-    <visual>
-      <geometry>
-        <box size="1 1 1"/>
-      </geometry>
-      <material name="red">
-        <color rgba="0.8 0.1 0.1 1.0"/>
-      </material>
-      <origin xyz="30 0 0" rpy="0 0 0"/>
-    </visual>
-    <collision>
-      <geometry>
-        <box size="1 1 1"/>
-      </geometry>
-    </collision>
-    <inertial>
-      <mass value="1.0"/>
-      <inertia ixx="0.1" ixy="0.0" ixz="0.0" iyy="0.1" iyz="0.0" izz="0.1"/>
-    </inertial>
-  </link>
-  <joint name="fixed_joint" type="fixed">
-    <parent link="base_link"/>
-    <child link="base_linkaa"/>
-  </joint>
-  <!-- <link name="base_linkaaa"> -->
-    <!-- <pose>30 0 0 0 0 0</pose> -->
-    <!-- <origin xyz="30 0 0 0" rpy="0 0 0 0"/> -->
-    <!-- You can leave this link empty if you don't need a specific geometry or inertial properties for the base -->
-<!--
-     <visual>
-      <geometry>
-        <box size="1 1 1"/>
-      </geometry>
-      <material name="red">
-        <color rgba="0.8 0.1 0.1 1.0"/>
-      </material>
-    </visual>
-    <collision>
-      <geometry>
-        <box size="1 1 1"/>
-      </geometry>
-    </collision>
-    <inertial>
-      <mass value="1.0"/>
-      <inertia ixx="0.1" ixy="0.0" ixz="0.0" iyy="0.1" iyz="0.0" izz="0.1"/>
-    </inertial>
-  </link> -->
-  <!-- Box link -->
-  <!-- <link name="box_link">
-    <visual>
-      <geometry>
-        <box size="1 1 1"/>
-      </geometry>
-      <material name="red">
-        <color rgba="0.8 0.1 0.1 1.0"/>
-      </material>
-    </visual>
-    <collision>
-      <geometry>
-        <box size="1 1 1"/>
-      </geometry>
-    </collision>
-    <inertial>
-      <mass value="1.0"/>
-      <inertia ixx="0.1" ixy="0.0" ixz="0.0" iyy="0.1" iyz="0.0" izz="0.1"/>
-    </inertial>
-  </link> -->
-  <!-- Joint (fixed) -->
-  <!-- <joint name="fixed_joint" type="fixed">
-    <parent link="base_link"/>
-    <child link="box_link"/>
-    <origin xyz="0 0 0" rpy="0 0 0"/>
-  </joint> -->
-  <!-- <gazebo reference="base_linka">
-    <material> Gazebo/Red</material>
-  </gazebo> -->
+  <!-- Define the macro with an optional block parameter -->
+  <xacro:macro name="my_link" params="name length:=1.0 radius:=0.5 **extra">
+    <!-- Define a default extra block -->
+    <xacro:property name="default_extra">
+      <origin xyz="0 0 0" rpy="0 0 0"/>
+    </xacro:property>
+    <!-- Use the parameters in the macro -->
+    <link name="${name}">
+      <visual>
+        <geometry>
+          <cylinder length="${length}" radius="${radius}" />
+        </geometry>
+      </visual>
+      <collision>
+        <geometry>
+          <cylinder length="${length}" radius="${radius}" />
+        </geometry>
+      </collision>
+      <inertial>
+        <mass value="1.0"/>
+        <origin xyz="0 0 0" rpy="0 0 0"/>
+        <inertia ixx="1.0" ixy="0.0" ixz="0.0" iyy="1.0" iyz="0.0" izz="1.0"/>
+      </inertial>
+      <!-- Insert the extra block if provided, else use the default -->
+      <xacro:insert_block name="extra" />
+    </link>
+  </xacro:macro>
+  <!-- Example usage without extra settings -->
+  <xacro:my_link name="link3">
+    <extra>
+      <!-- This block is intentionally left empty to avoid errors -->
+    </extra>
+  </xacro:my_link>
 </robot>

File: xacros/macro.xacro (robot description, xacro)
@@ -1,5 +1,4 @@
 <?xml version="1.0"?>
 <robot xmlns:xacro="http://www.ros.org/wiki/xacro">
-    <!-- <xacro:macro name="drone_arm" params="num parent_link dis_from_center length diameter arm_incline_angle arm_mesh prop_mesh prop_size_multiplier amass aixx aixy aixz aiyy aiyz aizz rmass rixx rixy rixz riyy riyz rizz angle">  -->
     <xacro:macro name="drone_arm" params="num parent_link dis_from_center length diameter arm_incline_angle arm_mesh prop_mesh prop_size_multiplier rmass rixx rixy rixz riyy riyz rizz angle">
         <xacro:property name="core_arm_joint" value="core_arm_joint_${num}" />
@@ -14,7 +13,5 @@
             <origin xyz="0 0 0" rpy="0 0 ${angle}"/>
         </joint>
-        <!-- <xacro:link_creator link_name="${arm_link}" pose_xyz="0 ${cos(arm_incline_angle) * (length / 2.0) + dis_from_center} ${sin(arm_incline_angle) * (length / 2.0)}" pose_rpy="${arm_incline_angle + 1.57079632679} 0 0" mesh_path="${arm_mesh}" scale_xyz="${diameter} ${diameter} ${length}" mass="${amass}" ixx="${aixx}" ixy="${aixy}" ixz="${aixz}" iyy="${aiyy}" iyz="${aiyz}" izz="${aizz}"/> -->
-        <xacro:link_creator link_name="${arm_link}" pose_xyz="0 ${cos(arm_incline_angle) * (length / 2.0) + dis_from_center} ${sin(arm_incline_angle) * (length / 2.0)}" pose_rpy="${arm_incline_angle + 1.57079632679} 0 0" mesh_path="${arm_mesh}" scale_xyz="${diameter} ${diameter} ${length}" mass="0.2" ixx="0" ixy="0" ixz="0" iyy="0" iyz="0" izz="0"/>
-        <!-- <xacro:link_creator_no_mass link_name="${arm_link}" pose_xyz="0 ${cos(arm_incline_angle) * (length / 2.0) + dis_from_center} ${sin(arm_incline_angle) * (length / 2.0)}" pose_rpy="${arm_incline_angle + 1.57079632679} 0 0" mesh_path="${arm_mesh}" scale_xyz="${diameter} ${diameter} ${length}"/> -->
+        <xacro:link_creator_i link_name="${arm_link}" pose_xyz="0 ${cos(arm_incline_angle) * (length / 2.0) + dis_from_center} ${sin(arm_incline_angle) * (length / 2.0)}" pose_rpy="${arm_incline_angle + 1.57079632679} 0 0" mesh_path="${arm_mesh}" scale_xyz="${diameter} ${diameter} ${length}" mass="0.2" ixx="0" ixy="0" ixz="0" iyy="0" iyz="0" izz="0"/>
         <joint name="${rotor_joint}" type="continuous">
             <parent link="${arm_link}"/>
@@ -25,9 +22,11 @@
         </joint>
         <gazebo reference="${rotor_joint}">
-            <ode>
-                <implicit_spring_damper>1</implicit_spring_damper>
-            </ode>
+            <physics>
+                <ode>
+                    <implicit_spring_damper>1</implicit_spring_damper>
+                </ode>
+            </physics>
         </gazebo>
-        <xacro:link_creator link_name="${prop_link}" pose_xyz="0 0 0.03" pose_rpy="0 0 0" mesh_path="${prop_mesh}" scale_xyz="${prop_size_multiplier} ${prop_size_multiplier} ${prop_size_multiplier}" mass="${rmass}" ixx="${rixx}" ixy="${rixy}" ixz="${rixz}" iyy="${riyy}" iyz="${riyz}" izz="${rizz}"/>
+        <xacro:prop_link_creator link_name="${prop_link}" pose_xyz="0 0 0.03" pose_rpy="0 0 0" mesh_path="${prop_mesh}" scale_xyz="${prop_size_multiplier} ${prop_size_multiplier} ${prop_size_multiplier}" mass="${rmass}" ixx="${rixx}" ixy="${rixy}" ixz="${rixz}" iyy="${riyy}" iyz="${riyz}" izz="${rizz}"/>
         <gazebo>
             <plugin name="${rotor_blade_0}" filename="libLiftDragPlugin.so">
@@ -65,5 +64,5 @@
         </gazebo>
     </xacro:macro>
-    <xacro:macro name="link_creator" params="link_name pose_xyz pose_rpy mesh_path scale_xyz mass ixx ixy ixz iyy iyz izz">
+    <xacro:macro name="link_creator_foundation" params="link_name pose_xyz pose_rpy mesh_path scale_xyz **extra_collision **seperate_collider **extra_visual **extra_settings">
         <link name="${link_name}">
             <visual>
@@ -71,63 +70,76 @@
                     <mesh filename="${mesh_path}" scale="${scale_xyz}"/>
                 </geometry>
-                <material name="red">
-                    <color rgba="0.8 0.1 0.1 1.0"/>
-                </material>
                 <origin xyz="${pose_xyz}" rpy="${pose_rpy}"/>
+                <xacro:insert_block name="extra_visual"/>
             </visual>
             <collision>
                 <geometry>
-                    <mesh filename="${mesh_path}" scale="${scale_xyz}"/>
+                    <!-- <xacro:unless value="${seperate_collider}">
+                        <mesh filename="${mesh_path}" scale="${scale_xyz}"/>
+                    </xacro:unless> -->
+                    <xacro:insert_block name="seperate_collider"/>
                 </geometry>
                 <origin xyz="${pose_xyz}" rpy="${pose_rpy}"/>
+                <xacro:insert_block name="extra_collision"/>
             </collision>
-            <inertial>
-                <mass value="${mass}"/>
-                <inertia ixx="${ixx}" ixy="${ixy}" ixz="${ixz}" iyy="${iyy}" iyz="${iyz}" izz="${izz}"/>
-            </inertial>
+            <xacro:insert_block name="extra_settings"/>
         </link>
     </xacro:macro>
-    <xacro:macro name="link_creator_center_mass" params="link_name pose_xyz pose_rpy mesh_path scale_xyz mass_xyz mass_rpy mass ixx ixy ixz iyy iyz izz">
-        <link name="${link_name}">
-            <visual>
-                <geometry>
-                    <mesh filename="${mesh_path}" scale="${scale_xyz}"/>
-                </geometry>
-                <material name="red">
-                    <color rgba="0.8 0.1 0.1 1.0"/>
-                </material>
-                <origin xyz="${pose_xyz}" rpy="${pose_rpy}"/>
-            </visual>
-            <collision>
-                <geometry>
-                    <mesh filename="${mesh_path}" scale="${scale_xyz}"/>
-                </geometry>
-                <origin xyz="${pose_xyz}" rpy="${pose_rpy}"/>
-            </collision>
-            <inertial>
-                <mass value="${mass}"/>
-                <inertia ixx="${ixx}" ixy="${ixy}" ixz="${ixz}" iyy="${iyy}" iyz="${iyz}" izz="${izz}"/>
-                <origin xyz="${mass_xyz}" rpy="${mass_rpy}"/>
-            </inertial>
-        </link>
+    <xacro:macro name="link_creator" params="link_name pose_xyz pose_rpy mesh_path scale_xyz">
+        <xacro:link_creator_foundation link_name="${link_name}" pose_xyz="${pose_xyz}" pose_rpy="${pose_rpy}" mesh_path="${mesh_path}" scale_xyz="${scale_xyz}">
+            <extra_collision/>
+            <seperate_collider><mesh filename="${mesh_path}" scale="${scale_xyz}"/></seperate_collider>
+            <extra_visual/>
+            <extra_settings/>
+        </xacro:link_creator_foundation>
     </xacro:macro>
-    <xacro:macro name="link_creator_no_mass" params="link_name pose_xyz pose_rpy mesh_path scale_xyz">
-        <link name="${link_name}">
-            <visual>
-                <geometry>
-                    <mesh filename="${mesh_path}" scale="${scale_xyz}"/>
-                </geometry>
-                <material name="red">
-                    <color rgba="0.8 0.1 0.1 1.0"/>
-                </material>
-                <origin xyz="${pose_xyz}" rpy="${pose_rpy}"/>
-            </visual>
-            <collision>
-                <geometry>
-                    <mesh filename="${mesh_path}" scale="${scale_xyz}"/>
-                </geometry>
-                <origin xyz="${pose_xyz}" rpy="${pose_rpy}"/>
-            </collision>
-        </link>
+    <xacro:macro name="link_creator_i_foundation" params="link_name pose_xyz pose_rpy mesh_path scale_xyz center_mass_xyz:='0 0 0' mass ixx ixy ixz iyy iyz izz **extra_collision **seperate_collider **extra_visual **extra_settings">
+        <xacro:link_creator_foundation link_name="${link_name}" pose_xyz="${pose_xyz}" pose_rpy="${pose_rpy}" mesh_path="${mesh_path}" scale_xyz="${scale_xyz}">
+            <extra_collision><xacro:insert_block name="extra_collision"/></extra_collision>
+            <seperate_collider><xacro:insert_block name="seperate_collider"/></seperate_collider>
+            <extra_visual><xacro:insert_block name="extra_visual"/></extra_visual>
+            <extra_settings>
+                <inertial>
+                    <origin xyz="${center_mass_xyz}" rpy="0 0 0"/>
+                    <mass value="${mass}"/>
+                    <inertia ixx="${ixx}" ixy="${ixy}" ixz="${ixz}" iyy="${iyy}" iyz="${iyz}" izz="${izz}"/>
+                </inertial>
+                <xacro:insert_block name="extra_settings"/>
+            </extra_settings>
+        </xacro:link_creator_foundation>
+    </xacro:macro>
+    <xacro:macro name="link_creator_i" params="link_name pose_xyz pose_rpy mesh_path scale_xyz center_mass_xyz:='0 0 0' mass ixx ixy ixz iyy iyz izz">
+        <xacro:link_creator_i_foundation link_name="${link_name}" pose_xyz="${pose_xyz}" pose_rpy="${pose_rpy}" mesh_path="${mesh_path}" scale_xyz="${scale_xyz}" center_mass_xyz="${center_mass_xyz}" mass="${mass}" ixx="${ixx}" ixy="${ixy}" ixz="${ixz}" iyy="${iyy}" iyz="${iyz}" izz="${izz}">
+            <extra_collision/>
+            <seperate_collider><mesh filename="${mesh_path}" scale="${scale_xyz}"/></seperate_collider>
+            <extra_visual/>
+            <extra_settings/>
+        </xacro:link_creator_i_foundation>
+    </xacro:macro>
+    <xacro:macro name="prop_link_creator" params="link_name pose_xyz pose_rpy mesh_path scale_xyz cyliner_r:='0.25' cylinder_l='0.01' mass ixx ixy ixz iyy iyz izz">
+        <xacro:link_creator_i_foundation link_name="${link_name}" pose_xyz="${pose_xyz}" pose_rpy="${pose_rpy}" mesh_path="${mesh_path}" scale_xyz="${scale_xyz}" mass="${mass}"  ixx="${ixx}" ixy="${ixy}" ixz="${ixz}" iyy="${iyy}" iyz="${iyz}" izz="${izz}">
+            <extra_collision>
+                <surface>
+                    <contact>
+                        <ode/>
+                    </contact>
+                    <friction>
+                        <ode/>
+                    </friction>
+                </surface>
+            </extra_collision>
+            <seperate_collider>
+                <cylinder radius="${cyliner_r}" length="${cylinder_l}"/>
+            </seperate_collider>
+            <extra_visual/>
+            <extra_settings>
+                <velocity_decay/>
+                <gazebo reference="${link_name}">
+                    <material>Gazebo/Red</material>
+                    <gravity>1</gravity>
+                    <self_collide>0</self_collide>
+                </gazebo>
+            </extra_settings>
+        </xacro:link_creator_i_foundation>
     </xacro:macro>
 </robot>
