Commit message: fixed imu instability...but still doesn't fly cuz of some lift issues

File: models/copterPIX/robot.urdf.xacro (robot description, xacro)
@@ -6,7 +6,4 @@
   <xacro:property name="prop_cw_mesh" value="$(find drone)/STLs/iris_prop_cw.dae"/>
   <xacro:property name="prop_ccw_mesh" value="$(find drone)/STLs/iris_prop_ccw.dae"/>
-    <!-- <xacro:property name="hex_mesh" value="hexagonal_prism_height_1_outer_diameter_1.stl"/>
-  <xacro:property name="prop_cw_mesh" value="iris_prop_cw.dae"/>
-  <xacro:property name="prop_ccw_mesh" value="iris_prop_ccw.dae"/> -->
   <!-- Base link -->
   <link name="base_link">
@@ -20,5 +17,5 @@
   </joint>
   <xacro:property name="g_mms_to_kg_ms" value="1000000000" />
-  <xacro:property name="mass" value="26.0" />
+  <!-- <xacro:property name="mass" value="26.0" />
   <xacro:property name="ixx" value="${373162267137.9 / g_mms_to_kg_ms}"/>
   <xacro:property name="ixy" value="${19971359238.18 / g_mms_to_kg_ms}"/>
@@ -26,5 +23,12 @@
   <xacro:property name="iyy" value="${595713038514.03 / g_mms_to_kg_ms}"/>
   <xacro:property name="iyz" value="${50504029566.32 / g_mms_to_kg_ms}"/>
-  <xacro:property name="izz" value="${574188826210.05 / g_mms_to_kg_ms}"/>
+  <xacro:property name="izz" value="${574188826210.05 / g_mms_to_kg_ms}"/> -->
+  <xacro:property name="mass" value="20.0" />
+  <xacro:property name="ixx" value="${0.1}"/>
+  <xacro:property name="ixy" value="${0}"/>
+  <xacro:property name="ixz" value="${0}"/>
+  <xacro:property name="iyy" value="${0.1}"/>
+  <xacro:property name="iyz" value="${0}"/>
+  <xacro:property name="izz" value="${0.1}"/>
   <xacro:link_creator_i link_name="core_link" pose_xyz="0 0 0" pose_rpy="0 0 0" mesh_path="${hex_mesh}" scale_xyz="0.4 0.4 0.04" center_mass_xyz="0 0 -0.18" mass="${mass}" ixx="${ixx}" ixy="${ixy}" ixz="${ixz}" iyy="${iyy}" iyz="${iyz}" izz="${izz}"/>
   <joint name="leg_0_link_joint" type="fixed">
@@ -32,24 +36,24 @@
     <child link="leg_0_link"/>
   </joint>
-  <!-- <xacro:link_creator link_name="leg_0_link" pose_xyz="0 0.198 -0.305" pose_rpy="0.305 0 0" mesh_path="$(find drone)/STLs/hexagonal_prism_height_1_outer_diameter_1.stl" scale_xyz="0.024 0.024 0.61" mass="0.0" ixx="0.0" ixy="0.0" ixz="0.0" iyy="0.0" iyz="0.0" izz="0.0"/> -->
-  <xacro:link_creator link_name="leg_0_link" pose_xyz="0 0.198 -0.305" pose_rpy="0.305 0 0" mesh_path="${hex_mesh}" scale_xyz="0.024 0.024 0.61"/>
+  <xacro:link_creator_i link_name="leg_0_link" pose_xyz="0 0.198 -0.305" pose_rpy="0.305 0 0" mesh_path="$(find drone)/STLs/hexagonal_prism_height_1_outer_diameter_1.stl" scale_xyz="0.024 0.024 0.61" mass="0.2" ixx="0.0" ixy="0.0" ixz="0.0" iyy="0.0" iyz="0.0" izz="0.0"/>
+  <!-- <xacro:link_creator link_name="leg_0_link" pose_xyz="0 0.198 -0.305" pose_rpy="0.305 0 0" mesh_path="${hex_mesh}" scale_xyz="0.024 0.024 0.61"/> -->
   <joint name="leg_1_link_joint" type="fixed">
     <parent link="core_link"/>
     <child link="leg_1_link"/>
   </joint>
-  <!-- <xacro:link_creator link_name="leg_1_link" pose_xyz="0 -0.198 -0.305" pose_rpy="-0.305 0 0" mesh_path="$(find drone)/STLs/hexagonal_prism_height_1_outer_diameter_1.stl" scale_xyz="0.024 0.024 0.61" mass="0.0" ixx="0.0" ixy="0.0" ixz="0.0" iyy="0.0" iyz="0.0" izz="0.0"/> -->
-  <xacro:link_creator link_name="leg_1_link" pose_xyz="0 -0.198 -0.305" pose_rpy="-0.305 0 0" mesh_path="${hex_mesh}" scale_xyz="0.024 0.024 0.61"/>
+  <xacro:link_creator_i link_name="leg_1_link" pose_xyz="0 -0.198 -0.305" pose_rpy="-0.305 0 0" mesh_path="$(find drone)/STLs/hexagonal_prism_height_1_outer_diameter_1.stl" scale_xyz="0.024 0.024 0.61" mass="0.2" ixx="0.0" ixy="0.0" ixz="0.0" iyy="0.0" iyz="0.0" izz="0.0"/>
+  <!-- <xacro:link_creator link_name="leg_1_link" pose_xyz="0 -0.198 -0.305" pose_rpy="-0.305 0 0" mesh_path="${hex_mesh}" scale_xyz="0.024 0.024 0.61"/> -->
   <joint name="feet_0_link_joint" type="fixed">
     <parent link="core_link"/>
     <child link="feet_0_link"/>
   </joint>
-  <!-- <xacro:link_creator link_name="feet_0_link" pose_xyz="0 0.29 -0.6" pose_rpy="0 1.57079633 0" mesh_path="$(find drone)/STLs/hexagonal_prism_height_1_outer_diameter_1.stl" scale_xyz="0.024 0.024 0.58" mass="0.0" ixx="0.0" ixy="0.0" ixz="0.0" iyy="0.0" iyz="0.0" izz="0.0"/> -->
-  <xacro:link_creator link_name="feet_0_link" pose_xyz="0 0.29 -0.6" pose_rpy="0 1.57079633 0" mesh_path="${hex_mesh}" scale_xyz="0.024 0.024 0.58"/>
+  <xacro:link_creator_i link_name="feet_0_link" pose_xyz="0 0.29 -0.6" pose_rpy="0 1.57079633 0" mesh_path="$(find drone)/STLs/hexagonal_prism_height_1_outer_diameter_1.stl" scale_xyz="0.024 0.024 0.58" mass="0.2" ixx="0.0" ixy="0.0" ixz="0.0" iyy="0.0" iyz="0.0" izz="0.0"/>
+  <!-- <xacro:link_creator link_name="feet_0_link" pose_xyz="0 0.29 -0.6" pose_rpy="0 1.57079633 0" mesh_path="${hex_mesh}" scale_xyz="0.024 0.024 0.58"/> -->
   <joint name="feet_1_link_joint" type="fixed">
     <parent link="core_link"/>
     <child link="feet_1_link"/>
   </joint>
-  <!-- <xacro:link_creator link_name="feet_1_link" pose_xyz="0 -0.29 -0.6" pose_rpy="0 1.57079633 0" mesh_path="$(find drone)/STLs/hexagonal_prism_height_1_outer_diameter_1.stl" scale_xyz="0.024 0.024 0.58" mass="0.0" ixx="0.0" ixy="0.0" ixz="0.0" iyy="0.0" iyz="0.0" izz="0.0"/> -->
-  <xacro:link_creator link_name="feet_1_link" pose_xyz="0 -0.29 -0.6" pose_rpy="0 1.57079633 0" mesh_path="${hex_mesh}" scale_xyz="0.024 0.024 0.58"/>
+  <xacro:link_creator_i link_name="feet_1_link" pose_xyz="0 -0.29 -0.6" pose_rpy="0 1.57079633 0" mesh_path="$(find drone)/STLs/hexagonal_prism_height_1_outer_diameter_1.stl" scale_xyz="0.024 0.024 0.58" mass="0.2" ixx="0.0" ixy="0.0" ixz="0.0" iyy="0.0" iyz="0.0" izz="0.0"/>
+  <!-- <xacro:link_creator link_name="feet_1_link" pose_xyz="0 -0.29 -0.6" pose_rpy="0 1.57079633 0" mesh_path="${hex_mesh}" scale_xyz="0.024 0.024 0.58"/> -->
   <!-- Define the drone arms using the macro -->
   <xacro:property name="deg_to_rad" value="0.0174533" />

File: xacros/macro.xacro (robot description, xacro)
@@ -22,9 +22,9 @@
         </joint>
         <gazebo reference="${rotor_joint}">
-            <physics>
+            <!-- <physics> -->
                 <ode>
                     <implicit_spring_damper>1</implicit_spring_damper>
                 </ode>
-            </physics>
+            <!-- </physics> -->
         </gazebo>
         <xacro:prop_link_creator link_name="${prop_link}" pose_xyz="0 0 0.03" pose_rpy="0 0 0" mesh_path="${prop_mesh}" scale_xyz="${prop_size_multiplier} ${prop_size_multiplier} ${prop_size_multiplier}" mass="${rmass}" ixx="${rixx}" ixy="${rixy}" ixz="${rixz}" iyy="${riyy}" iyz="${riyz}" izz="${rizz}"/>

Commit message: able to takeoff but unstable

File: models/copterPIX/robot.urdf.xacro (robot description, xacro)
@@ -24,5 +24,5 @@
   <xacro:property name="iyz" value="${50504029566.32 / g_mms_to_kg_ms}"/>
   <xacro:property name="izz" value="${574188826210.05 / g_mms_to_kg_ms}"/> -->
-  <xacro:property name="mass" value="20.0" />
+  <xacro:property name="mass" value="2.5" />
   <xacro:property name="ixx" value="${0.1}"/>
   <xacro:property name="ixy" value="${0}"/>
@@ -64,10 +64,16 @@
   <xacro:drone_arm num="4" parent_link="core_link" dis_from_center="0.175" length="0.56" diameter="0.025" arm_incline_angle="${4 * deg_to_rad}" arm_mesh="${hex_mesh}" prop_mesh="${prop_ccw_mesh}" prop_size_multiplier="2.04" amass="0.2" aixx="0" aixy="0" aixz="0" aiyy="0" aiyz="0" aizz="0" rmass="0.2" rixx="0.000312" rixy="0" rixz="0" riyy="0.0053345" riyz="0" rizz="0.005363328" angle="${60 * deg_to_rad}"/>
   <xacro:drone_arm num="5" parent_link="core_link" dis_from_center="0.175" length="0.56" diameter="0.025" arm_incline_angle="${4 * deg_to_rad}" arm_mesh="${hex_mesh}" prop_mesh="${prop_cw_mesh}" prop_size_multiplier="2.04" amass="0.2" aixx="0" aixy="0" aixz="0" aiyy="0" aiyz="0" aizz="0" rmass="0.2" rixx="0.000312" rixy="0" rixz="0" riyy="0.0053345" riyz="0" rizz="0.005363328" angle="${240 * deg_to_rad}"/> -->
-  <xacro:drone_arm num="0" parent_link="core_link" dis_from_center="0.175" length="0.56" diameter="0.025" arm_incline_angle="${4 * deg_to_rad}" arm_mesh="${hex_mesh}" prop_mesh="${prop_cw_mesh}" prop_size_multiplier="2.04" rmass="0.1" rixx="0.000312" rixy="0" rixz="0" riyy="0.0053345" riyz="0" rizz="0.005363328" angle="${0 * deg_to_rad}"/>
-  <xacro:drone_arm num="1" parent_link="core_link" dis_from_center="0.175" length="0.56" diameter="0.025" arm_incline_angle="${4 * deg_to_rad}" arm_mesh="${hex_mesh}" prop_mesh="${prop_ccw_mesh}" prop_size_multiplier="2.04" rmass="0.1" rixx="0.000312" rixy="0" rixz="0" riyy="0.0053345" riyz="0" rizz="0.005363328" angle="${180 * deg_to_rad}"/>
-  <xacro:drone_arm num="2" parent_link="core_link" dis_from_center="0.175" length="0.56" diameter="0.025" arm_incline_angle="${4 * deg_to_rad}" arm_mesh="${hex_mesh}" prop_mesh="${prop_cw_mesh}" prop_size_multiplier="2.04" rmass="0.1" rixx="0.000312" rixy="0" rixz="0" riyy="0.0053345" riyz="0" rizz="0.005363328" angle="${120 * deg_to_rad}"/>
-  <xacro:drone_arm num="3" parent_link="core_link" dis_from_center="0.175" length="0.56" diameter="0.025" arm_incline_angle="${4 * deg_to_rad}" arm_mesh="${hex_mesh}" prop_mesh="${prop_ccw_mesh}" prop_size_multiplier="2.04" rmass="0.1" rixx="0.000312" rixy="0" rixz="0" riyy="0.0053345" riyz="0" rizz="0.005363328" angle="${300 * deg_to_rad}"/>
-  <xacro:drone_arm num="4" parent_link="core_link" dis_from_center="0.175" length="0.56" diameter="0.025" arm_incline_angle="${4 * deg_to_rad}" arm_mesh="${hex_mesh}" prop_mesh="${prop_ccw_mesh}" prop_size_multiplier="2.04" rmass="0.1" rixx="0.000312" rixy="0" rixz="0" riyy="0.0053345" riyz="0" rizz="0.005363328" angle="${60 * deg_to_rad}"/>
-  <xacro:drone_arm num="5" parent_link="core_link" dis_from_center="0.175" length="0.56" diameter="0.025" arm_incline_angle="${4 * deg_to_rad}" arm_mesh="${hex_mesh}" prop_mesh="${prop_cw_mesh}" prop_size_multiplier="2.04" rmass="0.1" rixx="0.000312" rixy="0" rixz="0" riyy="0.0053345" riyz="0" rizz="0.005363328" angle="${240 * deg_to_rad}"/>
+  <!-- <xacro:drone_arm num="0" parent_link="core_link" dis_from_center="0.175" length="0.56" diameter="0.025" arm_incline_angle="${4 * deg_to_rad}" arm_mesh="${hex_mesh}" prop_mesh="${prop_cw_mesh}" cw="true" prop_size_multiplier="2.04" rmass="0.2" rixx="0.000312" rixy="0" rixz="0" riyy="0.0053345" riyz="0" rizz="0.005363328" angle="${0 * deg_to_rad}"/>
+  <xacro:drone_arm num="1" parent_link="core_link" dis_from_center="0.175" length="0.56" diameter="0.025" arm_incline_angle="${4 * deg_to_rad}" arm_mesh="${hex_mesh}" prop_mesh="${prop_ccw_mesh}" cw="false" prop_size_multiplier="2.04" rmass="0.2" rixx="0.000312" rixy="0" rixz="0" riyy="0.0053345" riyz="0" rizz="0.005363328" angle="${180 * deg_to_rad}"/>
+  <xacro:drone_arm num="2" parent_link="core_link" dis_from_center="0.175" length="0.56" diameter="0.025" arm_incline_angle="${4 * deg_to_rad}" arm_mesh="${hex_mesh}" prop_mesh="${prop_cw_mesh}" cw="true" prop_size_multiplier="2.04" rmass="0.2" rixx="0.000312" rixy="0" rixz="0" riyy="0.0053345" riyz="0" rizz="0.005363328" angle="${120 * deg_to_rad}"/>
+  <xacro:drone_arm num="3" parent_link="core_link" dis_from_center="0.175" length="0.56" diameter="0.025" arm_incline_angle="${4 * deg_to_rad}" arm_mesh="${hex_mesh}" prop_mesh="${prop_ccw_mesh}" cw="false" prop_size_multiplier="2.04" rmass="0.2" rixx="0.000312" rixy="0" rixz="0" riyy="0.0053345" riyz="0" rizz="0.005363328" angle="${300 * deg_to_rad}"/>
+  <xacro:drone_arm num="4" parent_link="core_link" dis_from_center="0.175" length="0.56" diameter="0.025" arm_incline_angle="${4 * deg_to_rad}" arm_mesh="${hex_mesh}" prop_mesh="${prop_ccw_mesh}" cw="false" prop_size_multiplier="2.04" rmass="0.2" rixx="0.000312" rixy="0" rixz="0" riyy="0.0053345" riyz="0" rizz="0.005363328" angle="${60 * deg_to_rad}"/>
+  <xacro:drone_arm num="5" parent_link="core_link" dis_from_center="0.175" length="0.56" diameter="0.025" arm_incline_angle="${4 * deg_to_rad}" arm_mesh="${hex_mesh}" prop_mesh="${prop_cw_mesh}" cw="true" prop_size_multiplier="2.04" rmass="0.2" rixx="0.000312" rixy="0" rixz="0" riyy="0.0053345" riyz="0" rizz="0.005363328" angle="${240 * deg_to_rad}"/> -->
+  <xacro:drone_arm num="0" parent_link="core_link" dis_from_center="0.175" length="0.56" diameter="0.025" arm_incline_angle="${4 * deg_to_rad}" arm_mesh="${hex_mesh}" prop_mesh="${prop_cw_mesh}"  cw="true"  prop_size_multiplier="2.04" rmass="0.025" rixx="0.00000975" rixy="0" rixz="0" riyy="0.000166704" riyz="0" rizz="0.000167604" angle="${0 * deg_to_rad}"/>
+  <xacro:drone_arm num="1" parent_link="core_link" dis_from_center="0.175" length="0.56" diameter="0.025" arm_incline_angle="${4 * deg_to_rad}" arm_mesh="${hex_mesh}" prop_mesh="${prop_ccw_mesh}" cw="false" prop_size_multiplier="2.04" rmass="0.025" rixx="0.00000975" rixy="0" rixz="0" riyy="0.000166704" riyz="0" rizz="0.000167604" angle="${180 * deg_to_rad}"/>
+  <xacro:drone_arm num="2" parent_link="core_link" dis_from_center="0.175" length="0.56" diameter="0.025" arm_incline_angle="${4 * deg_to_rad}" arm_mesh="${hex_mesh}" prop_mesh="${prop_cw_mesh}"  cw="true"  prop_size_multiplier="2.04" rmass="0.025" rixx="0.00000975" rixy="0" rixz="0" riyy="0.000166704" riyz="0" rizz="0.000167604" angle="${120 * deg_to_rad}"/>
+  <xacro:drone_arm num="3" parent_link="core_link" dis_from_center="0.175" length="0.56" diameter="0.025" arm_incline_angle="${4 * deg_to_rad}" arm_mesh="${hex_mesh}" prop_mesh="${prop_ccw_mesh}" cw="false" prop_size_multiplier="2.04" rmass="0.025" rixx="0.00000975" rixy="0" rixz="0" riyy="0.000166704" riyz="0" rizz="0.000167604" angle="${300 * deg_to_rad}"/>
+  <xacro:drone_arm num="4" parent_link="core_link" dis_from_center="0.175" length="0.56" diameter="0.025" arm_incline_angle="${4 * deg_to_rad}" arm_mesh="${hex_mesh}" prop_mesh="${prop_ccw_mesh}" cw="false" prop_size_multiplier="2.04" rmass="0.025" rixx="0.00000975" rixy="0" rixz="0" riyy="0.000166704" riyz="0" rizz="0.000167604" angle="${60 * deg_to_rad}"/>
+  <xacro:drone_arm num="5" parent_link="core_link" dis_from_center="0.175" length="0.56" diameter="0.025" arm_incline_angle="${4 * deg_to_rad}" arm_mesh="${hex_mesh}" prop_mesh="${prop_cw_mesh}"  cw="true"  prop_size_multiplier="2.04" rmass="0.025" rixx="0.00000975" rixy="0" rixz="0" riyy="0.000166704" riyz="0" rizz="0.000167604" angle="${240 * deg_to_rad}"/>
   <gazebo>
     <link name='imu_link'>

File: xacros/macro.xacro (robot description, xacro)
@@ -1,5 +1,5 @@
 <?xml version="1.0"?>
 <robot xmlns:xacro="http://www.ros.org/wiki/xacro">
-    <xacro:macro name="drone_arm" params="num parent_link dis_from_center length diameter arm_incline_angle arm_mesh prop_mesh prop_size_multiplier rmass rixx rixy rixz riyy riyz rizz angle">
+    <xacro:macro name="drone_arm" params="num parent_link dis_from_center length diameter arm_incline_angle arm_mesh prop_mesh cw prop_size_multiplier amass:='0.2' aixx:='0' aixy:='0' aixz:='0' aiyy:='0' aiyz:='0' aizz:='0' rmass rixx rixy rixz riyy riyz rizz angle">
         <xacro:property name="core_arm_joint" value="core_arm_joint_${num}" />
         <xacro:property name="arm_link" value="arm_link_${num}" />
@@ -13,5 +13,5 @@
             <origin xyz="0 0 0" rpy="0 0 ${angle}"/>
         </joint>
-        <xacro:link_creator_i link_name="${arm_link}" pose_xyz="0 ${cos(arm_incline_angle) * (length / 2.0) + dis_from_center} ${sin(arm_incline_angle) * (length / 2.0)}" pose_rpy="${arm_incline_angle + 1.57079632679} 0 0" mesh_path="${arm_mesh}" scale_xyz="${diameter} ${diameter} ${length}" mass="0.2" ixx="0" ixy="0" ixz="0" iyy="0" iyz="0" izz="0"/>
+        <xacro:link_creator_i link_name="${arm_link}" pose_xyz="0 ${cos(arm_incline_angle) * (length / 2.0) + dis_from_center} ${sin(arm_incline_angle) * (length / 2.0)}" pose_rpy="${arm_incline_angle + 1.57079632679} 0 0" mesh_path="${arm_mesh}" scale_xyz="${diameter} ${diameter} ${length}" mass="${amass}" ixx="${aixx}" ixy="${aixy}" ixz="${aixz}" iyy="${aiyy}" iyz="${aiyz}" izz="${aizz}"/>
         <joint name="${rotor_joint}" type="continuous">
             <parent link="${arm_link}"/>
@@ -28,39 +28,77 @@
             <!-- </physics> -->
         </gazebo>
-        <xacro:prop_link_creator link_name="${prop_link}" pose_xyz="0 0 0.03" pose_rpy="0 0 0" mesh_path="${prop_mesh}" scale_xyz="${prop_size_multiplier} ${prop_size_multiplier} ${prop_size_multiplier}" mass="${rmass}" ixx="${rixx}" ixy="${rixy}" ixz="${rixz}" iyy="${riyy}" iyz="${riyz}" izz="${rizz}"/>
-        <gazebo>
-            <plugin name="${rotor_blade_0}" filename="libLiftDragPlugin.so">
-                <a0>0.3</a0>
-                <alpha_stall>1.4</alpha_stall>
-                <cla>4.2500</cla>
-                <cda>0.10</cda>
-                <cma>0.00</cma>
-                <cla_stall>-0.025</cla_stall>
-                <cda_stall>0.0</cda_stall>
-                <cma_stall>0.0</cma_stall>
-                <area>0.002</area>
-                <air_density>1.2041</air_density>
-                <cp>0.084 0 0</cp>
-                <forward>0 -1 0</forward>
-                <upward>0 0 1</upward>
-                <link_name>${prop_link}</link_name>
-            </plugin>
-            <plugin name="${rotor_blade_1}" filename="libLiftDragPlugin.so">
-                <a0>0.3</a0>
-                <alpha_stall>1.4</alpha_stall>
-                <cla>4.2500</cla>
-                <cda>0.10</cda>
-                <cma>0.00</cma>
-                <cla_stall>-0.025</cla_stall>
-                <cda_stall>0.0</cda_stall>
-                <cma_stall>0.0</cma_stall>
-                <area>0.002</area>
-                <air_density>1.2041</air_density>
-                <cp>-0.084 0 0</cp>
-                <forward>0 1 0</forward>
-                <upward>0 0 1</upward>
-                <link_name>${prop_link}</link_name>
-            </plugin>
-        </gazebo>
+        <xacro:prop_link_creator link_name="${prop_link}" pose_xyz="0 0 0.03" pose_rpy="0 -0 0" mesh_path="${prop_mesh}" scale_xyz="${prop_size_multiplier} ${prop_size_multiplier} ${prop_size_multiplier}" mass="${rmass}" ixx="${rixx}" ixy="${rixy}" ixz="${rixz}" iyy="${riyy}" iyz="${riyz}" izz="${rizz}"/>
+        <xacro:if value="${cw}">
+            <gazebo>
+                <plugin name="${rotor_blade_0}" filename="libLiftDragPlugin.so">
+                    <a0>0.3</a0>
+                    <alpha_stall>1.4</alpha_stall>
+                    <cla>4.2500</cla>
+                    <cda>0.10</cda>
+                    <cma>0.00</cma>
+                    <cla_stall>-0.025</cla_stall>
+                    <cda_stall>0.0</cda_stall>
+                    <cma_stall>0.0</cma_stall>
+                    <area>0.002</area>
+                    <air_density>1.2041</air_density>
+                    <cp>0.084 0 0</cp>
+                    <forward>0 -1 0</forward>
+                    <upward>0 0 1</upward>
+                    <link_name>${prop_link}</link_name>
+                </plugin>
+                <plugin name="${rotor_blade_1}" filename="libLiftDragPlugin.so">
+                    <a0>0.3</a0>
+                    <alpha_stall>1.4</alpha_stall>
+                    <cla>4.2500</cla>
+                    <cda>0.10</cda>
+                    <cma>0.00</cma>
+                    <cla_stall>-0.025</cla_stall>
+                    <cda_stall>0.0</cda_stall>
+                    <cma_stall>0.0</cma_stall>
+                    <area>0.002</area>
+                    <air_density>1.2041</air_density>
+                    <cp>-0.084 0 0</cp>
+                    <forward>0 1 0</forward>
+                    <upward>0 0 1</upward>
+                    <link_name>${prop_link}</link_name>
+                </plugin>
+            </gazebo>
+        </xacro:if>
+        <xacro:unless value="${cw}">
+            <gazebo>
+                <plugin name="${rotor_blade_0}" filename="libLiftDragPlugin.so">
+                    <a0>0.3</a0>
+                    <alpha_stall>1.4</alpha_stall>
+                    <cla>4.2500</cla>
+                    <cda>0.10</cda>
+                    <cma>0.00</cma>
+                    <cla_stall>-0.025</cla_stall>
+                    <cda_stall>0.0</cda_stall>
+                    <cma_stall>0.0</cma_stall>
+                    <area>0.002</area>
+                    <air_density>1.2041</air_density>
+                    <cp>0.084 0 0</cp>
+                    <forward>0 1 0</forward>
+                    <upward>0 0 1</upward>
+                    <link_name>${prop_link}</link_name>
+                </plugin>
+                <plugin name="${rotor_blade_1}" filename="libLiftDragPlugin.so">
+                    <a0>0.3</a0>
+                    <alpha_stall>1.4</alpha_stall>
+                    <cla>4.2500</cla>
+                    <cda>0.10</cda>
+                    <cma>0.00</cma>
+                    <cla_stall>-0.025</cla_stall>
+                    <cda_stall>0.0</cda_stall>
+                    <cma_stall>0.0</cma_stall>
+                    <area>0.002</area>
+                    <air_density>1.2041</air_density>
+                    <cp>-0.084 0 0</cp>
+                    <forward>0 -1 0</forward>
+                    <upward>0 0 1</upward>
+                    <link_name>${prop_link}</link_name>
+                </plugin>
+            </gazebo>
+        </xacro:unless>
     </xacro:macro>
     <xacro:macro name="link_creator_foundation" params="link_name pose_xyz pose_rpy mesh_path scale_xyz **extra_collision **seperate_collider **extra_visual **extra_settings">
