Commit message: not flying...

File: models/copterPIX/robot.urdf.xacro (robot description, xacro)
@@ -7,13 +7,13 @@
   <xacro:property name="prop_ccw_mesh" value="$(find drone)/STLs/iris_prop_ccw.dae"/>
   <!-- Base link -->
-  <link name="base_link">
+  <!-- <link name="base_link"> -->
     <!-- You can leave this link empty if you don't need a specific geometry or inertial properties for the base -->
-  </link>
+  <!-- </link> -->
   <!-- Joint (fixed) -->
-  <joint name="fixed_joint" type="fixed">
+  <!-- <joint name="fixed_joint" type="fixed">
     <parent link="base_link"/>
     <child link="core_link"/>
     <origin xyz="0 0 0.6" rpy="0 0 0"/>
-  </joint>
+  </joint> -->
   <xacro:property name="g_mms_to_kg_ms" value="1000000000" />
   <!-- <xacro:property name="mass" value="26.0" />
@@ -24,5 +24,5 @@
   <xacro:property name="iyz" value="${50504029566.32 / g_mms_to_kg_ms}"/>
   <xacro:property name="izz" value="${574188826210.05 / g_mms_to_kg_ms}"/> -->
-  <xacro:property name="mass" value="2.5" />
+  <xacro:property name="mass" value="2.0" />
   <xacro:property name="ixx" value="${0.1}"/>
   <xacro:property name="ixy" value="${0}"/>
@@ -30,30 +30,31 @@
   <xacro:property name="iyy" value="${0.1}"/>
   <xacro:property name="iyz" value="${0}"/>
-  <xacro:property name="izz" value="${0.1}"/>
-  <xacro:link_creator_i link_name="core_link" pose_xyz="0 0 0" pose_rpy="0 0 0" mesh_path="${hex_mesh}" scale_xyz="0.4 0.4 0.04" center_mass_xyz="0 0 -0.18" mass="${mass}" ixx="${ixx}" ixy="${ixy}" ixz="${ixz}" iyy="${iyy}" iyz="${iyz}" izz="${izz}"/>
+  <xacro:property name="izz" value="${0.15}"/>
+  <xacro:link_creator_i link_name="core_link" pose_xyz="0 0 0" pose_rpy="0 0 0" mesh_path="${hex_mesh}" scale_xyz="0.4 0.4 0.04" center_mass_xyz="0 0 -0.25" mass="${mass}" ixx="${ixx}" ixy="${ixy}" ixz="${ixz}" iyy="${iyy}" iyz="${iyz}" izz="${izz}"/>
+  <!-- <xacro:link_creator link_name="core_link" pose_xyz="0 0 0" pose_rpy="0 0 0" mesh_path="${hex_mesh}" scale_xyz="0.4 0.4 0.04"/> -->
   <joint name="leg_0_link_joint" type="fixed">
     <parent link="core_link"/>
     <child link="leg_0_link"/>
   </joint>
-  <xacro:link_creator_i link_name="leg_0_link" pose_xyz="0 0.198 -0.305" pose_rpy="0.305 0 0" mesh_path="$(find drone)/STLs/hexagonal_prism_height_1_outer_diameter_1.stl" scale_xyz="0.024 0.024 0.61" mass="0.2" ixx="0.0" ixy="0.0" ixz="0.0" iyy="0.0" iyz="0.0" izz="0.0"/>
-  <!-- <xacro:link_creator link_name="leg_0_link" pose_xyz="0 0.198 -0.305" pose_rpy="0.305 0 0" mesh_path="${hex_mesh}" scale_xyz="0.024 0.024 0.61"/> -->
+  <!-- <xacro:link_creator_i link_name="leg_0_link" pose_xyz="0 0.198 -0.305" pose_rpy="0.305 0 0" mesh_path="$(find drone)/STLs/hexagonal_prism_height_1_outer_diameter_1.stl" scale_xyz="0.024 0.024 0.61" mass="0.2" ixx="0.0" ixy="0.0" ixz="0.0" iyy="0.0" iyz="0.0" izz="0.0"/> -->
+  <xacro:link_creator link_name="leg_0_link" pose_xyz="0 0.198 -0.305" pose_rpy="0.305 0 0" mesh_path="${hex_mesh}" scale_xyz="0.024 0.024 0.61"/>
   <joint name="leg_1_link_joint" type="fixed">
     <parent link="core_link"/>
     <child link="leg_1_link"/>
   </joint>
-  <xacro:link_creator_i link_name="leg_1_link" pose_xyz="0 -0.198 -0.305" pose_rpy="-0.305 0 0" mesh_path="$(find drone)/STLs/hexagonal_prism_height_1_outer_diameter_1.stl" scale_xyz="0.024 0.024 0.61" mass="0.2" ixx="0.0" ixy="0.0" ixz="0.0" iyy="0.0" iyz="0.0" izz="0.0"/>
-  <!-- <xacro:link_creator link_name="leg_1_link" pose_xyz="0 -0.198 -0.305" pose_rpy="-0.305 0 0" mesh_path="${hex_mesh}" scale_xyz="0.024 0.024 0.61"/> -->
+  <!-- <xacro:link_creator_i link_name="leg_1_link" pose_xyz="0 -0.198 -0.305" pose_rpy="-0.305 0 0" mesh_path="$(find drone)/STLs/hexagonal_prism_height_1_outer_diameter_1.stl" scale_xyz="0.024 0.024 0.61" mass="0.2" ixx="0.0" ixy="0.0" ixz="0.0" iyy="0.0" iyz="0.0" izz="0.0"/> -->
+  <xacro:link_creator link_name="leg_1_link" pose_xyz="0 -0.198 -0.305" pose_rpy="-0.305 0 0" mesh_path="${hex_mesh}" scale_xyz="0.024 0.024 0.61"/>
   <joint name="feet_0_link_joint" type="fixed">
     <parent link="core_link"/>
     <child link="feet_0_link"/>
   </joint>
-  <xacro:link_creator_i link_name="feet_0_link" pose_xyz="0 0.29 -0.6" pose_rpy="0 1.57079633 0" mesh_path="$(find drone)/STLs/hexagonal_prism_height_1_outer_diameter_1.stl" scale_xyz="0.024 0.024 0.58" mass="0.2" ixx="0.0" ixy="0.0" ixz="0.0" iyy="0.0" iyz="0.0" izz="0.0"/>
-  <!-- <xacro:link_creator link_name="feet_0_link" pose_xyz="0 0.29 -0.6" pose_rpy="0 1.57079633 0" mesh_path="${hex_mesh}" scale_xyz="0.024 0.024 0.58"/> -->
+  <!-- <xacro:link_creator_i link_name="feet_0_link" pose_xyz="0 0.29 -0.6" pose_rpy="0 1.57079633 0" mesh_path="$(find drone)/STLs/hexagonal_prism_height_1_outer_diameter_1.stl" scale_xyz="0.024 0.024 0.58" mass="0.2" ixx="0.0" ixy="0.0" ixz="0.0" iyy="0.0" iyz="0.0" izz="0.0"/> -->
+  <xacro:link_creator link_name="feet_0_link" pose_xyz="0 0.29 -0.6" pose_rpy="0 1.57079633 0" mesh_path="${hex_mesh}" scale_xyz="0.024 0.024 0.58"/>
   <joint name="feet_1_link_joint" type="fixed">
     <parent link="core_link"/>
     <child link="feet_1_link"/>
   </joint>
-  <xacro:link_creator_i link_name="feet_1_link" pose_xyz="0 -0.29 -0.6" pose_rpy="0 1.57079633 0" mesh_path="$(find drone)/STLs/hexagonal_prism_height_1_outer_diameter_1.stl" scale_xyz="0.024 0.024 0.58" mass="0.2" ixx="0.0" ixy="0.0" ixz="0.0" iyy="0.0" iyz="0.0" izz="0.0"/>
-  <!-- <xacro:link_creator link_name="feet_1_link" pose_xyz="0 -0.29 -0.6" pose_rpy="0 1.57079633 0" mesh_path="${hex_mesh}" scale_xyz="0.024 0.024 0.58"/> -->
+  <!-- <xacro:link_creator_i link_name="feet_1_link" pose_xyz="0 -0.29 -0.6" pose_rpy="0 1.57079633 0" mesh_path="$(find drone)/STLs/hexagonal_prism_height_1_outer_diameter_1.stl" scale_xyz="0.024 0.024 0.58" mass="0.2" ixx="0.0" ixy="0.0" ixz="0.0" iyy="0.0" iyz="0.0" izz="0.0"/> -->
+  <xacro:link_creator link_name="feet_1_link" pose_xyz="0 -0.29 -0.6" pose_rpy="0 1.57079633 0" mesh_path="${hex_mesh}" scale_xyz="0.024 0.024 0.58"/>
   <!-- Define the drone arms using the macro -->
   <xacro:property name="deg_to_rad" value="0.0174533" />

File: xacros/macro.xacro (robot description, xacro)
@@ -1,5 +1,5 @@
 <?xml version="1.0"?>
 <robot xmlns:xacro="http://www.ros.org/wiki/xacro">
-    <xacro:macro name="drone_arm" params="num parent_link dis_from_center length diameter arm_incline_angle arm_mesh prop_mesh cw prop_size_multiplier amass:='0.2' aixx:='0' aixy:='0' aixz:='0' aiyy:='0' aiyz:='0' aizz:='0' rmass rixx rixy rixz riyy riyz rizz angle">
+    <xacro:macro name="drone_arm" params="num parent_link dis_from_center length diameter arm_incline_angle arm_mesh prop_mesh cw prop_size_multiplier amass:='0.001' aixx:='0' aixy:='0' aixz:='0' aiyy:='0' aiyz:='0' aizz:='0' rmass rixx rixy rixz riyy riyz rizz angle">
         <xacro:property name="core_arm_joint" value="core_arm_joint_${num}" />
         <xacro:property name="arm_link" value="arm_link_${num}" />
@@ -14,4 +14,5 @@
         </joint>
         <xacro:link_creator_i link_name="${arm_link}" pose_xyz="0 ${cos(arm_incline_angle) * (length / 2.0) + dis_from_center} ${sin(arm_incline_angle) * (length / 2.0)}" pose_rpy="${arm_incline_angle + 1.57079632679} 0 0" mesh_path="${arm_mesh}" scale_xyz="${diameter} ${diameter} ${length}" mass="${amass}" ixx="${aixx}" ixy="${aixy}" ixz="${aixz}" iyy="${aiyy}" iyz="${aiyz}" izz="${aizz}"/>
+        <!-- <xacro:link_creator link_name="${arm_link}" pose_xyz="0 ${cos(arm_incline_angle) * (length / 2.0) + dis_from_center} ${sin(arm_incline_angle) * (length / 2.0)}" pose_rpy="${arm_incline_angle + 1.57079632679} 0 0" mesh_path="${arm_mesh}" scale_xyz="${diameter} ${diameter} ${length}"/> -->
         <joint name="${rotor_joint}" type="continuous">
             <parent link="${arm_link}"/>
@@ -29,4 +30,7 @@
         </gazebo>
         <xacro:prop_link_creator link_name="${prop_link}" pose_xyz="0 0 0.03" pose_rpy="0 -0 0" mesh_path="${prop_mesh}" scale_xyz="${prop_size_multiplier} ${prop_size_multiplier} ${prop_size_multiplier}" mass="${rmass}" ixx="${rixx}" ixy="${rixy}" ixz="${rixz}" iyy="${riyy}" iyz="${riyz}" izz="${rizz}"/>
+        <xacro:property name="cp" value="0.008"/>
+        <xacro:property name="cp_negative" value="${-1 * cp}"/>
+        <xacro:property name="area" value="0.002"/> <!--used to be 0.002-->
         <xacro:if value="${cw}">
             <gazebo>
@@ -40,7 +44,7 @@
                     <cda_stall>0.0</cda_stall>
                     <cma_stall>0.0</cma_stall>
-                    <area>0.002</area>
+                    <area>${area}</area>
                     <air_density>1.2041</air_density>
-                    <cp>0.084 0 0</cp>
+                    <cp>${cp} 0 0</cp>
                     <forward>0 -1 0</forward>
                     <upward>0 0 1</upward>
@@ -56,7 +60,7 @@
                     <cda_stall>0.0</cda_stall>
                     <cma_stall>0.0</cma_stall>
-                    <area>0.002</area>
+                    <area>${area}</area>
                     <air_density>1.2041</air_density>
-                    <cp>-0.084 0 0</cp>
+                    <cp>${cp_negative} 0 0</cp>
                     <forward>0 1 0</forward>
                     <upward>0 0 1</upward>
@@ -76,7 +80,7 @@
                     <cda_stall>0.0</cda_stall>
                     <cma_stall>0.0</cma_stall>
-                    <area>0.002</area>
+                    <area>${area}</area>
                     <air_density>1.2041</air_density>
-                    <cp>0.084 0 0</cp>
+                    <cp>${cp} 0 0</cp>
                     <forward>0 1 0</forward>
                     <upward>0 0 1</upward>
@@ -92,7 +96,7 @@
                     <cda_stall>0.0</cda_stall>
                     <cma_stall>0.0</cma_stall>
-                    <area>0.002</area>
+                    <area>${area}</area>
                     <air_density>1.2041</air_density>
-                    <cp>-0.084 0 0</cp>
+                    <cp>${cp_negative} 0 0</cp>
                     <forward>0 -1 0</forward>
                     <upward>0 0 1</upward>
