Commit message: not working

File: models/copterPIX/robot.urdf.xacro (robot description, xacro)
@@ -1,4 +1,5 @@
 <?xml version="1.0" ?>
 <robot name="copterPIX" xmlns:xacro="http://www.ros.org/wiki/xacro">
+  <origin xyz="0 0 0.6" rpy="0 0 0"/>
   <xacro:include filename="$(find drone)/xacros/macro.xacro"/>
   <xacro:include filename="ardupilot_plugin.xacro"/>
@@ -6,14 +7,4 @@
   <xacro:property name="prop_cw_mesh" value="$(find drone)/STLs/iris_prop_cw.dae"/>
   <xacro:property name="prop_ccw_mesh" value="$(find drone)/STLs/iris_prop_ccw.dae"/>
-  <!-- Base link -->
-  <link name="base_link">
-    <!-- You can leave this link empty if you don't need a specific geometry or inertial properties for the base -->
-  </link>
-  <!-- Joint (fixed) -->
-  <joint name="fixed_joint" type="fixed">
-    <parent link="base_link"/>
-    <child link="core_link"/>
-    <origin xyz="0 0 0.6" rpy="0 0 0"/>
-  </joint>
   <xacro:property name="g_mms_to_kg_ms" value="1000000000"/>
   <!-- <xacro:property name="mass" value="26.0" />
@@ -32,13 +23,13 @@
   <xacro:property name="iyz" value="${0 * s}"/>
   <xacro:property name="izz" value="${1.6 * s}"/> -->
-  <xacro:property name="mass" value="26" />
-  <xacro:property name="s" value="50" />
-  <xacro:property name="ixx" value="${1}"/>
-  <xacro:property name="ixy" value="${0}"/>
-  <xacro:property name="ixz" value="${0}"/>
-  <xacro:property name="iyy" value="${1}"/>
-  <xacro:property name="iyz" value="${0}"/>
-  <xacro:property name="izz" value="${1.6}"/>
-  <xacro:link_creator_i_foundation link_name="core_link" pose_xyz="0 0 0" pose_rpy="0 0 0" mesh_path="${hex_mesh}" scale_xyz="0.4 0.4 0.04" center_mass_xyz="0 0 -0.15" mass="${mass}" ixx="${ixx}" ixy="${ixy}" ixz="${ixz}" iyy="${iyy}" iyz="${iyz}" izz="${izz}">
+  <xacro:property name="mass" value="4.5" />
+  <xacro:property name="s" value="2"/>
+  <xacro:property name="ixx" value="${0.5 * s}"/>
+  <xacro:property name="ixy" value="${0 * s}"/>
+  <xacro:property name="ixz" value="${0 * s}"/>
+  <xacro:property name="iyy" value="${0.5 * s}"/>
+  <xacro:property name="iyz" value="${0 * s}"/>
+  <xacro:property name="izz" value="${0.75 * s}"/>
+  <xacro:link_creator_i_foundation link_name="base_link" pose_xyz="0 0 0" pose_rpy="0 0 0" mesh_path="${hex_mesh}" scale_xyz="0.4 0.4 0.04" seperate_collider_xyzrpy="0 0 -0.3 0 0 0" center_mass_xyz="0 0 -0.5" mass="${mass}" ixx="${ixx}" ixy="${ixy}" ixz="${ixz}" iyy="${iyy}" iyz="${iyz}" izz="${izz}">
     <extra_collision>
       <surface>
@@ -57,11 +48,11 @@
       </surface>
     </extra_collision>
-    <seperate_collider><box filename="${hex_mesh}" scale="0.4 0.4 0.04"/></seperate_collider>
+    <seperate_collider><cylinder radius="0.45" length="0.62"/></seperate_collider>
     <extra_visual/>
     <extra_settings/>
   </xacro:link_creator_i_foundation>
-  <!-- <xacro:link_creator link_name="core_link" pose_xyz="0 0 0" pose_rpy="0 0 0" mesh_path="${hex_mesh}" scale_xyz="0.4 0.4 0.04"/> -->
+  <!-- <xacro:link_creator link_name="base_link" pose_xyz="0 0 0" pose_rpy="0 0 0" mesh_path="${hex_mesh}" scale_xyz="0.4 0.4 0.04"/> -->
   <joint name="leg_0_link_joint" type="fixed">
-    <parent link="core_link"/>
+    <parent link="base_link"/>
     <child link="leg_0_link"/>
   </joint>
@@ -69,5 +60,5 @@
   <xacro:link_creator link_name="leg_0_link" pose_xyz="0 0.198 -0.305" pose_rpy="0.305 0 0" mesh_path="${hex_mesh}" scale_xyz="0.024 0.024 0.61"/>
   <joint name="leg_1_link_joint" type="fixed">
-    <parent link="core_link"/>
+    <parent link="base_link"/>
     <child link="leg_1_link"/>
   </joint>
@@ -75,5 +66,5 @@
   <xacro:link_creator link_name="leg_1_link" pose_xyz="0 -0.198 -0.305" pose_rpy="-0.305 0 0" mesh_path="${hex_mesh}" scale_xyz="0.024 0.024 0.61"/>
   <joint name="feet_0_link_joint" type="fixed">
-    <parent link="core_link"/>
+    <parent link="base_link"/>
     <child link="feet_0_link"/>
   </joint>
@@ -81,5 +72,5 @@
   <xacro:link_creator link_name="feet_0_link" pose_xyz="0 0.29 -0.6" pose_rpy="0 1.57079633 0" mesh_path="${hex_mesh}" scale_xyz="0.024 0.024 0.58"/>
   <joint name="feet_1_link_joint" type="fixed">
-    <parent link="core_link"/>
+    <parent link="base_link"/>
     <child link="feet_1_link"/>
   </joint>
@@ -88,22 +79,22 @@
   <!-- Define the drone arms using the macro -->
   <xacro:property name="deg_to_rad" value="0.0174533" />
-  <!-- <xacro:drone_arm num="0" parent_link="core_link" dis_from_center="0.175" length="0.56" diameter="0.025" arm_incline_angle="${4 * deg_to_rad}" arm_mesh="${hex_mesh}" prop_mesh="${prop_cw_mesh}" prop_size_multiplier="2.04" amass="0.2" aixx="0" aixy="0" aixz="0" aiyy="0" aiyz="0" aizz="0" rmass="0.2" rixx="0.000312" rixy="0" rixz="0" riyy="0.0053345" riyz="0" rizz="0.005363328" angle="${0}"/>
-  <xacro:drone_arm num="1" parent_link="core_link" dis_from_center="0.175" length="0.56" diameter="0.025" arm_incline_angle="${4 * deg_to_rad}" arm_mesh="${hex_mesh}" prop_mesh="${prop_ccw_mesh}" prop_size_multiplier="2.04" amass="0.2" aixx="0" aixy="0" aixz="0" aiyy="0" aiyz="0" aizz="0" rmass="0.2" rixx="0.000312" rixy="0" rixz="0" riyy="0.0053345" riyz="0" rizz="0.005363328" angle="${180 * deg_to_rad}"/>
-  <xacro:drone_arm num="2" parent_link="core_link" dis_from_center="0.175" length="0.56" diameter="0.025" arm_incline_angle="${4 * deg_to_rad}" arm_mesh="${hex_mesh}" prop_mesh="${prop_cw_mesh}" prop_size_multiplier="2.04" amass="0.2" aixx="0" aixy="0" aixz="0" aiyy="0" aiyz="0" aizz="0" rmass="0.2" rixx="0.000312" rixy="0" rixz="0" riyy="0.0053345" riyz="0" rizz="0.005363328" angle="${120 * deg_to_rad}"/>
-  <xacro:drone_arm num="3" parent_link="core_link" dis_from_center="0.175" length="0.56" diameter="0.025" arm_incline_angle="${4 * deg_to_rad}" arm_mesh="${hex_mesh}" prop_mesh="${prop_ccw_mesh}" prop_size_multiplier="2.04" amass="0.2" aixx="0" aixy="0" aixz="0" aiyy="0" aiyz="0" aizz="0" rmass="0.2" rixx="0.000312" rixy="0" rixz="0" riyy="0.0053345" riyz="0" rizz="0.005363328" angle="${300 * deg_to_rad}"/>
-  <xacro:drone_arm num="4" parent_link="core_link" dis_from_center="0.175" length="0.56" diameter="0.025" arm_incline_angle="${4 * deg_to_rad}" arm_mesh="${hex_mesh}" prop_mesh="${prop_ccw_mesh}" prop_size_multiplier="2.04" amass="0.2" aixx="0" aixy="0" aixz="0" aiyy="0" aiyz="0" aizz="0" rmass="0.2" rixx="0.000312" rixy="0" rixz="0" riyy="0.0053345" riyz="0" rizz="0.005363328" angle="${60 * deg_to_rad}"/>
-  <xacro:drone_arm num="5" parent_link="core_link" dis_from_center="0.175" length="0.56" diameter="0.025" arm_incline_angle="${4 * deg_to_rad}" arm_mesh="${hex_mesh}" prop_mesh="${prop_cw_mesh}" prop_size_multiplier="2.04" amass="0.2" aixx="0" aixy="0" aixz="0" aiyy="0" aiyz="0" aizz="0" rmass="0.2" rixx="0.000312" rixy="0" rixz="0" riyy="0.0053345" riyz="0" rizz="0.005363328" angle="${240 * deg_to_rad}"/> -->
-  <!-- <xacro:drone_arm num="0" parent_link="core_link" dis_from_center="0.175" length="0.56" diameter="0.025" arm_incline_angle="${4 * deg_to_rad}" arm_mesh="${hex_mesh}" prop_mesh="${prop_cw_mesh}" cw="true" prop_size_multiplier="2.04" rmass="0.2" rixx="0.000312" rixy="0" rixz="0" riyy="0.0053345" riyz="0" rizz="0.005363328" angle="${0 * deg_to_rad}"/>
-  <xacro:drone_arm num="1" parent_link="core_link" dis_from_center="0.175" length="0.56" diameter="0.025" arm_incline_angle="${4 * deg_to_rad}" arm_mesh="${hex_mesh}" prop_mesh="${prop_ccw_mesh}" cw="false" prop_size_multiplier="2.04" rmass="0.2" rixx="0.000312" rixy="0" rixz="0" riyy="0.0053345" riyz="0" rizz="0.005363328" angle="${180 * deg_to_rad}"/>
-  <xacro:drone_arm num="2" parent_link="core_link" dis_from_center="0.175" length="0.56" diameter="0.025" arm_incline_angle="${4 * deg_to_rad}" arm_mesh="${hex_mesh}" prop_mesh="${prop_cw_mesh}" cw="true" prop_size_multiplier="2.04" rmass="0.2" rixx="0.000312" rixy="0" rixz="0" riyy="0.0053345" riyz="0" rizz="0.005363328" angle="${120 * deg_to_rad}"/>
-  <xacro:drone_arm num="3" parent_link="core_link" dis_from_center="0.175" length="0.56" diameter="0.025" arm_incline_angle="${4 * deg_to_rad}" arm_mesh="${hex_mesh}" prop_mesh="${prop_ccw_mesh}" cw="false" prop_size_multiplier="2.04" rmass="0.2" rixx="0.000312" rixy="0" rixz="0" riyy="0.0053345" riyz="0" rizz="0.005363328" angle="${300 * deg_to_rad}"/>
-  <xacro:drone_arm num="4" parent_link="core_link" dis_from_center="0.175" length="0.56" diameter="0.025" arm_incline_angle="${4 * deg_to_rad}" arm_mesh="${hex_mesh}" prop_mesh="${prop_ccw_mesh}" cw="false" prop_size_multiplier="2.04" rmass="0.2" rixx="0.000312" rixy="0" rixz="0" riyy="0.0053345" riyz="0" rizz="0.005363328" angle="${60 * deg_to_rad}"/>
-  <xacro:drone_arm num="5" parent_link="core_link" dis_from_center="0.175" length="0.56" diameter="0.025" arm_incline_angle="${4 * deg_to_rad}" arm_mesh="${hex_mesh}" prop_mesh="${prop_cw_mesh}" cw="true" prop_size_multiplier="2.04" rmass="0.2" rixx="0.000312" rixy="0" rixz="0" riyy="0.0053345" riyz="0" rizz="0.005363328" angle="${240 * deg_to_rad}"/> -->
-  <xacro:drone_arm num="0" parent_link="core_link" dis_from_center="0.175" length="0.56" diameter="0.025" arm_incline_angle="${6 * deg_to_rad}" arm_mesh="${hex_mesh}" prop_mesh="${prop_cw_mesh}"  cw="true"  prop_size_multiplier="2.04" rmass="0.025" rixx="0.00000975" rixy="0" rixz="0" riyy="0.000166704" riyz="0" rizz="0.000167604" angle="${0 * deg_to_rad}"/>
-  <xacro:drone_arm num="1" parent_link="core_link" dis_from_center="0.175" length="0.56" diameter="0.025" arm_incline_angle="${6 * deg_to_rad}" arm_mesh="${hex_mesh}" prop_mesh="${prop_ccw_mesh}" cw="false" prop_size_multiplier="2.04" rmass="0.025" rixx="0.00000975" rixy="0" rixz="0" riyy="0.000166704" riyz="0" rizz="0.000167604" angle="${180 * deg_to_rad}"/>
-  <xacro:drone_arm num="2" parent_link="core_link" dis_from_center="0.175" length="0.56" diameter="0.025" arm_incline_angle="${6 * deg_to_rad}" arm_mesh="${hex_mesh}" prop_mesh="${prop_cw_mesh}"  cw="true"  prop_size_multiplier="2.04" rmass="0.025" rixx="0.00000975" rixy="0" rixz="0" riyy="0.000166704" riyz="0" rizz="0.000167604" angle="${120 * deg_to_rad}"/>
-  <xacro:drone_arm num="3" parent_link="core_link" dis_from_center="0.175" length="0.56" diameter="0.025" arm_incline_angle="${6 * deg_to_rad}" arm_mesh="${hex_mesh}" prop_mesh="${prop_ccw_mesh}" cw="false" prop_size_multiplier="2.04" rmass="0.025" rixx="0.00000975" rixy="0" rixz="0" riyy="0.000166704" riyz="0" rizz="0.000167604" angle="${300 * deg_to_rad}"/>
-  <xacro:drone_arm num="4" parent_link="core_link" dis_from_center="0.175" length="0.56" diameter="0.025" arm_incline_angle="${6 * deg_to_rad}" arm_mesh="${hex_mesh}" prop_mesh="${prop_ccw_mesh}" cw="false" prop_size_multiplier="2.04" rmass="0.025" rixx="0.00000975" rixy="0" rixz="0" riyy="0.000166704" riyz="0" rizz="0.000167604" angle="${60 * deg_to_rad}"/>
-  <xacro:drone_arm num="5" parent_link="core_link" dis_from_center="0.175" length="0.56" diameter="0.025" arm_incline_angle="${6 * deg_to_rad}" arm_mesh="${hex_mesh}" prop_mesh="${prop_cw_mesh}"  cw="true"  prop_size_multiplier="2.04" rmass="0.025" rixx="0.00000975" rixy="0" rixz="0" riyy="0.000166704" riyz="0" rizz="0.000167604" angle="${240 * deg_to_rad}"/>
+  <!-- <xacro:drone_arm num="0" parent_link="base_link" dis_from_center="0.175" length="0.56" diameter="0.025" arm_incline_angle="${4 * deg_to_rad}" arm_mesh="${hex_mesh}" prop_mesh="${prop_cw_mesh}" prop_size_multiplier="2.04" amass="0.2" aixx="0" aixy="0" aixz="0" aiyy="0" aiyz="0" aizz="0" rmass="0.2" rixx="0.000312" rixy="0" rixz="0" riyy="0.0053345" riyz="0" rizz="0.005363328" angle="${0}"/>
+  <xacro:drone_arm num="1" parent_link="base_link" dis_from_center="0.175" length="0.56" diameter="0.025" arm_incline_angle="${4 * deg_to_rad}" arm_mesh="${hex_mesh}" prop_mesh="${prop_ccw_mesh}" prop_size_multiplier="2.04" amass="0.2" aixx="0" aixy="0" aixz="0" aiyy="0" aiyz="0" aizz="0" rmass="0.2" rixx="0.000312" rixy="0" rixz="0" riyy="0.0053345" riyz="0" rizz="0.005363328" angle="${180 * deg_to_rad}"/>
+  <xacro:drone_arm num="2" parent_link="base_link" dis_from_center="0.175" length="0.56" diameter="0.025" arm_incline_angle="${4 * deg_to_rad}" arm_mesh="${hex_mesh}" prop_mesh="${prop_cw_mesh}" prop_size_multiplier="2.04" amass="0.2" aixx="0" aixy="0" aixz="0" aiyy="0" aiyz="0" aizz="0" rmass="0.2" rixx="0.000312" rixy="0" rixz="0" riyy="0.0053345" riyz="0" rizz="0.005363328" angle="${120 * deg_to_rad}"/>
+  <xacro:drone_arm num="3" parent_link="base_link" dis_from_center="0.175" length="0.56" diameter="0.025" arm_incline_angle="${4 * deg_to_rad}" arm_mesh="${hex_mesh}" prop_mesh="${prop_ccw_mesh}" prop_size_multiplier="2.04" amass="0.2" aixx="0" aixy="0" aixz="0" aiyy="0" aiyz="0" aizz="0" rmass="0.2" rixx="0.000312" rixy="0" rixz="0" riyy="0.0053345" riyz="0" rizz="0.005363328" angle="${300 * deg_to_rad}"/>
+  <xacro:drone_arm num="4" parent_link="base_link" dis_from_center="0.175" length="0.56" diameter="0.025" arm_incline_angle="${4 * deg_to_rad}" arm_mesh="${hex_mesh}" prop_mesh="${prop_ccw_mesh}" prop_size_multiplier="2.04" amass="0.2" aixx="0" aixy="0" aixz="0" aiyy="0" aiyz="0" aizz="0" rmass="0.2" rixx="0.000312" rixy="0" rixz="0" riyy="0.0053345" riyz="0" rizz="0.005363328" angle="${60 * deg_to_rad}"/>
+  <xacro:drone_arm num="5" parent_link="base_link" dis_from_center="0.175" length="0.56" diameter="0.025" arm_incline_angle="${4 * deg_to_rad}" arm_mesh="${hex_mesh}" prop_mesh="${prop_cw_mesh}" prop_size_multiplier="2.04" amass="0.2" aixx="0" aixy="0" aixz="0" aiyy="0" aiyz="0" aizz="0" rmass="0.2" rixx="0.000312" rixy="0" rixz="0" riyy="0.0053345" riyz="0" rizz="0.005363328" angle="${240 * deg_to_rad}"/> -->
+  <!-- <xacro:drone_arm num="0" parent_link="base_link" dis_from_center="0.175" length="0.56" diameter="0.025" arm_incline_angle="${4 * deg_to_rad}" arm_mesh="${hex_mesh}" prop_mesh="${prop_cw_mesh}" cw="true" prop_size_multiplier="2.04" rmass="0.2" rixx="0.000312" rixy="0" rixz="0" riyy="0.0053345" riyz="0" rizz="0.005363328" angle="${0 * deg_to_rad}"/>
+  <xacro:drone_arm num="1" parent_link="base_link" dis_from_center="0.175" length="0.56" diameter="0.025" arm_incline_angle="${4 * deg_to_rad}" arm_mesh="${hex_mesh}" prop_mesh="${prop_ccw_mesh}" cw="false" prop_size_multiplier="2.04" rmass="0.2" rixx="0.000312" rixy="0" rixz="0" riyy="0.0053345" riyz="0" rizz="0.005363328" angle="${180 * deg_to_rad}"/>
+  <xacro:drone_arm num="2" parent_link="base_link" dis_from_center="0.175" length="0.56" diameter="0.025" arm_incline_angle="${4 * deg_to_rad}" arm_mesh="${hex_mesh}" prop_mesh="${prop_cw_mesh}" cw="true" prop_size_multiplier="2.04" rmass="0.2" rixx="0.000312" rixy="0" rixz="0" riyy="0.0053345" riyz="0" rizz="0.005363328" angle="${120 * deg_to_rad}"/>
+  <xacro:drone_arm num="3" parent_link="base_link" dis_from_center="0.175" length="0.56" diameter="0.025" arm_incline_angle="${4 * deg_to_rad}" arm_mesh="${hex_mesh}" prop_mesh="${prop_ccw_mesh}" cw="false" prop_size_multiplier="2.04" rmass="0.2" rixx="0.000312" rixy="0" rixz="0" riyy="0.0053345" riyz="0" rizz="0.005363328" angle="${300 * deg_to_rad}"/>
+  <xacro:drone_arm num="4" parent_link="base_link" dis_from_center="0.175" length="0.56" diameter="0.025" arm_incline_angle="${4 * deg_to_rad}" arm_mesh="${hex_mesh}" prop_mesh="${prop_ccw_mesh}" cw="false" prop_size_multiplier="2.04" rmass="0.2" rixx="0.000312" rixy="0" rixz="0" riyy="0.0053345" riyz="0" rizz="0.005363328" angle="${60 * deg_to_rad}"/>
+  <xacro:drone_arm num="5" parent_link="base_link" dis_from_center="0.175" length="0.56" diameter="0.025" arm_incline_angle="${4 * deg_to_rad}" arm_mesh="${hex_mesh}" prop_mesh="${prop_cw_mesh}" cw="true" prop_size_multiplier="2.04" rmass="0.2" rixx="0.000312" rixy="0" rixz="0" riyy="0.0053345" riyz="0" rizz="0.005363328" angle="${240 * deg_to_rad}"/> -->
+  <xacro:drone_arm num="0" parent_link="base_link" dis_from_center="0.175" length="0.56" diameter="0.025" arm_incline_angle="${6 * deg_to_rad}" arm_mesh="${hex_mesh}" prop_mesh="${prop_cw_mesh}"  cw="true"  prop_size_multiplier="2.04" rmass="0.025" rixx="0.00000975" rixy="0" rixz="0" riyy="0.000166704" riyz="0" rizz="0.000167604" angle="${0 * deg_to_rad}"/>
+  <xacro:drone_arm num="1" parent_link="base_link" dis_from_center="0.175" length="0.56" diameter="0.025" arm_incline_angle="${6 * deg_to_rad}" arm_mesh="${hex_mesh}" prop_mesh="${prop_ccw_mesh}" cw="false" prop_size_multiplier="2.04" rmass="0.025" rixx="0.00000975" rixy="0" rixz="0" riyy="0.000166704" riyz="0" rizz="0.000167604" angle="${180 * deg_to_rad}"/>
+  <xacro:drone_arm num="2" parent_link="base_link" dis_from_center="0.175" length="0.56" diameter="0.025" arm_incline_angle="${6 * deg_to_rad}" arm_mesh="${hex_mesh}" prop_mesh="${prop_cw_mesh}"  cw="true"  prop_size_multiplier="2.04" rmass="0.025" rixx="0.00000975" rixy="0" rixz="0" riyy="0.000166704" riyz="0" rizz="0.000167604" angle="${120 * deg_to_rad}"/>
+  <xacro:drone_arm num="3" parent_link="base_link" dis_from_center="0.175" length="0.56" diameter="0.025" arm_incline_angle="${6 * deg_to_rad}" arm_mesh="${hex_mesh}" prop_mesh="${prop_ccw_mesh}" cw="false" prop_size_multiplier="2.04" rmass="0.025" rixx="0.00000975" rixy="0" rixz="0" riyy="0.000166704" riyz="0" rizz="0.000167604" angle="${300 * deg_to_rad}"/>
+  <xacro:drone_arm num="4" parent_link="base_link" dis_from_center="0.175" length="0.56" diameter="0.025" arm_incline_angle="${6 * deg_to_rad}" arm_mesh="${hex_mesh}" prop_mesh="${prop_ccw_mesh}" cw="false" prop_size_multiplier="2.04" rmass="0.025" rixx="0.00000975" rixy="0" rixz="0" riyy="0.000166704" riyz="0" rizz="0.000167604" angle="${60 * deg_to_rad}"/>
+  <xacro:drone_arm num="5" parent_link="base_link" dis_from_center="0.175" length="0.56" diameter="0.025" arm_incline_angle="${6 * deg_to_rad}" arm_mesh="${hex_mesh}" prop_mesh="${prop_cw_mesh}"  cw="true"  prop_size_multiplier="2.04" rmass="0.025" rixx="0.00000975" rixy="0" rixz="0" riyy="0.000166704" riyz="0" rizz="0.000167604" angle="${240 * deg_to_rad}"/>
   <gazebo>
     <!-- <link name='odometry_sensorgt_link'>
@@ -124,5 +115,5 @@
     <joint name='odometry_sensorgt_joint' type='revolute'>
       <child>odometry_sensorgt_link</child>
-      <parent>core_link</parent>
+      <parent>base_link</parent>
       <axis>
         <xyz>0 0 1</xyz>
@@ -164,6 +155,6 @@
     </link>
     <joint name='imu_joint' type='fixed'>
+      <parent>base_link</parent>
       <child>imu_link</child>
-      <parent>core_link</parent>
       <axis>
         <xyz>0 0 1</xyz>
