Commit message: not working

File: xacros/macro.xacro (robot description, xacro)
@@ -2,5 +2,5 @@
 <robot xmlns:xacro="http://www.ros.org/wiki/xacro">
     <xacro:macro name="drone_arm" params="num parent_link dis_from_center length diameter arm_incline_angle arm_mesh prop_mesh cw prop_size_multiplier amass:='0.001' aixx:='0' aixy:='0' aixz:='0' aiyy:='0' aiyz:='0' aizz:='0' rmass rixx rixy rixz riyy riyz rizz angle">
-        <xacro:property name="core_arm_joint" value="core_arm_joint_${num}" />
+        <xacro:property name="base_arm_joint" value="base_arm_joint_${num}" />
         <xacro:property name="arm_link" value="arm_link_${num}" />
         <xacro:property name="rotor_joint" value="rotor_joint_${num}" />
@@ -8,5 +8,5 @@
         <xacro:property name="rotor_blade_0" value="rotor_${num}_blade_0" />
         <xacro:property name="rotor_blade_1" value="rotor_${num}_blade_1" />
-        <joint name="${core_arm_joint}" type="fixed">
+        <joint name="${base_arm_joint}" type="fixed">
             <parent link="${parent_link}"/>
             <child link="${arm_link}"/>
@@ -23,9 +23,9 @@
         </joint>
         <gazebo reference="${rotor_joint}">
-            <!-- <physics> -->
+            <physics>
                 <ode>
                     <implicit_spring_damper>1</implicit_spring_damper>
                 </ode>
-            <!-- </physics> -->
+            </physics>
         </gazebo>
         <xacro:prop_link_creator link_name="${prop_link}" pose_xyz="0 0 0.03" pose_rpy="0 -0 0" mesh_path="${prop_mesh}" scale_xyz="${prop_size_multiplier} ${prop_size_multiplier} ${prop_size_multiplier}" mass="${rmass}" ixx="${rixx}" ixy="${rixy}" ixz="${rixz}" iyy="${riyy}" iyz="${riyz}" izz="${rizz}"/>
@@ -106,5 +106,5 @@
         </xacro:unless>
     </xacro:macro>
-    <xacro:macro name="link_creator_foundation" params="link_name pose_xyz pose_rpy mesh_path scale_xyz **extra_collision **seperate_collider **extra_visual **extra_settings">
+    <xacro:macro name="link_creator_foundation" params="link_name pose_xyz pose_rpy mesh_path scale_xyz **extra_visual **extra_settings">
         <link name="${link_name}">
             <visual>
@@ -115,14 +115,4 @@
                 <xacro:insert_block name="extra_visual"/>
             </visual>
-            <collision>
-                <geometry>
-                    <!-- <xacro:unless value="${seperate_collider}">
-                        <mesh filename="${mesh_path}" scale="${scale_xyz}"/>
-                    </xacro:unless> -->
-                    <xacro:insert_block name="seperate_collider"/>
-                </geometry>
-                <origin xyz="${pose_xyz}" rpy="${pose_rpy}"/>
-                <xacro:insert_block name="extra_collision"/>
-            </collision>
             <xacro:insert_block name="extra_settings"/>
         </link>
@@ -130,16 +120,25 @@
     <xacro:macro name="link_creator" params="link_name pose_xyz pose_rpy mesh_path scale_xyz">
         <xacro:link_creator_foundation link_name="${link_name}" pose_xyz="${pose_xyz}" pose_rpy="${pose_rpy}" mesh_path="${mesh_path}" scale_xyz="${scale_xyz}">
-            <extra_collision/>
-            <seperate_collider><mesh filename="${mesh_path}" scale="${scale_xyz}"/></seperate_collider>
             <extra_visual/>
             <extra_settings/>
         </xacro:link_creator_foundation>
     </xacro:macro>
-    <xacro:macro name="link_creator_i_foundation" params="link_name pose_xyz pose_rpy mesh_path scale_xyz center_mass_xyz:='0 0 0' mass ixx ixy ixz iyy iyz izz **extra_collision **seperate_collider **extra_visual **extra_settings">
+    <xacro:macro name="link_creator_i_foundation" params="link_name pose_xyz pose_rpy mesh_path scale_xyz seperate_collider_xyzrpy:='100000000 0 0 0 0 0' center_mass_xyz:='0 0 0' mass ixx ixy ixz iyy iyz izz **extra_collision **seperate_collider **extra_visual **extra_settings">
         <xacro:link_creator_foundation link_name="${link_name}" pose_xyz="${pose_xyz}" pose_rpy="${pose_rpy}" mesh_path="${mesh_path}" scale_xyz="${scale_xyz}">
-            <extra_collision><xacro:insert_block name="extra_collision"/></extra_collision>
-            <seperate_collider><xacro:insert_block name="seperate_collider"/></seperate_collider>
             <extra_visual><xacro:insert_block name="extra_visual"/></extra_visual>
             <extra_settings>
+                <collision>
+                    <geometry>
+                        <xacro:insert_block name="seperate_collider"/>
+                    </geometry>
+                    <xacro:if value="${seperate_collider_xyzrpy == '100000000 0 0 0 0 0'}">
+                        <origin xyz="${pose_xyz}" rpy="${pose_rpy}"/>
+                    </xacro:if>
+                    <xacro:unless value="${seperate_collider_xyzrpy == '100000000 0 0 0 0 0'}">
+                        <xacro:property name="seperate_collider_xyzrpy_list" value="${seperate_collider_xyzrpy.split(' ')}" />
+                        <origin xyz="${seperate_collider_xyzrpy_list[0]} ${seperate_collider_xyzrpy_list[1]} ${seperate_collider_xyzrpy_list[2]}" rpy="${seperate_collider_xyzrpy_list[3]} ${seperate_collider_xyzrpy_list[4]} ${seperate_collider_xyzrpy_list[5]}"/>
+                    </xacro:unless>
+                    <xacro:insert_block name="extra_collision"/>
+                </collision>
                 <inertial>
                     <origin xyz="${center_mass_xyz}" rpy="0 0 0"/>
@@ -151,6 +150,6 @@
         </xacro:link_creator_foundation>
     </xacro:macro>
-    <xacro:macro name="link_creator_i" params="link_name pose_xyz pose_rpy mesh_path scale_xyz center_mass_xyz:='0 0 0' mass ixx ixy ixz iyy iyz izz">
-        <xacro:link_creator_i_foundation link_name="${link_name}" pose_xyz="${pose_xyz}" pose_rpy="${pose_rpy}" mesh_path="${mesh_path}" scale_xyz="${scale_xyz}" center_mass_xyz="${center_mass_xyz}" mass="${mass}" ixx="${ixx}" ixy="${ixy}" ixz="${ixz}" iyy="${iyy}" iyz="${iyz}" izz="${izz}">
+    <xacro:macro name="link_creator_i" params="link_name pose_xyz pose_rpy mesh_path scale_xyz seperate_collider_xyzrpy:='100000000 0 0 0 0 0' center_mass_xyz:='0 0 0' mass ixx ixy ixz iyy iyz izz">
+        <xacro:link_creator_i_foundation link_name="${link_name}" pose_xyz="${pose_xyz}" pose_rpy="${pose_rpy}" mesh_path="${mesh_path}" scale_xyz="${scale_xyz}" seperate_collider_xyzrpy="${seperate_collider_xyzrpy}" center_mass_xyz="${center_mass_xyz}" mass="${mass}" ixx="${ixx}" ixy="${ixy}" ixz="${ixz}" iyy="${iyy}" iyz="${iyz}" izz="${izz}">
             <extra_collision/>
             <seperate_collider><mesh filename="${mesh_path}" scale="${scale_xyz}"/></seperate_collider>
@@ -159,6 +158,6 @@
         </xacro:link_creator_i_foundation>
     </xacro:macro>
-    <xacro:macro name="prop_link_creator" params="link_name pose_xyz pose_rpy mesh_path scale_xyz cyliner_r:='0.25' cylinder_l='0.01' mass ixx ixy ixz iyy iyz izz">
-        <xacro:link_creator_i_foundation link_name="${link_name}" pose_xyz="${pose_xyz}" pose_rpy="${pose_rpy}" mesh_path="${mesh_path}" scale_xyz="${scale_xyz}" mass="${mass}"  ixx="${ixx}" ixy="${ixy}" ixz="${ixz}" iyy="${iyy}" iyz="${iyz}" izz="${izz}">
+    <xacro:macro name="prop_link_creator" params="link_name pose_xyz pose_rpy mesh_path scale_xyz cyliner_r:='0.25' cylinder_l='0.01' seperate_collider_xyzrpy:='100000000 0 0 0 0 0' center_mass_xyz:='0 0 0' mass ixx ixy ixz iyy iyz izz">
+        <xacro:link_creator_i_foundation link_name="${link_name}" pose_xyz="${pose_xyz}" pose_rpy="${pose_rpy}" mesh_path="${mesh_path}" scale_xyz="${scale_xyz}" seperate_collider_xyzrpy="${seperate_collider_xyzrpy}" center_mass_xyz="${center_mass_xyz}" mass="${mass}"  ixx="${ixx}" ixy="${ixy}" ixz="${ixz}" iyy="${iyy}" iyz="${iyz}" izz="${izz}">
             <extra_collision>
                 <surface>

Commit message: not working-imu not stable...

File: models/copterPIX/robot.urdf.xacro (robot description, xacro)
@@ -23,5 +23,5 @@
   <xacro:property name="iyz" value="${0 * s}"/>
   <xacro:property name="izz" value="${1.6 * s}"/> -->
-  <xacro:property name="mass" value="4.5" />
+  <xacro:property name="mass" value="4" />
   <xacro:property name="s" value="2"/>
   <xacro:property name="ixx" value="${0.5 * s}"/>

File: xacros/macro.xacro (robot description, xacro)
@@ -30,5 +30,5 @@
         </gazebo>
         <xacro:prop_link_creator link_name="${prop_link}" pose_xyz="0 0 0.03" pose_rpy="0 -0 0" mesh_path="${prop_mesh}" scale_xyz="${prop_size_multiplier} ${prop_size_multiplier} ${prop_size_multiplier}" mass="${rmass}" ixx="${rixx}" ixy="${rixy}" ixz="${rixz}" iyy="${riyy}" iyz="${riyz}" izz="${rizz}"/>
-        <xacro:property name="cp" value="0.13"/>
+        <xacro:property name="cp" value="0.07"/>
         <xacro:property name="cp_negative" value="${-1 * cp}"/>
         <xacro:property name="area" value="0.002"/> <!--used to be 0.002-->

Commit message: finally working!

File: models/copterPIX/robot.urdf.xacro (robot description, xacro)
@@ -7,5 +7,5 @@
   <xacro:property name="prop_cw_mesh" value="$(find drone)/STLs/iris_prop_cw.dae"/>
   <xacro:property name="prop_ccw_mesh" value="$(find drone)/STLs/iris_prop_ccw.dae"/>
-  <xacro:property name="g_mms_to_kg_ms" value="1000000000"/>
+  <!-- <xacro:property name="g_mms_to_kg_ms" value="1000000000"/> -->
   <!-- <xacro:property name="mass" value="26.0" />
   <xacro:property name="ixx" value="${373162267137.9 / g_mms_to_kg_ms}"/>
@@ -24,11 +24,11 @@
   <xacro:property name="izz" value="${1.6 * s}"/> -->
   <xacro:property name="mass" value="4" />
-  <xacro:property name="s" value="2"/>
-  <xacro:property name="ixx" value="${0.5 * s}"/>
+  <xacro:property name="s" value="1"/>
+  <xacro:property name="ixx" value="${0.08 * s}"/>
   <xacro:property name="ixy" value="${0 * s}"/>
   <xacro:property name="ixz" value="${0 * s}"/>
-  <xacro:property name="iyy" value="${0.5 * s}"/>
+  <xacro:property name="iyy" value="${0.08 * s}"/>
   <xacro:property name="iyz" value="${0 * s}"/>
-  <xacro:property name="izz" value="${0.75 * s}"/>
+  <xacro:property name="izz" value="${0.1 * s}"/>
   <xacro:link_creator_i_foundation link_name="base_link" pose_xyz="0 0 0" pose_rpy="0 0 0" mesh_path="${hex_mesh}" scale_xyz="0.4 0.4 0.04" seperate_collider_xyzrpy="0 0 -0.3 0 0 0" center_mass_xyz="0 0 -0.5" mass="${mass}" ixx="${ixx}" ixy="${ixy}" ixz="${ixz}" iyy="${iyy}" iyz="${iyz}" izz="${izz}">
     <extra_collision>
@@ -79,4 +79,9 @@
   <!-- Define the drone arms using the macro -->
   <xacro:property name="deg_to_rad" value="0.0174533" />
+  <xacro:property name="dfc" value = "0.175" />
+  <xacro:property name="dfc" value = "0.175" />
+  <xacro:property name="leng" value="0.56"/>
+  <xacro:property name="dia" value="0.025" />
+  <xacro:property name="aia" value="0.0" />
   <!-- <xacro:drone_arm num="0" parent_link="base_link" dis_from_center="0.175" length="0.56" diameter="0.025" arm_incline_angle="${4 * deg_to_rad}" arm_mesh="${hex_mesh}" prop_mesh="${prop_cw_mesh}" prop_size_multiplier="2.04" amass="0.2" aixx="0" aixy="0" aixz="0" aiyy="0" aiyz="0" aizz="0" rmass="0.2" rixx="0.000312" rixy="0" rixz="0" riyy="0.0053345" riyz="0" rizz="0.005363328" angle="${0}"/>
   <xacro:drone_arm num="1" parent_link="base_link" dis_from_center="0.175" length="0.56" diameter="0.025" arm_incline_angle="${4 * deg_to_rad}" arm_mesh="${hex_mesh}" prop_mesh="${prop_ccw_mesh}" prop_size_multiplier="2.04" amass="0.2" aixx="0" aixy="0" aixz="0" aiyy="0" aiyz="0" aizz="0" rmass="0.2" rixx="0.000312" rixy="0" rixz="0" riyy="0.0053345" riyz="0" rizz="0.005363328" angle="${180 * deg_to_rad}"/>
@@ -91,48 +96,11 @@
   <xacro:drone_arm num="4" parent_link="base_link" dis_from_center="0.175" length="0.56" diameter="0.025" arm_incline_angle="${4 * deg_to_rad}" arm_mesh="${hex_mesh}" prop_mesh="${prop_ccw_mesh}" cw="false" prop_size_multiplier="2.04" rmass="0.2" rixx="0.000312" rixy="0" rixz="0" riyy="0.0053345" riyz="0" rizz="0.005363328" angle="${60 * deg_to_rad}"/>
   <xacro:drone_arm num="5" parent_link="base_link" dis_from_center="0.175" length="0.56" diameter="0.025" arm_incline_angle="${4 * deg_to_rad}" arm_mesh="${hex_mesh}" prop_mesh="${prop_cw_mesh}" cw="true" prop_size_multiplier="2.04" rmass="0.2" rixx="0.000312" rixy="0" rixz="0" riyy="0.0053345" riyz="0" rizz="0.005363328" angle="${240 * deg_to_rad}"/> -->
-  <xacro:drone_arm num="0" parent_link="base_link" dis_from_center="0.175" length="0.56" diameter="0.025" arm_incline_angle="${6 * deg_to_rad}" arm_mesh="${hex_mesh}" prop_mesh="${prop_cw_mesh}"  cw="true"  prop_size_multiplier="2.04" rmass="0.025" rixx="0.00000975" rixy="0" rixz="0" riyy="0.000166704" riyz="0" rizz="0.000167604" angle="${0 * deg_to_rad}"/>
-  <xacro:drone_arm num="1" parent_link="base_link" dis_from_center="0.175" length="0.56" diameter="0.025" arm_incline_angle="${6 * deg_to_rad}" arm_mesh="${hex_mesh}" prop_mesh="${prop_ccw_mesh}" cw="false" prop_size_multiplier="2.04" rmass="0.025" rixx="0.00000975" rixy="0" rixz="0" riyy="0.000166704" riyz="0" rizz="0.000167604" angle="${180 * deg_to_rad}"/>
-  <xacro:drone_arm num="2" parent_link="base_link" dis_from_center="0.175" length="0.56" diameter="0.025" arm_incline_angle="${6 * deg_to_rad}" arm_mesh="${hex_mesh}" prop_mesh="${prop_cw_mesh}"  cw="true"  prop_size_multiplier="2.04" rmass="0.025" rixx="0.00000975" rixy="0" rixz="0" riyy="0.000166704" riyz="0" rizz="0.000167604" angle="${120 * deg_to_rad}"/>
-  <xacro:drone_arm num="3" parent_link="base_link" dis_from_center="0.175" length="0.56" diameter="0.025" arm_incline_angle="${6 * deg_to_rad}" arm_mesh="${hex_mesh}" prop_mesh="${prop_ccw_mesh}" cw="false" prop_size_multiplier="2.04" rmass="0.025" rixx="0.00000975" rixy="0" rixz="0" riyy="0.000166704" riyz="0" rizz="0.000167604" angle="${300 * deg_to_rad}"/>
-  <xacro:drone_arm num="4" parent_link="base_link" dis_from_center="0.175" length="0.56" diameter="0.025" arm_incline_angle="${6 * deg_to_rad}" arm_mesh="${hex_mesh}" prop_mesh="${prop_ccw_mesh}" cw="false" prop_size_multiplier="2.04" rmass="0.025" rixx="0.00000975" rixy="0" rixz="0" riyy="0.000166704" riyz="0" rizz="0.000167604" angle="${60 * deg_to_rad}"/>
-  <xacro:drone_arm num="5" parent_link="base_link" dis_from_center="0.175" length="0.56" diameter="0.025" arm_incline_angle="${6 * deg_to_rad}" arm_mesh="${hex_mesh}" prop_mesh="${prop_cw_mesh}"  cw="true"  prop_size_multiplier="2.04" rmass="0.025" rixx="0.00000975" rixy="0" rixz="0" riyy="0.000166704" riyz="0" rizz="0.000167604" angle="${240 * deg_to_rad}"/>
+  <xacro:drone_arm num="0" parent_link="base_link" dis_from_center="${dfc}" length="${leng}" diameter="${dia}" arm_incline_angle="${aia * deg_to_rad}" arm_mesh="${hex_mesh}" prop_mesh="${prop_cw_mesh}"  cw="true"  prop_size_multiplier="2.04" rmass="0.025" rixx="0.00000975" rixy="0" rixz="0" riyy="0.000166704" riyz="0" rizz="0.000167604" angle="${0 * deg_to_rad}"/>
+  <xacro:drone_arm num="1" parent_link="base_link" dis_from_center="${dfc}" length="${leng}" diameter="${dia}" arm_incline_angle="${aia * deg_to_rad}" arm_mesh="${hex_mesh}" prop_mesh="${prop_ccw_mesh}" cw="false" prop_size_multiplier="2.04" rmass="0.025" rixx="0.00000975" rixy="0" rixz="0" riyy="0.000166704" riyz="0" rizz="0.000167604" angle="${180 * deg_to_rad}"/>
+  <xacro:drone_arm num="2" parent_link="base_link" dis_from_center="${dfc}" length="${leng}" diameter="${dia}" arm_incline_angle="${aia * deg_to_rad}" arm_mesh="${hex_mesh}" prop_mesh="${prop_cw_mesh}"  cw="true"  prop_size_multiplier="2.04" rmass="0.025" rixx="0.00000975" rixy="0" rixz="0" riyy="0.000166704" riyz="0" rizz="0.000167604" angle="${120 * deg_to_rad}"/>
+  <xacro:drone_arm num="3" parent_link="base_link" dis_from_center="${dfc}" length="${leng}" diameter="${dia}" arm_incline_angle="${aia * deg_to_rad}" arm_mesh="${hex_mesh}" prop_mesh="${prop_ccw_mesh}" cw="false" prop_size_multiplier="2.04" rmass="0.025" rixx="0.00000975" rixy="0" rixz="0" riyy="0.000166704" riyz="0" rizz="0.000167604" angle="${300 * deg_to_rad}"/>
+  <xacro:drone_arm num="4" parent_link="base_link" dis_from_center="${dfc}" length="${leng}" diameter="${dia}" arm_incline_angle="${aia * deg_to_rad}" arm_mesh="${hex_mesh}" prop_mesh="${prop_ccw_mesh}" cw="false" prop_size_multiplier="2.04" rmass="0.025" rixx="0.00000975" rixy="0" rixz="0" riyy="0.000166704" riyz="0" rizz="0.000167604" angle="${60 * deg_to_rad}"/>
+  <xacro:drone_arm num="5" parent_link="base_link" dis_from_center="${dfc}" length="${leng}" diameter="${dia}" arm_incline_angle="${aia * deg_to_rad}" arm_mesh="${hex_mesh}" prop_mesh="${prop_cw_mesh}"  cw="true"  prop_size_multiplier="2.04" rmass="0.025" rixx="0.00000975" rixy="0" rixz="0" riyy="0.000166704" riyz="0" rizz="0.000167604" angle="${240 * deg_to_rad}"/>
   <gazebo>
-    <!-- <link name='odometry_sensorgt_link'>
-      <pose>0 0 0 0 -0 0</pose>
-      <inertial>
-        <pose>0 0 0 0 -0 0</pose>
-        <mass>0.15</mass>
-        <inertia>
-          <ixx>0.0001</ixx>
-          <ixy>0</ixy>
-          <ixz>0</ixz>
-          <iyy>0.0002</iyy>
-          <iyz>0</iyz>
-          <izz>0.0002</izz>
-        </inertia>
-      </inertial>
-    </link>
-    <joint name='odometry_sensorgt_joint' type='revolute'>
-      <child>odometry_sensorgt_link</child>
-      <parent>base_link</parent>
-      <axis>
-        <xyz>0 0 1</xyz>
-        <limit>
-          <lower>0</lower>
-          <upper>0</upper>
-          <effort>0</effort>
-          <velocity>0</velocity>
-        </limit>
-        <dynamics>
-          <damping>1.0</damping>
-        </dynamics>
-        <use_parent_model_frame>1</use_parent_model_frame>
-      </axis>
-      <physics>
-        <ode>
-          <implicit_spring_damper>1</implicit_spring_damper>
-        </ode>
-      </physics>
-    </joint> -->
     <link name='imu_link'>
       <inertial>
@@ -154,5 +122,5 @@
       </sensor>
     </link>
-    <joint name='imu_joint' type='fixed'>
+    <joint name='imu_joint' type='revolute'>
       <parent>base_link</parent>
       <child>imu_link</child>

File: xacros/macro.xacro (robot description, xacro)
@@ -1,5 +1,5 @@
 <?xml version="1.0"?>
 <robot xmlns:xacro="http://www.ros.org/wiki/xacro">
-    <xacro:macro name="drone_arm" params="num parent_link dis_from_center length diameter arm_incline_angle arm_mesh prop_mesh cw prop_size_multiplier amass:='0.001' aixx:='0' aixy:='0' aixz:='0' aiyy:='0' aiyz:='0' aizz:='0' rmass rixx rixy rixz riyy riyz rizz angle">
+    <xacro:macro name="drone_arm" params="num parent_link dis_from_center length diameter arm_incline_angle arm_mesh prop_mesh cw prop_size_multiplier amass:='0.01' aixx:='0.0001' aixy:='0' aixz:='0' aiyy:='0.0001' aiyz:='0' aizz:='0.0001' rmass rixx rixy rixz riyy riyz rizz angle">
         <xacro:property name="base_arm_joint" value="base_arm_joint_${num}" />
         <xacro:property name="arm_link" value="arm_link_${num}" />
@@ -11,5 +11,5 @@
             <parent link="${parent_link}"/>
             <child link="${arm_link}"/>
-            <origin xyz="0 0 0" rpy="0 0 ${angle}"/>
+            <origin xyz="0 0 0" rpy="0 0 ${angle + pi}"/>
         </joint>
         <xacro:link_creator_i link_name="${arm_link}" pose_xyz="0 ${cos(arm_incline_angle) * (length / 2.0) + dis_from_center} ${sin(arm_incline_angle) * (length / 2.0)}" pose_rpy="${arm_incline_angle + 1.57079632679} 0 0" mesh_path="${arm_mesh}" scale_xyz="${diameter} ${diameter} ${length}" mass="${amass}" ixx="${aixx}" ixy="${aixy}" ixz="${aixz}" iyy="${aiyy}" iyz="${aiyz}" izz="${aizz}"/>
@@ -30,5 +30,6 @@
         </gazebo>
         <xacro:prop_link_creator link_name="${prop_link}" pose_xyz="0 0 0.03" pose_rpy="0 -0 0" mesh_path="${prop_mesh}" scale_xyz="${prop_size_multiplier} ${prop_size_multiplier} ${prop_size_multiplier}" mass="${rmass}" ixx="${rixx}" ixy="${rixy}" ixz="${rixz}" iyy="${riyy}" iyz="${riyz}" izz="${rizz}"/>
-        <xacro:property name="cp" value="0.07"/>
+        <xacro:property name="cla" value="4.5"/>
+        <xacro:property name="cp" value="0.084"/>
         <xacro:property name="cp_negative" value="${-1 * cp}"/>
         <xacro:property name="area" value="0.002"/> <!--used to be 0.002-->
@@ -38,5 +39,5 @@
                     <a0>0.3</a0>
                     <alpha_stall>1.4</alpha_stall>
-                    <cla>4.2500</cla>
+                    <cla>${cla}</cla>
                     <cda>0.10</cda>
                     <cma>0.00</cma>
@@ -54,5 +55,5 @@
                     <a0>0.3</a0>
                     <alpha_stall>1.4</alpha_stall>
-                    <cla>4.2500</cla>
+                    <cla>${cla}</cla>
                     <cda>0.10</cda>
                     <cma>0.00</cma>
@@ -74,5 +75,5 @@
                     <a0>0.3</a0>
                     <alpha_stall>1.4</alpha_stall>
-                    <cla>4.2500</cla>
+                    <cla>${cla}</cla>
                     <cda>0.10</cda>
                     <cma>0.00</cma>
@@ -90,5 +91,5 @@
                     <a0>0.3</a0>
                     <alpha_stall>1.4</alpha_stall>
-                    <cla>4.2500</cla>
+                    <cla>${cla}</cla>
                     <cda>0.10</cda>
                     <cma>0.00</cma>
@@ -176,11 +177,11 @@
             <extra_settings>
                 <velocity_decay/>
-                <gazebo reference="${link_name}">
-                    <material>Gazebo/Red</material>
-                    <gravity>1</gravity>
-                    <self_collide>0</self_collide>
-                </gazebo>
             </extra_settings>
         </xacro:link_creator_i_foundation>
+        <gazebo reference="${link_name}">
+            <material>Gazebo/Red</material>
+            <gravity>1</gravity>
+            <self_collide>0</self_collide>
+        </gazebo>
     </xacro:macro>
 </robot>
