Commit message: understood why setting up inertia for the small part didn't work. its cuz its too small when automatically calculated so for extremely small parts, it is neccessary to set it your self!

File: models/copterPIX/robot.urdf.xacro (robot description, xacro)
@@ -25,25 +25,4 @@
   <!-- <xacro:link_creator_i link_name="base_link" pose_xyz="0 0 0" pose_rpy="0 0 0" mesh_path="${hex_mesh}" scale_xyz="0.4 0.4 0.04" center_mass_xyz="${center_of_mass}" mass="${mass}" ixx="${ixx}" ixy="${ixy}" ixz="${ixz}" iyy="${iyy}" iyz="${iyz}" izz="${izz}"/> -->
   <xacro:link_creator_i link_name="base_link" pose_xyz="0 0 0" pose_rpy="0 0 0" mesh_path="${hex_mesh}" scale_xyz="0.4 0.4 0.04" center_mass_xyz="${center_of_mass}" mass="${mass}"/>
-  <!-- <xacro:link_creator_i_foundation link_name="base_link" pose_xyz="0 0 0" pose_rpy="0 0 0" mesh_path="${hex_mesh}" scale_xyz="0.4 0.4 0.04" seperate_collider_xyzrpy="0 0 -0.3 0 0 0" center_mass_xyz="0 0 -0.5" mass="${mass}" ixx="${ixx}" ixy="${ixy}" ixz="${ixz}" iyy="${iyy}" iyz="${iyz}" izz="${izz}">
-    <extra_collision>
-      <surface>
-        <contact>
-          <ode>
-            <max_vel>100.0</max_vel>
-            <min_depth>0.001</min_depth>
-          </ode>
-        </contact>
-        <friction>
-          <ode>
-            <mu>100000.0</mu>
-            <mu2>100000.0</mu2>
-          </ode>
-        </friction>
-      </surface>
-    </extra_collision>
-    <seperate_collider><cylinder radius="0.45" length="0.62"/></seperate_collider>
-    <extra_visual/>
-    <extra_settings/>
-  </xacro:link_creator_i_foundation> -->
   <!-- <xacro:link_creator link_name="base_link" pose_xyz="0 0 0" pose_rpy="0 0 0" mesh_path="${hex_mesh}" scale_xyz="0.4 0.4 0.04"/> -->
   <joint name="leg_0_link_joint" type="fixed">
@@ -193,5 +172,5 @@
     </physics>
   </gazebo>
-  <xacro:link_creator_i link_name="fire_trigger_servo_link" mesh_path="Box" pose_xyz="0 0 0" pose_rpy="0 0 0" scale_xyz="0.04 0.009 0.009" mass="0.001"/>
+  <xacro:link_creator_i link_name="fire_trigger_servo_link" mesh_path="Box" pose_xyz="0 0 0" pose_rpy="0 0 0" scale_xyz="0.04 0.009 0.009" mass="0.05" iner="0.001 0 0 0.001 0 0.001"/>  <!--it is neccessary to specify the value here because the inertia becomes too small if done automatically for the following link with such small mass and size!-->
   <gazebo reference="fire_trigger_servo_link">
     <material>Gazebo/Red</material>

File: xacros/macro.xacro (robot description, xacro)
@@ -196,18 +196,5 @@
                 <xacro:if value="${iner == '100000000 0 0 0 0 0'}">
                     <xacro:property name="scale_xyz_list" value="${scale_xyz.split(' ')}" />
-                    <!-- <xacro:inertial_box mass="${mass}" x="${float(scale_xyz_list[0])}" y="${float(scale_xyz_list[1])}" z="${float(scale_xyz_list[2])}" xyz="${center_mass_xyz}" rpy="0 0 0"/> -->
-                    <inertial>
-                        <mass value="${mass}" />
-                        <!-- <inertia ixx="0.001" ixy="0" ixz="0" iyy="0.001" iyz="0" izz="0.001"/> -->
-                        <!-- <inertia ixx="${float(mass) * (float(scale_xyz_list[1]) * float(scale_xyz_list[1]) + float(scale_xyz_list[2]) * float(scale_xyz_list[2])) / 12}" ixy="0" ixz="0" iyy="${float(mass) * (float(scale_xyz_list[0])*float(scale_xyz_list[0])+float(scale_xyz_list[2])*float(scale_xyz_list[2])) / 12}" iyz="0" izz="${float(mass) * (float(scale_xyz_list[1]) * float(scale_xyz_list[1]) + float(scale_xyz_list[0]) * float(scale_xyz_list[0])) / 12}" /> -->
-                        <origin xyz="${center_mass_xyz}" rpy="0 0 0"/>
-                        <!-- <xacro:property name="scale_x" value="${float(scale_xyz_list[0])}"/>
-                        <xacro:property name="scale_y" value="${float(scale_xyz_list[1])}"/>
-                        <xacro:property name="scale_z" value="${float(scale_xyz_list[2])}"/>
-                        <xacro:property name="ixx" value="${mass * (scale_y * scale_y + scale_z * scale_z) / 12}"/>
-                        <xacro:property name="iyy" value="${mass * (scale_x * scale_x + scale_z * scale_z) / 12}"/>
-                        <xacro:property name="izz" value="${mass * (scale_x * scale_x + scale_y * scale_y) / 12}"/>
-                        <inertia ixx="${ixx}" ixy="0" ixz="0" iyy="${iyy}" iyz="0" izz="${izz}"/> --> not working kusemek for some reason the line 238 in robot.urdf.xacro file of copterPIX doesn't allow defualt value of inertia cuz this part where we define inertia is broken cuz its a revolute joint...?????why???
-                    </inertial>
+                    <xacro:inertial_box mass="${mass}" x="${float(scale_xyz_list[0])}" y="${float(scale_xyz_list[1])}" z="${float(scale_xyz_list[2])}" xyz="${center_mass_xyz}" rpy="0 0 0"/>
                 </xacro:if>
                 <xacro:if value="${iner != '100000000 0 0 0 0 0'}">

Commit message: everything working, but ros2 node for apply force still not done.(don't know how:(  test for applying force is the folder with all the shits, you can even delete it cuz no dependencies for it

File: models/copterPIX/robot.urdf.xacro (robot description, xacro)
@@ -17,18 +17,9 @@
   -->
   <xacro:property name="center_of_mass" value="0 0 0"/>
-  <!-- <xacro:property name="ixx" value="${10000000000 / g_mms_to_kg_ms}"/>
-  <xacro:property name="ixy" value="${0 / g_mms_to_kg_ms}"/>
-  <xacro:property name="ixz" value="${0 / g_mms_to_kg_ms}"/>
-  <xacro:property name="iyy" value="${10000000000 / g_mms_to_kg_ms}"/>
-  <xacro:property name="iyz" value="${0 / g_mms_to_kg_ms}"/>
-  <xacro:property name="izz" value="${16000000000 / g_mms_to_kg_ms}"/> -->
-  <!-- <xacro:link_creator_i link_name="base_link" pose_xyz="0 0 0" pose_rpy="0 0 0" mesh_path="${hex_mesh}" scale_xyz="0.4 0.4 0.04" center_mass_xyz="${center_of_mass}" mass="${mass}" ixx="${ixx}" ixy="${ixy}" ixz="${ixz}" iyy="${iyy}" iyz="${iyz}" izz="${izz}"/> -->
   <xacro:link_creator_i link_name="base_link" pose_xyz="0 0 0" pose_rpy="0 0 0" mesh_path="${hex_mesh}" scale_xyz="0.4 0.4 0.04" center_mass_xyz="${center_of_mass}" mass="${mass}"/>
-  <!-- <xacro:link_creator link_name="base_link" pose_xyz="0 0 0" pose_rpy="0 0 0" mesh_path="${hex_mesh}" scale_xyz="0.4 0.4 0.04"/> -->
   <joint name="leg_0_link_joint" type="fixed">
     <parent link="base_link"/>
     <child link="leg_0_link"/>
   </joint>
-  <!-- <xacro:link_creator_i link_name="leg_0_link" pose_xyz="0 0.198 -0.305" pose_rpy="0.305 0 0" mesh_path="${hex_mesh}" scale_xyz="0.024 0.024 0.61" mass="0.2" ixx="0.0" ixy="0.0" ixz="0.0" iyy="0.0" iyz="0.0" izz="0.0"/> -->
   <xacro:link_creator_i link_name="leg_0_link" pose_xyz="0 0.198 -0.305" pose_rpy="0.305 0 0" mesh_path="${hex_mesh}" scale_xyz="0.024 0.024 0.61" mass="0.5"/>
   <joint name="leg_1_link_joint" type="fixed">
@@ -36,5 +27,4 @@
     <child link="leg_1_link"/>
   </joint>
-  <!-- <xacro:link_creator_i link_name="leg_1_link" pose_xyz="0 -0.198 -0.305" pose_rpy="-0.305 0 0" mesh_path="${hex_mesh}" scale_xyz="0.024 0.024 0.61" mass="0.2" ixx="0.0" ixy="0.0" ixz="0.0" iyy="0.0" iyz="0.0" izz="0.0"/> -->
   <xacro:link_creator_i link_name="leg_1_link" pose_xyz="0 -0.198 -0.305" pose_rpy="-0.305 0 0" mesh_path="${hex_mesh}" scale_xyz="0.024 0.024 0.61" mass="0.5"/>
   <joint name="feet_0_link_joint" type="fixed">
@@ -42,5 +32,4 @@
     <child link="feet_0_link"/>
   </joint>
-  <!-- <xacro:link_creator_i link_name="feet_0_link" pose_xyz="0 0.29 -0.6" pose_rpy="0 1.57079633 0" mesh_path="${hex_mesh}" scale_xyz="0.024 0.024 0.58" mass="0.2" ixx="0.0" ixy="0.0" ixz="0.0" iyy="0.0" iyz="0.0" izz="0.0"/> -->
   <xacro:link_creator_i link_name="feet_0_link" pose_xyz="0 0.29 -0.6" pose_rpy="0 1.57079633 0" mesh_path="${hex_mesh}" scale_xyz="0.024 0.024 0.58" mass="0.5"/>
   <joint name="feet_1_link_joint" type="fixed">
@@ -48,5 +37,4 @@
     <child link="feet_1_link"/>
   </joint>
-  <!-- <xacro:link_creator_i link_name="feet_1_link" pose_xyz="0 -0.29 -0.6" pose_rpy="0 1.57079633 0" mesh_path="${hex_mesh}" scale_xyz="0.024 0.024 0.58" mass="0.2" ixx="0.0" ixy="0.0" ixz="0.0" iyy="0.0" iyz="0.0" izz="0.0"/> -->
   <xacro:link_creator_i link_name="feet_1_link" pose_xyz="0 -0.29 -0.6" pose_rpy="0 1.57079633 0" mesh_path="${hex_mesh}" scale_xyz="0.024 0.024 0.58" mass="0.5"/>
   <!-- Define the drone arms using the macro -->
@@ -71,59 +59,4 @@
   <xacro:drone_arm num="4" parent_link="base_link" dis_from_center="${dfc}" length="${leng}" diameter="${dia}" arm_incline_angle="${aia * deg_to_rad}" arm_mesh="${hex_mesh}" prop_mesh="${prop_ccw_mesh}" cw="false" prop_size_multiplier="${psm}" cylinder_d="${cylinder_d}" cylinder_l="${cylinder_l}" a_mass="${a_mass}"  cla="${cla}" cp="${cp}" area="${area}" r_mass="${r_mass}" r_iner="${r_iner}" angle="${60 * deg_to_rad}"/>
   <xacro:drone_arm num="5" parent_link="base_link" dis_from_center="${dfc}" length="${leng}" diameter="${dia}" arm_incline_angle="${aia * deg_to_rad}" arm_mesh="${hex_mesh}" prop_mesh="${prop_cw_mesh}"  cw="true"  prop_size_multiplier="${psm}" cylinder_d="${cylinder_d}" cylinder_l="${cylinder_l}" a_mass="${a_mass}"  cla="${cla}" cp="${cp}" area="${area}" r_mass="${r_mass}" r_iner="${r_iner}" angle="${240 * deg_to_rad}"/>
-  <!-- <gazebo>
-    <link name='imu_link'>
-      <inertial>
-        <pose>0 0 0 0 0 0</pose>
-        <mass>0.15</mass>
-        <inertia>
-          <ixx>0.00001</ixx>
-          <ixy>0</ixy>
-          <ixz>0</ixz>
-          <iyy>0.00002</iyy>
-          <iyz>0</iyz>
-          <izz>0.00002</izz>
-        </inertia>
-      </inertial> -->
-      <!-- <visual name='imu_vis'>
-        <geometry>
-          <box>
-            <size>0.1 0.1 0.1</size>
-          </box>
-        </geometry>
-        <material>
-          <script>
-            <name>Gazebo/DarkGrey</name>
-          </script>
-        </material>
-      </visual> -->
-      <!-- <sensor name="imu_sensor" type="imu">
-        <pose>0 0 0 3.141593 0 0</pose>
-        <always_on>1</always_on>
-        <update_rate>1000.0</update_rate>
-      </sensor>
-    </link>
-    <joint name='imu_joint' type='revolute'>
-      <parent>base_link</parent>
-      <child>imu_link</child>
-      <axis>
-        <xyz>0 0 1</xyz>
-        <limit>
-          <lower>0</lower>
-          <upper>0</upper>
-          <effort>0</effort>
-          <velocity>0</velocity>
-        </limit>
-        <dynamics>
-          <damping>1.0</damping>
-        </dynamics>
-        <use_parent_model_frame>1</use_parent_model_frame>
-      </axis>
-      <physics>
-        <ode>
-          <implicit_spring_damper>1</implicit_spring_damper>
-        </ode>
-      </physics>
-    </joint>
-  </gazebo> -->
   <joint name="imu_joint" type="revolute">
     <parent link="base_link"/>

File: xacros/macro.xacro (robot description, xacro)
@@ -2,5 +2,4 @@
 <robot xmlns:xacro="http://www.ros.org/wiki/xacro">
     <xacro:include filename="inertial_macros.xacro"/>
-    <!-- <xacro:macro name="drone_arm" params="num parent_link dis_from_center length diameter arm_incline_angle arm_mesh prop_mesh cw prop_size_multiplier cylinder_r cylinder_l amass aixx:='0.0001' aixy:='0' aixz:='0' aiyy:='0.0001' aiyz:='0' aizz:='0.0001' cla cp area rmass rixx rixy rixz riyy riyz rizz angle">  -->
     <xacro:macro name="drone_arm" params="num parent_link dis_from_center length diameter arm_incline_angle arm_mesh prop_mesh cw prop_size_multiplier cylinder_d cylinder_l a_mass a_iner:='100000000 0 0 0 0 0' cla cp area r_mass r_iner angle">
         <xacro:property name="base_arm_joint" value="base_arm_joint_${num}" />
@@ -15,5 +14,4 @@
             <origin xyz="0 0 0" rpy="0 0 ${angle + pi}"/>
         </joint>
-        <!-- <xacro:link_creator_i link_name="${arm_link}" pose_xyz="0 ${cos(arm_incline_angle) * (length / 2.0) + dis_from_center} ${sin(arm_incline_angle) * (length / 2.0)}" pose_rpy="${arm_incline_angle + 1.57079632679} 0 0" mesh_path="${arm_mesh}" scale_xyz="${diameter} ${diameter} ${length}" mass="${amass}" ixx="${aixx}" ixy="${aixy}" ixz="${aixz}" iyy="${aiyy}" iyz="${aiyz}" izz="${aizz}"/> -->
         <xacro:link_creator_i link_name="${arm_link}" pose_xyz="0 ${cos(arm_incline_angle) * (length / 2.0) + dis_from_center} ${sin(arm_incline_angle) * (length / 2.0)}" pose_rpy="${arm_incline_angle + 1.57079632679} 0 0" mesh_path="${arm_mesh}" scale_xyz="${diameter} ${diameter} ${length}" mass="${a_mass}" iner="${a_iner}"/>
         <joint name="${rotor_joint}" type="continuous">
