Commit message: fixed the copterPIX and now its fully working! also made iris but its not working

File: models/copterPIX/robot.urdf.xacro (robot description, xacro)
@@ -1,11 +1,9 @@
 <?xml version="1.0" ?>
 <robot name="copterPIX" xmlns:xacro="http://www.ros.org/wiki/xacro">
-  <xacro:include filename="$(find drone)/xacros/macro.xacro"/>
   <xacro:include filename="$(find drone)/xacros/drone_maker.xacro"/>
   <xacro:include filename="ardupilot_plugin.xacro"/>
+  <xacro:property name="hex_mesh" value="$(find drone)/meshes/hexagonal_prism_height_1_outer_diameter_1.stl"/>
   <xacro:property name="prop_cw_mesh" value="$(find drone)/meshes/iris_prop_cw.dae"/>
   <xacro:property name="prop_ccw_mesh" value="$(find drone)/meshes/iris_prop_ccw.dae"/>
-  <xacro:property name="prop_meshs" value="${prop_cw_mesh} ${prop_ccw_mesh} ${prop_cw_mesh} ${prop_ccw_mesh} ${prop_ccw_mesh} ${prop_cw_mesh}"/>
-  <xacro:property name="hex_mesh" value="$(find drone)/meshes/hexagonal_prism_height_1_outer_diameter_1.stl"/>
 <!--
   <xacro:property name="ixx" value="${373162267137.9 / g_mms_to_kg_ms}"/>  these values are not valid, they are stupid wrong
@@ -21,10 +19,10 @@
   <xacro:property name="base_pose_rpy" value="0 0 0"/>
   <xacro:property name="base_scale_xyz" value="0.4 0.4 0.04"/>
-  <xacro:property name="base_center_of_mass" value=""/>
+  <xacro:property name="base_center_of_mass" value="0 0 0"/>
   <xacro:property name="base_mass" value="19" />
   <xacro:property name="base_iner" value="None"/>
   <xacro:property name="number_of_arms" value="6"/>
   <xacro:property name="arm_angles" value="0 180 120 300 60 240"/>
-  <xacro:property name="cws" value="true false true false false true"/>
+  <xacro:property name="cws" value="1 0 1 0 0 1"/>  <!-- 1: true 0: false -->
   <xacro:property name="prop_meshs" value="${prop_cw_mesh} ${prop_ccw_mesh} ${prop_cw_mesh} ${prop_ccw_mesh} ${prop_ccw_mesh} ${prop_cw_mesh}"/>
   <xacro:property name="dis_from_center" value="0.175"/>
@@ -49,48 +47,47 @@
                      arm_incline_angle="${arm_incline_angle}" arm_mesh="${arm_mesh}" prop_size_multiplier="${prop_size_multiplier}"
                      cylinder_d="${cylinder_d}" cylinder_l="${cylinder_l}" a_mass="${a_mass}" a_iner="${a_iner}"
-                     cla="${cla}" area="${area}" r_mass="${r_mass}"  r_iner="${r_iner}">
-    <extra_settings>
-      <joint name="leg_0_link_joint" type="fixed">
-        <parent link="base_link"/>
-        <child link="leg_0_link"/>
-      </joint>
-      <xacro:link_creator_i link_name="leg_0_link" pose_xyz="0 0.198 -0.305" pose_rpy="0.305 0 0" mesh_path="${hex_mesh}" scale_xyz="0.024 0.024 0.61" mass="0.5"/>
-      <joint name="leg_1_link_joint" type="fixed">
-        <parent link="base_link"/>
-        <child link="leg_1_link"/>
-      </joint>
-      <xacro:link_creator_i link_name="leg_1_link" pose_xyz="0 -0.198 -0.305" pose_rpy="-0.305 0 0" mesh_path="${hex_mesh}" scale_xyz="0.024 0.024 0.61" mass="0.5"/>
-      <joint name="feet_0_link_joint" type="fixed">
-        <parent link="base_link"/>
-        <child link="feet_0_link"/>
-      </joint>
-      <xacro:link_creator_i link_name="feet_0_link" pose_xyz="0 0.29 -0.6" pose_rpy="0 1.57079633 0" mesh_path="${hex_mesh}" scale_xyz="0.024 0.024 0.58" mass="0.5"/>
-      <joint name="feet_1_link_joint" type="fixed">
-        <parent link="base_link"/>
-        <child link="feet_1_link"/>
-      </joint>
-      <xacro:link_creator_i link_name="feet_1_link" pose_xyz="0 -0.29 -0.6" pose_rpy="0 1.57079633 0" mesh_path="${hex_mesh}" scale_xyz="0.024 0.024 0.58" mass="0.5"/>
-      <joint name="fire_trigger_servo_joint" type="revolute">
-        <parent link="base_link"/>
-        <child link="fire_trigger_servo_link"/>
-        <origin xyz="0 0 -0.45" rpy="0 0 0"/>
-        <axis xyz="0 0 1"/>
-        <limit effort="10000" velocity="4" lower="${pi * -0.5}" upper="${pi * 0.5}"/>
-        <dynamics damping="0.1" friction="0"/>
-      </joint>
-      <gazebo reference="fire_trigger_servo_joint">
-        <physics>
-          <ode>
-            <implicit_spring_damper>1.0</implicit_spring_damper>
-          </ode>
-        </physics>
-      </gazebo>
-      <xacro:link_creator_i link_name="fire_trigger_servo_link" mesh_path="Box" pose_xyz="0 0 0" pose_rpy="0 0 0" scale_xyz="0.04 0.009 0.009" mass="0.05" iner="0.001 0 0 0.001 0 0.001"/>  <!--it is neccessary to specify the value here because the inertia becomes too small if done automatically for the following link with such small mass and size!-->
-      <gazebo reference="fire_trigger_servo_link">
-        <material>Gazebo/Red</material>
-        <self_collide>0</self_collide>
-      </gazebo>
-    </extra_settings>
+                     cla="${cla}" cp="${cp}" area="${area}" r_mass="${r_mass}"  r_iner="${r_iner}">
   </xacro:drone_maker>
+  <joint name="leg_0_link_joint" type="fixed">
+    <parent link="base_link"/>
+    <child link="leg_0_link"/>
+  </joint>
+  <xacro:link_creator_i link_name="leg_0_link" pose_xyz="0 0.198 -0.305" pose_rpy="0.305 0 0" mesh_path="${hex_mesh}" scale_xyz="0.024 0.024 0.61" mass="0.5"/>
+  <joint name="leg_1_link_joint" type="fixed">
+    <parent link="base_link"/>
+    <child link="leg_1_link"/>
+  </joint>
+  <xacro:link_creator_i link_name="leg_1_link" pose_xyz="0 -0.198 -0.305" pose_rpy="-0.305 0 0" mesh_path="${hex_mesh}" scale_xyz="0.024 0.024 0.61" mass="0.5"/>
+  <joint name="feet_0_link_joint" type="fixed">
+    <parent link="base_link"/>
+    <child link="feet_0_link"/>
+  </joint>
+  <xacro:link_creator_i link_name="feet_0_link" pose_xyz="0 0.29 -0.6" pose_rpy="0 1.57079633 0" mesh_path="${hex_mesh}" scale_xyz="0.024 0.024 0.58" mass="0.5"/>
+  <joint name="feet_1_link_joint" type="fixed">
+    <parent link="base_link"/>
+    <child link="feet_1_link"/>
+  </joint>
+  <xacro:link_creator_i link_name="feet_1_link" pose_xyz="0 -0.29 -0.6" pose_rpy="0 1.57079633 0" mesh_path="${hex_mesh}" scale_xyz="0.024 0.024 0.58" mass="0.5"/>
+  <joint name="fire_trigger_servo_joint" type="revolute">
+    <parent link="base_link"/>
+    <child link="fire_trigger_servo_link"/>
+    <origin xyz="0 0 -0.45" rpy="0 0 0"/>
+    <axis xyz="0 0 1"/>
+    <limit effort="10000" velocity="4" lower="${pi * -0.5}" upper="${pi * 0.5}"/>
+    <dynamics damping="0.1" friction="0"/>
+  </joint>
+  <gazebo reference="fire_trigger_servo_joint">
+    <physics>
+      <ode>
+        <implicit_spring_damper>1</implicit_spring_damper>
+      </ode>
+    </physics>
+  </gazebo>
+<!-- it is neccessary to specify the value here because the inertia becomes too small if done automatically for the following link with such small mass and size! -->
+  <xacro:link_creator_i link_name="fire_trigger_servo_link" mesh_path="Box" pose_xyz="0 0 0" pose_rpy="0 0 0" scale_xyz="0.04 0.009 0.009" mass="0.505" iner="0.001 0 0 0.001 0 0.001"/>
+  <gazebo reference="fire_trigger_servo_link">
+    <material>Gazebo/Red</material>
+    <self_collide>0</self_collide>
+  </gazebo>
 </robot>
 <!--

File: xacros/drone_maker.xacro (robot description, xacro)
@@ -1,18 +1,19 @@
 <?xml version="1.0" ?>
-<xmlns:xacro="http://www.ros.org/wiki/xacro">
+<robot xmlns:xacro="http://www.ros.org/wiki/xacro">
     <xacro:include filename="macro.xacro"/>
+    <xacro:property name="deg_to_rad" value="0.0174533"/>
     <xacro:macro name="drone_maker" params="base_mesh:='Box' base_pose_xyz:='0 0 0' base_pose_rpy:='0 0 0' base_scale_xyz:='0.4 0.4 0.04' base_center_of_mass:='0 0 0' base_mass base_iner:='None'
                                             number_of_arms arm_angles cws prop_meshs
                                             dis_from_center length diameter arm_incline_angle:='0' arm_mesh prop_size_multiplier
-                                            cylinder_d cylinder_l a_mass a_iner:='None' cla cp area r_mass r_iner
-                                            **extra_settings">
+                                            cylinder_d cylinder_l a_mass a_iner:='None' cla cp area r_mass r_iner">
+        <xacro:property name="base_pose_rpy_list" value="${base_pose_rpy.split(' ')}" />
+        <xacro:property name="base_pose_rpy_converted" value="${float(base_pose_rpy_list[0]) * deg_to_rad} ${float(base_pose_rpy_list[1]) * deg_to_rad} ${float(base_pose_rpy_list[2]) * deg_to_rad}" />
         <!-- Define base_link! -->
-        <xacro:link_creator_i link_name="base_link" pose_xyz="${base_pose_xyz}" pose_rpy="${base_pose_rpy}" mesh_path="${base_mesh}"
+        <xacro:link_creator_i link_name="base_link" pose_xyz="${base_pose_xyz}" pose_rpy="${base_pose_rpy_converted}" mesh_path="${base_mesh}"
                                 scale_xyz="${base_scale_xyz}" center_mass_xyz="${base_center_of_mass}" mass="${base_mass}" iner="${base_iner}"/>
         <!-- Define arms! -->
+        <xacro:property name="arm_angle_list" value="${arm_angles.split(' ')}" />
+        <xacro:property name="cw_list" value="${cws.split(' ')}" />
         <xacro:property name="prop_mesh_list" value="${prop_meshs.split(' ')}" />
-        <xacro:property name="cw_list" value="${cws.split(' ')}" />
-        <xacro:property name="arm_angle_list" value="${arm_angles.split(' ')}" />
-        <xacro:property name="deg_to_rad" value="0.0174533"/>
         <!-- Recursive macro definition -->
         <xacro:macro name="create_arms" params="i">
@@ -21,7 +22,7 @@
                 <xacro:property name="counter" value="${number_of_arms - i}" />
                 <xacro:drone_arm num="${counter}" parent_link="base_link" dis_from_center="${dis_from_center}" length="${length}" diameter="${diameter}"
-                                arm_incline_angle="${arm_incline_angle * deg_to_rad}" arm_mesh="${arm_mesh}" prop_mesh="${prop_mesh_list[counter]}" cw="cw_list[counter]"
+                                arm_incline_angle="${arm_incline_angle * deg_to_rad}" arm_mesh="${arm_mesh}" prop_mesh="${prop_mesh_list[counter]}" cw="${cw_list[counter]}"
                                 prop_size_multiplier="${prop_size_multiplier}" cylinder_d="${cylinder_d}" cylinder_l="${cylinder_l}" a_mass="${a_mass}" a_iner="${a_iner}" cla="${cla}" cp="${cp}"
-                                area="${area}" r_mass="${r_mass}" r_iner="${r_iner}" angle="${arm_angle_list[counter] * deg_to_rad}"/>
+                                area="${area}" r_mass="${r_mass}" r_iner="${r_iner}" angle="${float(arm_angle_list[counter]) * deg_to_rad}"/>
                 <!-- Recursively call the macro with a decremented count -->
                 <xacro:create_arms i="${i - 1}"/>
@@ -64,7 +65,6 @@
         </gazebo>
         <!-- end Define IMU! -->
-        <!-- Insert extra settings here!!! -->
-        <xacro:insert_block name="extra_settings"/>
-    </robot>
+    </xacro:macro>
+</robot>
 <!--
     THIS FILE DEFINES THE BASICS OF THE DRONE:
@@ -72,4 +72,3 @@
     ARMS
     IMU
-    and extra_settings tag is for adding extra settings to the model like legs, guns servos and more!
  -->

File: xacros/inertial_macros.xacro (robot description, xacro)
@@ -1,4 +1,4 @@
-<?xml version="1.0"?>
-<robot xmlns:xacro="http://www.ros.org/wiki/xacro" >
+<?xml version="1.0" ?>
+<robot xmlns:xacro="http://www.ros.org/wiki/xacro">
     <!-- Specify some standard inertial calculations https://en.wikipedia.org/wiki/List_of_moments_of_inertia -->
     <!-- These make use of xacro's mathematical functionality -->

File: xacros/macro.xacro (robot description, xacro)
@@ -1,3 +1,3 @@
-<?xml version="1.0"?>
+<?xml version="1.0" ?>
 <robot xmlns:xacro="http://www.ros.org/wiki/xacro">
     <xacro:include filename="inertial_macros.xacro"/>
@@ -160,5 +160,5 @@
         </xacro:link_creator_foundation>
     </xacro:macro>
-    <xacro:macro name="link_creator_i_foundation" params="link_name pose_xyz pose_rpy mesh_path:='Box' col_mesh_path:='None' scale_xyz col_scale_xyz:='100000000 0 0' seperate_collider_xyzrpy:='None' center_mass_xyz:='0 0 0' mass iner:='None' **extra_collision **extra_visual **extra_settings">
+    <xacro:macro name="link_creator_i_foundation" params="link_name pose_xyz pose_rpy mesh_path:='Box' col_mesh_path:='None' scale_xyz col_scale_xyz:='None' seperate_collider_xyzrpy:='None' center_mass_xyz:='0 0 0' mass iner:='None' **extra_collision **extra_visual **extra_settings">
         <xacro:link_creator_foundation link_name="${link_name}" pose_xyz="${pose_xyz}" pose_rpy="${pose_rpy}" mesh_path="${mesh_path}" scale_xyz="${scale_xyz}">
             <extra_visual><xacro:insert_block name="extra_visual"/></extra_visual>
@@ -166,25 +166,25 @@
                 <collision>
                     <geometry>
-                        <xacro:if value="${col_scale_xyz == '100000000 0 0'}">
-                            <xacro:if value="${col_mesh_path == 'None'}">
+                        <xacro:if value="${str(col_scale_xyz) == 'None'}">
+                            <xacro:if value="${str(col_mesh_path) == 'None'}">
                                 <xacro:set_mesh mesh="${mesh_path}" scale="${scale_xyz}" />
                             </xacro:if>
-                            <xacro:if value="${col_mesh_path != 'None'}">
+                            <xacro:if value="${str(col_mesh_path) != 'None'}">
                                 <xacro:set_mesh mesh="${col_mesh_path}" scale="${scale_xyz}" />
                             </xacro:if>
                         </xacro:if>
-                        <xacro:if value="${col_scale_xyz != '100000000 0 0'}">
-                            <xacro:if value="${col_mesh_path == 'None'}">
+                        <xacro:if value="${str(col_scale_xyz) != 'None'}">
+                            <xacro:if value="${str(col_mesh_path) == 'None'}">
                                 <xacro:set_mesh mesh="${mesh_path}" scale="${col_scale_xyz}" />
                             </xacro:if>
-                            <xacro:if value="${col_mesh_path != 'None'}">
+                            <xacro:if value="${str(col_mesh_path) != 'None'}">
                                 <xacro:set_mesh mesh="${col_mesh_path}" scale="${col_scale_xyz}" />
                             </xacro:if>
                         </xacro:if>
                     </geometry>
-                    <xacro:if value="${seperate_collider_xyzrpy == 'None'}">
+                    <xacro:if value="${str(seperate_collider_xyzrpy) == 'None'}">
                         <origin xyz="${pose_xyz}" rpy="${pose_rpy}"/>
                     </xacro:if>
-                    <xacro:if value="${seperate_collider_xyzrpy != 'None'}">
+                    <xacro:if value="${str(seperate_collider_xyzrpy) != 'None'}">
                         <xacro:property name="seperate_collider_xyzrpy_list" value="${seperate_collider_xyzrpy.split(' ')}" />
                         <origin xyz="${seperate_collider_xyzrpy_list[0]} ${seperate_collider_xyzrpy_list[1]} ${seperate_collider_xyzrpy_list[2]}" rpy="${seperate_collider_xyzrpy_list[3]} ${seperate_collider_xyzrpy_list[4]} ${seperate_collider_xyzrpy_list[5]}"/>
@@ -208,5 +208,5 @@
         </xacro:link_creator_foundation>
     </xacro:macro>
-    <xacro:macro name="link_creator_i" params="link_name pose_xyz pose_rpy mesh_path:='Box' col_mesh_path:='None' scale_xyz col_scale_xyz:='100000000 0 0' seperate_collider_xyzrpy:='None' center_mass_xyz:='0 0 0' mass iner:='None'">
+    <xacro:macro name="link_creator_i" params="link_name pose_xyz pose_rpy mesh_path:='Box' col_mesh_path:='None' scale_xyz col_scale_xyz:='None' seperate_collider_xyzrpy:='None' center_mass_xyz:='0 0 0' mass iner:='None'">
         <xacro:link_creator_i_foundation link_name="${link_name}" pose_xyz="${pose_xyz}" pose_rpy="${pose_rpy}" mesh_path="${mesh_path}" col_mesh_path="${col_mesh_path}" scale_xyz="${scale_xyz}" col_scale_xyz="${col_scale_xyz}" seperate_collider_xyzrpy="${seperate_collider_xyzrpy}" center_mass_xyz="${center_mass_xyz}" mass="${mass}" iner="${iner}">
             <extra_collision/>
