Commit message: now can specify the number of blades a prop has

File: models/copterPIX/robot.urdf.xacro (robot description, xacro)
@@ -35,7 +35,4 @@
   <xacro:property name="a_mass" value="0.5"/>
   <xacro:property name="a_iner" value="None"/>
-  <xacro:property name="cla" value="4.3"/>
-  <xacro:property name="cp" value="0.2"/>
-  <xacro:property name="area" value="0.01"/>
   <xacro:property name="r_mass" value="0.2"/>
   <xacro:property name="r_iner" value="0.000312 0 0 0.0053345 0 0.005363328"/>
@@ -49,4 +46,16 @@
   <xacro:property name="ardu_cmd_max" value="2.5"/>
   <xacro:property name="ardu_cmd_min" value="-2.5"/>
+  <xacro:property name="number_of_blades" value="2"/>
+  <xacro:property name="lift_a0" value="0.3"/>
+  <xacro:property name="lift_alpha_stall" value="1.4"/>
+  <xacro:property name="lift_cla" value="4.3"/>
+  <xacro:property name="lift_cda" value="0.10"/>
+  <xacro:property name="lift_cma" value="0.00"/>
+  <xacro:property name="lift_cla_stall" value="-0.025"/>
+  <xacro:property name="lift_sda_stall" value="0.0"/>
+  <xacro:property name="lift_cma_stall" value="0.0"/>
+  <xacro:property name="lift_area" value="0.01"/>
+  <xacro:property name="lift_air_density" value="1.2041"/>
+  <xacro:property name="lift_cp" value="0.2"/>
   <xacro:drone_maker base_mesh="${base_mesh}" base_pose_xyz ="${base_pose_xyz}" base_pose_rpy="${base_pose_rpy}" base_scale_xyz="${base_scale_xyz}"
                      base_center_of_mass="${base_center_of_mass}" base_mass="${base_mass}" base_iner="${base_iner}"
@@ -55,8 +64,11 @@
                      arm_incline_angle="${arm_incline_angle}" arm_mesh="${arm_mesh}" prop_size_multiplier="${prop_size_multiplier}"
                      cylinder_d="${cylinder_d}" cylinder_l="${cylinder_l}" a_mass="${a_mass}" a_iner="${a_iner}"
-                     cla="${cla}" cp="${cp}" area="${area}" r_mass="${r_mass}"  r_iner="${r_iner}"
+                     r_mass="${r_mass}"  r_iner="${r_iner}"
                      ardu_multiplier="${ardu_multiplier}" ardu_offset="${ardu_offset}"
                      ardu_p_gain="${ardu_p_gain}" ardu_i_gain="${ardu_i_gain}" ardu_d_gain="${ardu_d_gain}"
-                     ardu_i_max="${ardu_i_max}" ardu_i_min="${ardu_i_min}" ardu_cmd_max="${ardu_cmd_max}" ardu_cmd_min="${ardu_cmd_min}">
+                     ardu_i_max="${ardu_i_max}" ardu_i_min="${ardu_i_min}" ardu_cmd_max="${ardu_cmd_max}" ardu_cmd_min="${ardu_cmd_min}"
+                     number_of_blades="${number_of_blades}" lift_a0="${lift_a0}" lift_alpha_stall="${lift_alpha_stall}" lift_cla="${lift_cla}" lift_cda="${lift_cda}"
+                     lift_cma="${lift_cma}" lift_cla_stall="${lift_cla_stall}" lift_sda_stall="${lift_sda_stall}" lift_cma_stall="${lift_cma_stall}"
+                     lift_area="${lift_area}" lift_air_density="${lift_air_density}" lift_cp="${lift_cp}">
     <extra_ardupilot_plugin_settings>
       <xacro:extra_channel channel="6" _type="POSITION" _multiplier="1" _jointName="fire_trigger_servo_joint"

File: models/iris/robot.urdf.xacro (robot description, xacro)
@@ -14,5 +14,5 @@
   <xacro:property name="number_of_arms" value="4"/>
   <xacro:property name="arm_angles" value="45 225 135 315"/>
-  <xacro:property name="cws" value="0 0 1 1"/>
+  <xacro:property name="cws" value="0 0 1 1"/> <!-- 1: true 0: false -->
   <xacro:property name="prop_meshs" value="${prop_ccw_mesh} ${prop_ccw_mesh} ${prop_cw_mesh} ${prop_cw_mesh}"/>
   <xacro:property name="dis_from_center" value="0.08"/>
@@ -26,7 +26,4 @@
   <xacro:property name="a_mass" value="0.08"/>
   <xacro:property name="a_iner" value="None"/>
-  <xacro:property name="cla" value="4.25"/>
-  <xacro:property name="cp" value="0.084"/>
-  <xacro:property name="area" value="0.002"/>
   <xacro:property name="r_mass" value="0.025"/>
   <xacro:property name="r_iner" value="9.75e-06 0 0 0.000166704 0 0.000167604"/>
@@ -40,4 +37,16 @@
   <xacro:property name="ardu_cmd_max" value="2.5"/>
   <xacro:property name="ardu_cmd_min" value="-2.5"/>
+  <xacro:property name="number_of_blades" value="2"/>
+  <xacro:property name="lift_a0" value="0.3"/>
+  <xacro:property name="lift_alpha_stall" value="1.4"/>
+  <xacro:property name="lift_cla" value="4.25"/>
+  <xacro:property name="lift_cda" value="0.10"/>
+  <xacro:property name="lift_cma" value="0.00"/>
+  <xacro:property name="lift_cla_stall" value="-0.025"/>
+  <xacro:property name="lift_sda_stall" value="0.0"/>
+  <xacro:property name="lift_cma_stall" value="0.0"/>
+  <xacro:property name="lift_area" value="0.002"/>
+  <xacro:property name="lift_air_density" value="1.2041"/>
+  <xacro:property name="lift_cp" value="0.084"/>
   <xacro:drone_maker base_mesh="${base_mesh}" base_pose_xyz ="${base_pose_xyz}" base_pose_rpy="${base_pose_rpy}" base_scale_xyz="${base_scale_xyz}"
                      base_center_of_mass="${base_center_of_mass}" base_mass="${base_mass}" base_iner="${base_iner}"
@@ -46,8 +55,11 @@
                      arm_incline_angle="${arm_incline_angle}" arm_mesh="${arm_mesh}" prop_size_multiplier="${prop_size_multiplier}"
                      cylinder_d="${cylinder_d}" cylinder_l="${cylinder_l}" a_mass="${a_mass}" a_iner="${a_iner}"
-                     cla="${cla}" cp="${cp}" area="${area}" r_mass="${r_mass}"  r_iner="${r_iner}"
+                     r_mass="${r_mass}"  r_iner="${r_iner}"
                      ardu_multiplier="${ardu_multiplier}" ardu_offset="${ardu_offset}"
                      ardu_p_gain="${ardu_p_gain}" ardu_i_gain="${ardu_i_gain}" ardu_d_gain="${ardu_d_gain}"
-                     ardu_i_max="${ardu_i_max}" ardu_i_min="${ardu_i_min}" ardu_cmd_max="${ardu_cmd_max}" ardu_cmd_min="${ardu_cmd_min}">
+                     ardu_i_max="${ardu_i_max}" ardu_i_min="${ardu_i_min}" ardu_cmd_max="${ardu_cmd_max}" ardu_cmd_min="${ardu_cmd_min}"
+                     number_of_blades="${number_of_blades}" lift_a0="${lift_a0}" lift_alpha_stall="${lift_alpha_stall}" lift_cla="${lift_cla}" lift_cda="${lift_cda}"
+                     lift_cma="${lift_cma}" lift_cla_stall="${lift_cla_stall}" lift_sda_stall="${lift_sda_stall}" lift_cma_stall="${lift_cma_stall}"
+                     lift_area="${lift_area}" lift_air_density="${lift_air_density}" lift_cp="${lift_cp}">
     <extra_ardupilot_plugin_settings>
     </extra_ardupilot_plugin_settings>

File: models/simple_box/robot.urdf.xacro (robot description, xacro)
@@ -39,4 +39,6 @@
 <xacro:macro name="aaa" params="">
   <xacro:property name="b" value="base_link"/>
+  <xacro:property name="aasdf" value="1 0 0"/>
+  <xacro:property name="scale_list" value="${aasdf.split(' ')}" />
   <!-- Recursive macro definition -->
   <xacro:macro name="create_joints" params="i">
@@ -45,5 +47,5 @@
         <parent link="${b}"/>
         <child link="box_${i}"/>
-        <origin xyz="0 0 ${i}"/>
+        <origin xyz="${int(scale_list[0]) * i * sin(90)} ${int(scale_list[0]) * i * sin(pi)} ${int(scale_list[2]) * i}"/>
       </joint>
       <link name="box_${i}">

File: xacros/ardupilot_plugin.xacro (robot description, xacro)
@@ -25,6 +25,8 @@
                 <fdm_port_in>9002</fdm_port_in>
                 <fdm_port_out>9003</fdm_port_out>
-                <modelXYZToAirplaneXForwardZDown>0 0 0 3.141593 0 0</modelXYZToAirplaneXForwardZDown>
-                <gazeboXYZToNED>0 0 0 3.141593 0 0</gazeboXYZToNED>
+                <!-- <modelXYZToAirplaneXForwardZDown>0 0 0 3.141593 0 0</modelXYZToAirplaneXForwardZDown>
+                <gazeboXYZToNED>0 0 0 3.141593 0 0</gazeboXYZToNED> -->
+                <modelXYZToAirplaneXForwardZDown>0 0 0 ${pi} 0 0</modelXYZToAirplaneXForwardZDown>
+                <gazeboXYZToNED>0 0 0 ${pi} 0 0</gazeboXYZToNED>
                 <imuName>imu_link::imu_sensor</imuName>
                 <connectionTimeoutMaxCount>5</connectionTimeoutMaxCount>

File: xacros/drone_maker.xacro (robot description, xacro)
@@ -7,7 +7,10 @@
                                             number_of_arms arm_angles cws prop_meshs
                                             dis_from_center length diameter arm_incline_angle:='0' arm_mesh prop_size_multiplier
-                                            cylinder_d cylinder_l a_mass a_iner:='None' cla cp area r_mass r_iner
+                                            cylinder_d cylinder_l a_mass a_iner:='None' r_mass r_iner
                                             ardu_multiplier ardu_offset ardu_p_gain ardu_i_gain ardu_d_gain
                                             ardu_i_max ardu_i_min ardu_cmd_max ardu_cmd_min
+                                            number_of_blades lift_a0 lift_alpha_stall
+                                            lift_cla lift_cda lift_cma lift_cla_stall lift_sda_stall lift_cma_stall
+                                            lift_area lift_air_density lift_cp
                                             **extra_ardupilot_plugin_settings">
         <xacro:property name="base_pose_rpy_list" value="${base_pose_rpy.split(' ')}" />
@@ -23,9 +26,13 @@
             <xacro:if value="${i > 0}">
                 <!-- Here define the arm -->
-                <xacro:property name="counter" value="${number_of_arms - i}" />
+                <xacro:property name="counter" value="${int(number_of_arms) - i}" />
                 <xacro:drone_arm num="${counter}" parent_link="base_link" dis_from_center="${dis_from_center}" length="${length}" diameter="${diameter}"
                                 arm_incline_angle="${arm_incline_angle * deg_to_rad}" arm_mesh="${arm_mesh}" prop_mesh="${prop_mesh_list[counter]}" cw="${cw_list[counter]}"
-                                prop_size_multiplier="${prop_size_multiplier}" cylinder_d="${cylinder_d}" cylinder_l="${cylinder_l}" a_mass="${a_mass}" a_iner="${a_iner}" cla="${cla}" cp="${cp}"
-                                area="${area}" r_mass="${r_mass}" r_iner="${r_iner}" angle="${float(arm_angle_list[counter]) * deg_to_rad}"/>
+                                prop_size_multiplier="${prop_size_multiplier}" cylinder_d="${cylinder_d}" cylinder_l="${cylinder_l}"
+                                a_mass="${a_mass}" a_iner="${a_iner}" r_mass="${r_mass}" r_iner="${r_iner}" angle="${float(arm_angle_list[counter]) * deg_to_rad}"
+                                number_of_blades="${number_of_blades}"
+                                lift_a0="${lift_a0}" lift_alpha_stall="${lift_alpha_stall}" lift_cla="${lift_cla}" lift_cda="${lift_cda}"
+                                lift_cma="${lift_cma}" lift_cla_stall="${lift_cla_stall}" lift_sda_stall="${lift_sda_stall}" lift_cma_stall="${lift_cma_stall}"
+                                lift_area="${lift_area}" lift_air_density="${lift_air_density}" lift_cp="${lift_cp}"/>
                 <!-- Recursively call the macro with a decremented count -->
                 <xacro:create_arms i="${i - 1}"/>
@@ -33,5 +40,5 @@
         </xacro:macro>
         <!-- Initial call to the macro with the desired number of joints -->
-        <xacro:create_arms i="${number_of_arms}"/>
+        <xacro:create_arms i="${int(number_of_arms)}"/>
         <!-- end Define arms! -->
         <!-- Define IMU! -->

File: xacros/macro.xacro (robot description, xacro)
@@ -2,11 +2,12 @@
 <robot xmlns:xacro="http://www.ros.org/wiki/xacro">
     <xacro:include filename="inertial_macros.xacro"/>
-    <xacro:macro name="drone_arm" params="num parent_link dis_from_center length diameter arm_incline_angle arm_mesh prop_mesh cw prop_size_multiplier cylinder_d cylinder_l a_mass a_iner:='None' cla cp area r_mass r_iner angle">
+    <xacro:macro name="drone_arm" params="num parent_link dis_from_center length diameter arm_incline_angle arm_mesh prop_mesh cw
+                                          prop_size_multiplier cylinder_d cylinder_l a_mass a_iner:='None' r_mass r_iner angle
+                                          number_of_blades lift_a0 lift_alpha_stall lift_cla lift_cda lift_cma lift_cla_stall lift_sda_stall lift_cma_stall
+                                          lift_area lift_air_density lift_cp">
         <xacro:property name="base_arm_joint" value="base_arm_joint_${num}" />
         <xacro:property name="arm_link" value="arm_link_${num}" />
         <xacro:property name="rotor_joint" value="rotor_joint_${num}" />
         <xacro:property name="prop_link" value="prop_link_${num}" />
-        <xacro:property name="rotor_blade_0" value="rotor_${num}_blade_0" />
-        <xacro:property name="rotor_blade_1" value="rotor_${num}_blade_1" />
         <joint name="${base_arm_joint}" type="fixed">
             <parent link="${parent_link}"/>
@@ -29,78 +30,87 @@
             </physics>
         </gazebo>
-        <xacro:prop_link_creator link_name="${prop_link}" pose_xyz="0 0 0.03" pose_rpy="0 -0 0" mesh_path="${prop_mesh}" scale_xyz="${prop_size_multiplier} ${prop_size_multiplier} ${prop_size_multiplier}" col_scale_xyz="${cylinder_d} 0 ${cylinder_l}" mass="${r_mass}" iner="${r_iner}"/>
-        <xacro:property name="cp_negative" value="${-1 * cp}"/>
-        <xacro:if value="${cw}">
-            <gazebo>
-                <plugin name="${rotor_blade_0}" filename="libLiftDragPlugin.so">
-                    <a0>0.3</a0>
-                    <alpha_stall>1.4</alpha_stall>
-                    <cla>${cla}</cla>
-                    <cda>0.10</cda>
-                    <cma>0.00</cma>
-                    <cla_stall>-0.025</cla_stall>
-                    <cda_stall>0.0</cda_stall>
-                    <cma_stall>0.0</cma_stall>
-                    <area>${area}</area>
-                    <air_density>1.2041</air_density>
-                    <cp>${cp} 0 0</cp>
-                    <forward>0 -1 0</forward>
-                    <upward>0 0 1</upward>
-                    <link_name>${prop_link}</link_name>
-                </plugin>
-                <plugin name="${rotor_blade_1}" filename="libLiftDragPlugin.so">
-                    <a0>0.3</a0>
-                    <alpha_stall>1.4</alpha_stall>
-                    <cla>${cla}</cla>
-                    <cda>0.10</cda>
-                    <cma>0.00</cma>
-                    <cla_stall>-0.025</cla_stall>
-                    <cda_stall>0.0</cda_stall>
-                    <cma_stall>0.0</cma_stall>
-                    <area>${area}</area>
-                    <air_density>1.2041</air_density>
-                    <cp>${cp_negative} 0 0</cp>
-                    <forward>0 1 0</forward>
-                    <upward>0 0 1</upward>
-                    <link_name>${prop_link}</link_name>
-                </plugin>
-            </gazebo>
-        </xacro:if>
-        <xacro:unless value="${cw}">
-            <gazebo>
-                <plugin name="${rotor_blade_0}" filename="libLiftDragPlugin.so">
-                    <a0>0.3</a0>
-                    <alpha_stall>1.4</alpha_stall>
-                    <cla>${cla}</cla>
-                    <cda>0.10</cda>
-                    <cma>0.00</cma>
-                    <cla_stall>-0.025</cla_stall>
-                    <cda_stall>0.0</cda_stall>
-                    <cma_stall>0.0</cma_stall>
-                    <area>${area}</area>
-                    <air_density>1.2041</air_density>
-                    <cp>${cp} 0 0</cp>
-                    <forward>0 1 0</forward>
-                    <upward>0 0 1</upward>
-                    <link_name>${prop_link}</link_name>
-                </plugin>
-                <plugin name="${rotor_blade_1}" filename="libLiftDragPlugin.so">
-                    <a0>0.3</a0>
-                    <alpha_stall>1.4</alpha_stall>
-                    <cla>${cla}</cla>
-                    <cda>0.10</cda>
-                    <cma>0.00</cma>
-                    <cla_stall>-0.025</cla_stall>
-                    <cda_stall>0.0</cda_stall>
-                    <cma_stall>0.0</cma_stall>
-                    <area>${area}</area>
-                    <air_density>1.2041</air_density>
-                    <cp>${cp_negative} 0 0</cp>
-                    <forward>0 -1 0</forward>
-                    <upward>0 0 1</upward>
-                    <link_name>${prop_link}</link_name>
-                </plugin>
-            </gazebo>
-        </xacro:unless>
+        <xacro:prop_link_creator link_name="${prop_link}" pose_xyz="0 0 0.03" pose_rpy="0 -0 0" mesh_path="${prop_mesh}"
+                                 scale_xyz="${prop_size_multiplier} ${prop_size_multiplier} ${prop_size_multiplier}"
+                                 col_scale_xyz="${cylinder_d} 0 ${cylinder_l}" mass="${r_mass}" iner="${r_iner}"/>
+        <xacro:property name="direction" value="${(int(cw) * 2) - 1}"/>
+        <xacro:macro name="create_blades" params="i">
+            <xacro:if value="${i > 0}">
+                <!-- Here define the arm -->
+                <xacro:property name="counter" value="${number_of_blades - i}"/>
+                <xacro:property name="directed_multiplier" value="${multiplier * ((int(cw_list[counter]) * (-2)) + 1)}"/>
+                <xacro:property name="rotor_blade" value="rotor_${num}_blade_${counter}"/>
+                <xacro:property name="blade_angle" value="${(pi / number_of_blades) * counter}"/>
+                <gazebo>
+                    <plugin name="${rotor_blade}" filename="libLiftDragPlugin.so">
+                        <a0>${lift_a0}</a0>
+                        <alpha_stall>${lift_alpha_stall}</alpha_stall>
+                        <cla>${lift_cla}</cla>
+                        <cda>${lift_cda}</cda>
+                        <cma>${lift_cma}</cma>
+                        <cla_stall>${lift_cla_stall}</cla_stall>
+                        <cda_stall>${lift_sda_stall}</cda_stall>
+                        <cma_stall>${lift_cma_stall}</cma_stall>
+                        <area>${lift_area}</area>
+                        <air_density>${lift_air_density}</air_density>
+                        <cp>${cos(blade_angle) * lift_cp} ${sin(blade_angle) * lift_cp} 0</cp>
+                        <!-- <forward>${sin(blade_angle * direction)} ${cos(blade_angle * direction * -1)} 0</forward> -->
+                        <forward>0 ${direction} 0</forward>
+                        <upward>0 0 1</upward>
+                        <link_name>${prop_link}</link_name>
+                    </plugin>
+                </gazebo>
+                <!-- Recursively call the macro with a decremented count -->
+                <xacro:create_blades i="${i - 1}"/>
+            </xacro:if>
+        </xacro:macro>
+        <!-- Initial call to the macro with the desired number of joints -->
+        <xacro:create_blades i="${int(number_of_blades)}"/>
+        <!-- end Define arms! -->
+            <!-- <plugin name="${rotor_blade_0}" filename="libLiftDragPlugin.so">
+                <a0>${lift_a0}</a0> lift_a0 lift_alpha_stall lift_cla lift_cda lift_cma lift_cla_stall lift_sda_stall lift_cma_stall lift_area lift_air_density
+                <alpha_stall>${lift_alpha_stall}</alpha_stall>
+                <cla>${lift_cla}</cla>
+                <cda>${lift_cda}</cda>
+                <cma>${lift_cma}</cma>
+                <cla_stall>${lift_cla_stall}</cla_stall>
+                <cda_stall>${lift_sda_stall}</cda_stall>
+                <cma_stall>${lift_cma_stall}</cma_stall>
+                <area>${lift_area}</area>
+                <air_density>${lift_air_density}</air_density>
+                <cp>${cp} 0 0</cp>
+                <forward>0 ${direction * -1} 0</forward>
+                <upward>0 0 1</upward>
+                <link_name>${prop_link}</link_name>
+            </plugin>
+            <plugin name="${rotor_blade_1}" filename="libLiftDragPlugin.so">
+                <a0>0.3</a0>
+                <alpha_stall>1.4</alpha_stall>
+                <cla>${cla}</cla>
+                <cda>0.10</cda>
+                <cma>0.00</cma>
+                <cla_stall>-0.025</cla_stall>
+                <cda_stall>0.0</cda_stall>
+                <cma_stall>0.0</cma_stall>
+                <area>${area}</area>
+                <air_density>1.2041</air_density>
+                <cp>${cp * -1} 0 0</cp>
+                <forward>0 ${direction} 0</forward>
+                <upward>0 0 1</upward>
+                <link_name>${prop_link}</link_name>
+            </plugin> -->
+                <!-- <a0>0.3</a0>
+                <alpha_stall>1.4</alpha_stall>
+                <cla>${cla}</cla>
+                <cda>0.10</cda>
+                <cma>0.00</cma>
+                <cla_stall>-0.025</cla_stall>
+                <cda_stall>0.0</cda_stall>
+                <cma_stall>0.0</cma_stall>
+                <area>${area}</area>
+                <air_density>1.2041</air_density>
+                <cp>${cp} 0 0</cp>
+                <forward>0 ${direction * -1} 0</forward>
+                <upward>0 0 1</upward>
+                <link_name>${prop_link}</link_name>  -->
         <gazebo reference="${arm_link}">
             <visual>
