Commit message: lift fixed

File: models/copterPIX/robot.urdf.xacro (robot description, xacro)
@@ -55,5 +55,5 @@
   <xacro:property name="lift_sda_stall" value="0.0"/>
   <xacro:property name="lift_cma_stall" value="0.0"/>
-  <xacro:property name="lift_area" value="0.01"/>
+  <xacro:property name="lift_area" value="0.008"/>
   <xacro:property name="lift_air_density" value="1.2041"/>
   <xacro:property name="lift_cp" value="0.2"/>

File: xacros/ardupilot_plugin.xacro (robot description, xacro)
@@ -25,6 +25,4 @@
                 <fdm_port_in>9002</fdm_port_in>
                 <fdm_port_out>9003</fdm_port_out>
-                <!-- <modelXYZToAirplaneXForwardZDown>0 0 0 3.141593 0 0</modelXYZToAirplaneXForwardZDown>
-                <gazeboXYZToNED>0 0 0 3.141593 0 0</gazeboXYZToNED> -->
                 <modelXYZToAirplaneXForwardZDown>0 0 0 ${pi} 0 0</modelXYZToAirplaneXForwardZDown>
                 <gazeboXYZToNED>0 0 0 ${pi} 0 0</gazeboXYZToNED>

File: xacros/drone_maker.xacro (robot description, xacro)
@@ -3,5 +3,5 @@
     <xacro:include filename="macro.xacro"/>
     <xacro:include filename="ardupilot_plugin.xacro"/>
-    <xacro:property name="deg_to_rad" value="0.0174533"/>
+    <xacro:property name="deg_to_rad" value="0.0174532925"/>
     <xacro:macro name="drone_maker" params="base_mesh:='Box' base_pose_xyz:='0 0 0' base_pose_rpy:='0 0 0' base_scale_xyz:='0.4 0.4 0.04' base_center_of_mass:='0 0 0' base_mass base_iner:='None'
                                             number_of_arms arm_angles cws prop_meshs

File: xacros/macro.xacro (robot description, xacro)
@@ -33,12 +33,12 @@
                                  scale_xyz="${prop_size_multiplier} ${prop_size_multiplier} ${prop_size_multiplier}"
                                  col_scale_xyz="${cylinder_d} 0 ${cylinder_l}" mass="${r_mass}" iner="${r_iner}"/>
-        <xacro:property name="direction" value="${(int(cw) * 2) - 1}"/>
+        <xacro:property name="direction" value="${(float(cw) * 2) - 1}"/>
         <xacro:macro name="create_blades" params="i">
             <xacro:if value="${i > 0}">
                 <!-- Here define the arm -->
                 <xacro:property name="counter" value="${number_of_blades - i}"/>
-                <xacro:property name="directed_multiplier" value="${multiplier * ((int(cw_list[counter]) * (-2)) + 1)}"/>
                 <xacro:property name="rotor_blade" value="rotor_${num}_blade_${counter}"/>
-                <xacro:property name="blade_angle" value="${(pi / number_of_blades) * counter}"/>
+                <xacro:property name="blade_angle" value="${((2 * pi) / float(number_of_blades)) * float(counter)}"/>
+                <!-- <xacro:property name="blade_angle" value="${(num * pi) / 12}"/> -->
                 <gazebo>
                     <plugin name="${rotor_blade}" filename="libLiftDragPlugin.so">
@@ -53,7 +53,6 @@
                         <area>${lift_area}</area>
                         <air_density>${lift_air_density}</air_density>
-                        <cp>${cos(blade_angle) * lift_cp} ${sin(blade_angle) * lift_cp} 0</cp>
-                        <!-- <forward>${sin(blade_angle * direction)} ${cos(blade_angle * direction * -1)} 0</forward> -->
-                        <forward>0 ${direction} 0</forward>
+                        <cp>${cos(float(blade_angle)) * float(lift_cp)} ${sin(float(blade_angle)) * float(lift_cp)} 0</cp>
+                        <forward>${cos(float(blade_angle) - ((pi / 2) * direction))} ${sin(float(blade_angle) - ((pi / 2) * direction))} 0</forward>
                         <upward>0 0 1</upward>
                         <link_name>${prop_link}</link_name>
@@ -67,68 +66,4 @@
         <xacro:create_blades i="${int(number_of_blades)}"/>
         <!-- end Define arms! -->
-            <!-- <plugin name="${rotor_blade_0}" filename="libLiftDragPlugin.so">
-                <a0>${lift_a0}</a0> lift_a0 lift_alpha_stall lift_cla lift_cda lift_cma lift_cla_stall lift_sda_stall lift_cma_stall lift_area lift_air_density
-                <alpha_stall>${lift_alpha_stall}</alpha_stall>
-                <cla>${lift_cla}</cla>
-                <cda>${lift_cda}</cda>
-                <cma>${lift_cma}</cma>
-                <cla_stall>${lift_cla_stall}</cla_stall>
-                <cda_stall>${lift_sda_stall}</cda_stall>
-                <cma_stall>${lift_cma_stall}</cma_stall>
-                <area>${lift_area}</area>
-                <air_density>${lift_air_density}</air_density>
-                <cp>${cp} 0 0</cp>
-                <forward>0 ${direction * -1} 0</forward>
-                <upward>0 0 1</upward>
-                <link_name>${prop_link}</link_name>
-            </plugin>
-            <plugin name="${rotor_blade_1}" filename="libLiftDragPlugin.so">
-                <a0>0.3</a0>
-                <alpha_stall>1.4</alpha_stall>
-                <cla>${cla}</cla>
-                <cda>0.10</cda>
-                <cma>0.00</cma>
-                <cla_stall>-0.025</cla_stall>
-                <cda_stall>0.0</cda_stall>
-                <cma_stall>0.0</cma_stall>
-                <area>${area}</area>
-                <air_density>1.2041</air_density>
-                <cp>${cp * -1} 0 0</cp>
-                <forward>0 ${direction} 0</forward>
-                <upward>0 0 1</upward>
-                <link_name>${prop_link}</link_name>
-            </plugin> -->
-                <!-- <a0>0.3</a0>
-                <alpha_stall>1.4</alpha_stall>
-                <cla>${cla}</cla>
-                <cda>0.10</cda>
-                <cma>0.00</cma>
-                <cla_stall>-0.025</cla_stall>
-                <cda_stall>0.0</cda_stall>
-                <cma_stall>0.0</cma_stall>
-                <area>${area}</area>
-                <air_density>1.2041</air_density>
-                <cp>${cp} 0 0</cp>
-                <forward>0 ${direction * -1} 0</forward>
-                <upward>0 0 1</upward>
-                <link_name>${prop_link}</link_name>  -->
-        <gazebo reference="${arm_link}">
-            <visual>
-                <material>
-                    <script>
-                        <name>Gazebo/DarkGrey</name>
-                    </script>
-                </material>
-            </visual>
-        </gazebo>
-        <gazebo reference="${prop_link}">
-            <visual>
-                <material>
-                    <script>
-                        <name>Gazebo/DarkGrey</name>
-                    </script>
-                </material>
-            </visual>
-        </gazebo>
     </xacro:macro>
     <xacro:macro name="set_mesh" params="mesh scale">
@@ -163,4 +98,13 @@
             <xacro:insert_block name="extra_settings"/>
         </link>
+        <gazebo reference="${link_name}">
+            <visual>
+                <material>
+                    <script>
+                        <name>Gazebo/DarkGrey</name>
+                    </script>
+                </material>
+            </visual>
+        </gazebo>
     </xacro:macro>
     <xacro:macro name="link_creator" params="link_name pose_xyz pose_rpy mesh_path:='Box' scale_xyz">
@@ -211,5 +155,5 @@
                         <origin xyz="${center_mass_xyz}" rpy="0 0 0"/>
                         <mass value="${mass}"/>
-                        <inertia ixx="${iner_list[0]}" ixy="${iner_list[1]}" ixz="${iner_list[2]}" iyy="${iner_list[3]}" iyz="${iner_list[4]}" izz="${iner_list[5]}"/>
+                        <inertia ixx="${float(iner_list[0])}" ixy="${float(iner_list[1])}" ixz="${float(iner_list[2])}" iyy="${iner_list[3]}" iyz="${float(iner_list[4])}" izz="${float(iner_list[5])}"/>
                     </inertial>
                 </xacro:if>

Commit message: still working on the readme.md, also the weird moment the drone gets when it falls its still unsloved. don't know why. try make the prop direction different for next troubleshoot

File: models/copterPIX/robot.urdf.xacro (robot description, xacro)
@@ -29,4 +29,5 @@
   <xacro:property name="diameter" value="0.025"/>
   <xacro:property name="arm_incline_angle" value="5"/>
+  <xacro:property name="rotor_dis_from_arm" value="0.03"/>
   <xacro:property name="arm_mesh" value="${hex_mesh}"/>
   <xacro:property name="prop_size_multiplier" value="2.34"/>
@@ -62,5 +63,5 @@
                      number_of_arms="${number_of_arms}" arm_angles="${arm_angles}" cws="${cws}" prop_meshs="${prop_meshs}"
                      dis_from_center="${dis_from_center}" length="${length}" diameter="${diameter}"
-                     arm_incline_angle="${arm_incline_angle}" arm_mesh="${arm_mesh}" prop_size_multiplier="${prop_size_multiplier}"
+                     arm_incline_angle="${arm_incline_angle}" rotor_dis_from_arm="${rotor_dis_from_arm}" arm_mesh="${arm_mesh}" prop_size_multiplier="${prop_size_multiplier}"
                      cylinder_d="${cylinder_d}" cylinder_l="${cylinder_l}" a_mass="${a_mass}" a_iner="${a_iner}"
                      r_mass="${r_mass}"  r_iner="${r_iner}"

File: models/iris/robot.urdf.xacro (robot description, xacro)
@@ -20,4 +20,5 @@
   <xacro:property name="diameter" value="0.01"/>
   <xacro:property name="arm_incline_angle" value="0"/>
+  <xacro:property name="rotor_dis_from_arm" value="0.015"/>
   <xacro:property name="arm_mesh" value="${hex_mesh}"/>
   <xacro:property name="prop_size_multiplier" value="1"/>
@@ -53,5 +54,5 @@
                      number_of_arms="${number_of_arms}" arm_angles="${arm_angles}" cws="${cws}" prop_meshs="${prop_meshs}"
                      dis_from_center="${dis_from_center}" length="${length}" diameter="${diameter}"
-                     arm_incline_angle="${arm_incline_angle}" arm_mesh="${arm_mesh}" prop_size_multiplier="${prop_size_multiplier}"
+                     arm_incline_angle="${arm_incline_angle}" rotor_dis_from_arm="${rotor_dis_from_arm}" arm_mesh="${arm_mesh}" prop_size_multiplier="${prop_size_multiplier}"
                      cylinder_d="${cylinder_d}" cylinder_l="${cylinder_l}" a_mass="${a_mass}" a_iner="${a_iner}"
                      r_mass="${r_mass}"  r_iner="${r_iner}"

File: models/simple_box/robot.urdf.xacro (robot description, xacro)
@@ -37,31 +37,30 @@
     </link>
   </xacro:macro>
-<xacro:macro name="aaa" params="">
-  <xacro:property name="b" value="base_link"/>
-  <xacro:property name="aasdf" value="1 0 0"/>
-  <xacro:property name="scale_list" value="${aasdf.split(' ')}" />
-  <!-- Recursive macro definition -->
-  <xacro:macro name="create_joints" params="i">
-    <xacro:if value="${i > 0}">
-      <joint name="base_child_joint_${i}" type="fixed">
-        <parent link="${b}"/>
-        <child link="box_${i}"/>
-        <origin xyz="${int(scale_list[0]) * i * sin(90)} ${int(scale_list[0]) * i * sin(pi)} ${int(scale_list[2]) * i}"/>
-      </joint>
-      <link name="box_${i}">
-        <visual>
-          <geometry>
-            <box size="1 1 1"/>
-          </geometry>
-          <origin xyz="0 0 0"/>
-        </visual>
-      </link>
-      <!-- Recursively call the macro with a decremented count -->
-      <xacro:create_joints i="${i - 1}"/>
-    </xacro:if>
-  </xacro:macro>
-  <!-- Initial call to the macro with the desired number of joints -->
-  <xacro:create_joints i="5"/>
-  </xacro:macro>
+  <xacro:macro name="aaa" params="">
+    <xacro:property name="b" value="base_link"/>
+    <xacro:property name="aasdf" value="1 0 0"/>
+    <xacro:property name="scale_list" value="${aasdf.split(' ')}" />
+    <xacro:macro name="create_joints" params="i">
+      <xacro:if value="${i > 0}">
+        <joint name="base_child_joint_${i}" type="fixed">
+          <parent link="${b}"/>
+          <child link="box_${i}"/>
+          <!-- <origin xyz="${int(scale_list[0]) * i * sin(90)} ${int(scale_list[0]) * i * sin(pi)} ${int(scale_list[2]) * i}"/> -->
+          <origin xyz="0 1 0" rpy="${((2 * pi) / 360) * 30} 0 ${((2 * pi) / 6) * (6 - i)}"/>
+          <!-- <origin xyz="0 1 0" rpy="0 0 0"/> -->
+        </joint>
+        <link name="box_${i}">
+          <visual>
+            <geometry>
+              <box size="1 1 1"/>
+            </geometry>
+            <origin xyz="0 0 0"/>
+          </visual>
+        </link>
+        <xacro:create_joints i="${i - 1}"/>
+      </xacro:if>
+    </xacro:macro>
+    <xacro:create_joints i="6"/>
+    </xacro:macro>
   <xacro:aaa />
   <link name="base_link">

File: xacros/arm_macro.xacro (robot description, xacro)
@@ -2,5 +2,5 @@
 <robot xmlns:xacro="http://www.ros.org/wiki/xacro">
     <xacro:include filename="link_macros.xacro"/>
-    <xacro:macro name="drone_arm" params="num parent_link dis_from_center length diameter arm_incline_angle arm_mesh prop_mesh cw
+    <xacro:macro name="drone_arm" params="num parent_link dis_from_center length diameter arm_incline_angle rotor_dis_from_arm arm_mesh prop_mesh cw
                                           prop_size_multiplier cylinder_d cylinder_l a_mass a_iner:='None' r_mass r_iner angle
                                           number_of_blades lift_a0 lift_alpha_stall lift_cla lift_cda lift_cma lift_cla_stall lift_sda_stall lift_cma_stall
@@ -19,5 +19,6 @@
             <parent link="${arm_link}"/>
             <child link="${prop_link}"/>
-            <origin xyz="0 ${cos(arm_incline_angle) * length + dis_from_center} ${sin(arm_incline_angle) * length}" rpy="${arm_incline_angle} 0 0"/>
+            <!-- <origin xyz="0 ${(cos(arm_incline_angle) * float(length)) - (sin(arm_incline_angle) * float(rotor_dis_from_arm))} ${(sin(arm_incline_angle) * float(length)) + (cos(arm_incline_angle) * float(rotor_dis_from_arm))}" rpy="${arm_incline_angle} 0 0"/> -->
+            <origin xyz="0 ${(cos(arm_incline_angle) * float(length + dis_from_center)) - (sin(arm_incline_angle) * float(rotor_dis_from_arm))} ${(sin(arm_incline_angle) * float(length)) + (cos(arm_incline_angle) * float(rotor_dis_from_arm))}" rpy="${arm_incline_angle} 0 0"/>
             <axis xyz="0 0 1"/>
             <dynamics damping="0.004"/>
@@ -30,7 +31,23 @@
             </physics>
         </gazebo>
-        <xacro:prop_link_creator link_name="${prop_link}" pose_xyz="0 0 0.03" pose_rpy="0 -0 0" mesh_path="${prop_mesh}"
-                                 scale_xyz="${prop_size_multiplier} ${prop_size_multiplier} ${prop_size_multiplier}"
-                                 col_scale_xyz="${cylinder_d} 0 ${cylinder_l}" mass="${r_mass}" iner="${r_iner}"/>
+        <xacro:link_creator_i_foundation link_name="${prop_link}" pose_xyz="0 0 0" pose_rpy="0 0 0" mesh_path="${prop_mesh}" col_mesh_path="Cylinder"
+                                         scale_xyz="${prop_size_multiplier} ${prop_size_multiplier} ${prop_size_multiplier}" col_scale_xyz="${cylinder_d} 0 ${cylinder_l}"
+                                         seperate_collider_xyzrpy="None"
+                                         center_mass_xyz="0 0 0" mass="${r_mass}"  iner="${r_iner}">
+            <extra_collision>
+                <surface>
+                    <contact>
+                        <ode/>
+                    </contact>
+                    <friction>
+                        <ode/>
+                    </friction>
+                </surface>
+            </extra_collision>
+            <extra_visual/>
+            <extra_settings>
+                <velocity_decay/>
+            </extra_settings>
+        </xacro:link_creator_i_foundation>
         <xacro:property name="direction" value="${(float(cw) * 2) - 1}"/>
         <xacro:macro name="create_blades" params="i">

File: xacros/drone_maker.xacro (robot description, xacro)
@@ -6,5 +6,5 @@
     <xacro:macro name="drone_maker" params="base_mesh:='Box' base_pose_xyz:='0 0 0' base_pose_rpy:='0 0 0' base_scale_xyz:='0.4 0.4 0.04' base_center_of_mass:='0 0 0' base_mass base_iner:='None'
                                             number_of_arms arm_angles cws prop_meshs
-                                            dis_from_center length diameter arm_incline_angle:='0' arm_mesh prop_size_multiplier
+                                            dis_from_center length diameter arm_incline_angle:='0' rotor_dis_from_arm arm_mesh prop_size_multiplier
                                             cylinder_d cylinder_l a_mass a_iner:='None' r_mass r_iner
                                             ardu_multiplier ardu_offset ardu_p_gain ardu_i_gain ardu_d_gain
@@ -28,5 +28,6 @@
                 <xacro:property name="counter" value="${int(number_of_arms) - i}" />
                 <xacro:drone_arm num="${counter}" parent_link="base_link" dis_from_center="${dis_from_center}" length="${length}" diameter="${diameter}"
-                                arm_incline_angle="${arm_incline_angle * deg_to_rad}" arm_mesh="${arm_mesh}" prop_mesh="${prop_mesh_list[counter]}" cw="${cw_list[counter]}"
+                                arm_incline_angle="${arm_incline_angle * deg_to_rad}" rotor_dis_from_arm="${rotor_dis_from_arm}" arm_mesh="${arm_mesh}"
+                                prop_mesh="${prop_mesh_list[counter]}" cw="${cw_list[counter]}"
                                 prop_size_multiplier="${prop_size_multiplier}" cylinder_d="${cylinder_d}" cylinder_l="${cylinder_l}"
                                 a_mass="${a_mass}" a_iner="${a_iner}" r_mass="${r_mass}" r_iner="${r_iner}" angle="${float(arm_angle_list[counter]) * deg_to_rad}"

File: xacros/link_macros.xacro (robot description, xacro)
@@ -104,24 +104,3 @@
         </xacro:link_creator_i_foundation>
     </xacro:macro>
-    <xacro:macro name="prop_link_creator" params="link_name pose_xyz pose_rpy mesh_path scale_xyz col_scale_xyz seperate_collider_xyzrpy:='None' center_mass_xyz:='0 0 0' mass iner">
-        <xacro:link_creator_i_foundation link_name="${link_name}" pose_xyz="${pose_xyz}" pose_rpy="${pose_rpy}" mesh_path="${mesh_path}" col_mesh_path="Cylinder" scale_xyz="${scale_xyz}" col_scale_xyz="${col_scale_xyz}" seperate_collider_xyzrpy="${seperate_collider_xyzrpy}" center_mass_xyz="${center_mass_xyz}" mass="${mass}"  iner="${iner}">
-            <extra_collision>
-                <surface>
-                    <contact>
-                        <ode/>
-                    </contact>
-                    <friction>
-                        <ode/>
-                    </friction>
-                </surface>
-            </extra_collision>
-            <extra_visual/>
-            <extra_settings>
-                <velocity_decay/>
-            </extra_settings>
-        </xacro:link_creator_i_foundation>
-        <!-- <gazebo reference="${link_name}">
-            <self_collide>0</self_collide>
-        </gazebo> -->
-    </xacro:macro>
 </robot>
