Commit message: added m16 and positioned it and the fire trigger(red thing)

File: models/copterPIX/robot.urdf.xacro (robot description, xacro)
@@ -5,4 +5,5 @@
   <xacro:property name="prop_cw_mesh" value="$(find drone)/meshes/iris_prop_cw.dae"/>
   <xacro:property name="prop_ccw_mesh" value="$(find drone)/meshes/iris_prop_ccw.dae"/>
+  <xacro:property name="M16_mesh" value="$(find drone)/meshes/M16.stl"/>
 <!--
   <xacro:property name="ixx" value="${373162267137.9 / g_mms_to_kg_ms}"/>  these values are not valid, they are stupid wrong
@@ -17,5 +18,5 @@
   <xacro:property name="base_pose_xyz" value="0 0 0"/>
   <xacro:property name="base_pose_rpy" value="0 0 0"/>
-  <xacro:property name="base_scale_xyz" value="0.4 0.4 0.04"/>
+  <xacro:property name="base_scale_xyz" value="0.4 0.4 0.05"/>
   <xacro:property name="base_center_of_mass" value="0 0 0"/>
   <xacro:property name="base_mass" value="19" />
@@ -73,5 +74,5 @@
                      lift_area="${lift_area}" lift_air_density="${lift_air_density}" lift_cp="${lift_cp}">
     <extra_ardupilot_plugin_settings>
-      <xacro:extra_channel channel="6" _type="POSITION" _multiplier="1" _jointName="fire_trigger_servo_joint"
+      <xacro:extra_channel channel="6" _type="POSITION" _multiplier="2" _jointName="fire_trigger_servo_joint"
                                           _offset="0" _p_gain="1" _i_gain="0" _d_gain="0"
                                           _i_max="0" _i_min="0" _cmd_max="2.5" _cmd_min="-2.5"/>
@@ -101,5 +102,5 @@
     <parent link="base_link"/>
     <child link="fire_trigger_servo_link"/>
-    <origin xyz="0 0 -0.45" rpy="0 0 0"/>
+    <origin xyz="-0.08 0.015 -0.412" rpy="0 0 0"/>
     <axis xyz="0 0 1"/>
     <limit effort="10000" velocity="4" lower="${pi * -0.5}" upper="${pi * 0.5}"/>
@@ -119,4 +120,10 @@
     <self_collide>0</self_collide>
   </gazebo>
+  <joint name="M16_joint" type="fixed">
+    <parent link="base_link"/>
+    <child link="M16_link"/>
+    <origin xyz="0.05 0 -0.35" rpy="0 0 0"/>
+  </joint>
+  <xacro:link_creator_i link_name="M16_link" pose_xyz="0 0 0" pose_rpy="0 0 0" mesh_path="${M16_mesh}" scale_xyz="1 1 1" mass="1.9" center_mass_xyz="0 0 -0.025" iner_box_scale_xyz="0.75 0.055 0.14"/>
 </robot>
 <!--

File: xacros/link_macros.xacro (robot description, xacro)
@@ -49,5 +49,5 @@
         </xacro:link_creator_foundation>
     </xacro:macro>
-    <xacro:macro name="link_creator_i_foundation" params="link_name pose_xyz pose_rpy mesh_path:='Box' col_mesh_path:='None' scale_xyz col_scale_xyz:='None' seperate_collider_xyzrpy:='None' center_mass_xyz:='0 0 0' mass iner:='None' **extra_collision **extra_visual **extra_settings">
+    <xacro:macro name="link_creator_i_foundation" params="link_name pose_xyz pose_rpy mesh_path:='Box' col_mesh_path:='None' scale_xyz col_scale_xyz:='None' seperate_collider_xyzrpy:='None' center_mass_xyz:='0 0 0' mass iner:='None' iner_box_scale_xyz:='None' **extra_collision **extra_visual **extra_settings">
         <xacro:link_creator_foundation link_name="${link_name}" pose_xyz="${pose_xyz}" pose_rpy="${pose_rpy}" mesh_path="${mesh_path}" scale_xyz="${scale_xyz}">
             <extra_visual><xacro:insert_block name="extra_visual"/></extra_visual>
@@ -82,6 +82,12 @@
                 </collision>
                 <xacro:if value="${str(iner) == 'None'}">
-                    <xacro:property name="scale_xyz_list" value="${scale_xyz.split(' ')}" />
-                    <xacro:inertial_box mass="${mass}" x="${float(scale_xyz_list[0])}" y="${float(scale_xyz_list[1])}" z="${float(scale_xyz_list[2])}" xyz="${center_mass_xyz}" rpy="0 0 0"/>
+                    <xacro:if value="${str(iner_box_scale_xyz) == 'None'}">
+                        <xacro:property name="scale_xyz_list" value="${scale_xyz.split(' ')}" />
+                        <xacro:inertial_box mass="${mass}" x="${float(scale_xyz_list[0])}" y="${float(scale_xyz_list[1])}" z="${float(scale_xyz_list[2])}" xyz="${center_mass_xyz}" rpy="0 0 0"/>
+                    </xacro:if>
+                    <xacro:if value="${str(iner_box_scale_xyz) != 'None'}">
+                        <xacro:property name="iner_box_scale_xyz_list" value="${iner_box_scale_xyz.split(' ')}" />
+                        <xacro:inertial_box mass="${mass}" x="${float(iner_box_scale_xyz_list[0])}" y="${float(iner_box_scale_xyz_list[1])}" z="${float(iner_box_scale_xyz_list[2])}" xyz="${center_mass_xyz}" rpy="0 0 0"/>
+                    </xacro:if>
                 </xacro:if>
                 <xacro:if value="${str(iner) != 'None'}">
@@ -97,6 +103,6 @@
         </xacro:link_creator_foundation>
     </xacro:macro>
-    <xacro:macro name="link_creator_i" params="link_name pose_xyz pose_rpy mesh_path:='Box' col_mesh_path:='None' scale_xyz col_scale_xyz:='None' seperate_collider_xyzrpy:='None' center_mass_xyz:='0 0 0' mass iner:='None'">
-        <xacro:link_creator_i_foundation link_name="${link_name}" pose_xyz="${pose_xyz}" pose_rpy="${pose_rpy}" mesh_path="${mesh_path}" col_mesh_path="${col_mesh_path}" scale_xyz="${scale_xyz}" col_scale_xyz="${col_scale_xyz}" seperate_collider_xyzrpy="${seperate_collider_xyzrpy}" center_mass_xyz="${center_mass_xyz}" mass="${mass}" iner="${iner}">
+    <xacro:macro name="link_creator_i" params="link_name pose_xyz pose_rpy mesh_path:='Box' col_mesh_path:='None' scale_xyz col_scale_xyz:='None' seperate_collider_xyzrpy:='None' center_mass_xyz:='0 0 0' mass iner:='None' iner_box_scale_xyz:='None'">
+        <xacro:link_creator_i_foundation link_name="${link_name}" pose_xyz="${pose_xyz}" pose_rpy="${pose_rpy}" mesh_path="${mesh_path}" col_mesh_path="${col_mesh_path}" scale_xyz="${scale_xyz}" col_scale_xyz="${col_scale_xyz}" seperate_collider_xyzrpy="${seperate_collider_xyzrpy}" center_mass_xyz="${center_mass_xyz}" mass="${mass}" iner="${iner}" iner_box_scale_xyz="${iner_box_scale_xyz}">
             <extra_collision/>
             <extra_visual/>

Commit message: ros2 node for publishing force is working(apply_force_node.cpp) but the ApplyForcePlugin.cpp for gazebo is not

File: models/copterPIX/robot.urdf.xacro (robot description, xacro)
@@ -5,5 +5,5 @@
   <xacro:property name="prop_cw_mesh" value="$(find drone)/meshes/iris_prop_cw.dae"/>
   <xacro:property name="prop_ccw_mesh" value="$(find drone)/meshes/iris_prop_ccw.dae"/>
-  <xacro:property name="M16_mesh" value="$(find drone)/meshes/M16.stl"/>
+  <xacro:property name="m16_mesh" value="$(find drone)/meshes/M16.stl"/>
 <!--
   <xacro:property name="ixx" value="${373162267137.9 / g_mms_to_kg_ms}"/>  these values are not valid, they are stupid wrong
@@ -120,10 +120,15 @@
     <self_collide>0</self_collide>
   </gazebo>
-  <joint name="M16_joint" type="fixed">
+  <joint name="m16_joint" type="fixed">
     <parent link="base_link"/>
-    <child link="M16_link"/>
+    <child link="m16_link"/>
     <origin xyz="0.05 0 -0.35" rpy="0 0 0"/>
   </joint>
-  <xacro:link_creator_i link_name="M16_link" pose_xyz="0 0 0" pose_rpy="0 0 0" mesh_path="${M16_mesh}" scale_xyz="1 1 1" mass="1.9" center_mass_xyz="0 0 -0.025" iner_box_scale_xyz="0.75 0.055 0.14"/>
+  <xacro:link_creator_i link_name="m16_link" pose_xyz="0 0 0" pose_rpy="0 0 0" mesh_path="${m16_mesh}" scale_xyz="1 1 1" mass="1.9" center_mass_xyz="0 0 -0.025" iner_box_scale_xyz="0.75 0.055 0.14"/>
+  <!-- <gazebo>
+    <plugin name="apply_force_plugin" filename="libApplyForcePlugin.so">
+      <link_name>base_link</link_name>
+    </plugin>
+  </gazebo> -->
 </robot>
 <!--

Commit message: added drone_gazebo_plugin made by me for applying force on the drone. everything working! also .gitignore added

File: models/copterPIX/robot.urdf.xacro (robot description, xacro)
@@ -33,6 +33,4 @@
   <xacro:property name="arm_mesh" value="${hex_mesh}"/>
   <xacro:property name="prop_size_multiplier" value="2.34"/>
-  <xacro:property name="cylinder_d" value="0.55"/>
-  <xacro:property name="cylinder_l" value="0.02"/>
   <xacro:property name="a_mass" value="0.5"/>
   <xacro:property name="a_iner" value="None"/>
@@ -48,4 +46,5 @@
   <xacro:property name="ardu_cmd_max" value="2.5"/>
   <xacro:property name="ardu_cmd_min" value="-2.5"/>
+  <xacro:property name="prop_col_scale_xyz" value="0.55 0.06 0.03"/>
   <xacro:property name="number_of_blades" value="2"/>
   <xacro:property name="lift_a0" value="0.3"/>
@@ -65,6 +64,5 @@
                      dis_from_center="${dis_from_center}" length="${length}" diameter="${diameter}"
                      arm_incline_angle="${arm_incline_angle}" rotor_dis_from_arm="${rotor_dis_from_arm}" arm_mesh="${arm_mesh}" prop_size_multiplier="${prop_size_multiplier}"
-                     cylinder_d="${cylinder_d}" cylinder_l="${cylinder_l}" a_mass="${a_mass}" a_iner="${a_iner}"
-                     r_mass="${r_mass}"  r_iner="${r_iner}"
+                     prop_col_scale_xyz="${prop_col_scale_xyz}" a_mass="${a_mass}" a_iner="${a_iner}" r_mass="${r_mass}"  r_iner="${r_iner}"
                      ardu_multiplier="${ardu_multiplier}" ardu_offset="${ardu_offset}"
                      ardu_p_gain="${ardu_p_gain}" ardu_i_gain="${ardu_i_gain}" ardu_d_gain="${ardu_d_gain}"
@@ -74,5 +72,5 @@
                      lift_area="${lift_area}" lift_air_density="${lift_air_density}" lift_cp="${lift_cp}">
     <extra_ardupilot_plugin_settings>
-      <xacro:extra_channel channel="6" _type="POSITION" _multiplier="2" _jointName="fire_trigger_servo_joint"
+      <xacro:extra_channel channel="6" _type="POSITION" _multiplier="-200" _jointName="fire_trigger_servo_joint"
                                           _offset="0" _p_gain="1" _i_gain="0" _d_gain="0"
                                           _i_max="0" _i_min="0" _cmd_max="2.5" _cmd_min="-2.5"/>
@@ -102,5 +100,5 @@
     <parent link="base_link"/>
     <child link="fire_trigger_servo_link"/>
-    <origin xyz="-0.08 0.015 -0.412" rpy="0 0 0"/>
+    <origin xyz="-0.08 -0.015 -0.412" rpy="0 0 0"/>
     <axis xyz="0 0 1"/>
     <limit effort="10000" velocity="4" lower="${pi * -0.5}" upper="${pi * 0.5}"/>
@@ -120,16 +118,29 @@
     <self_collide>0</self_collide>
   </gazebo>
+  <xacro:property name="m16_position" value="0.05 0 -0.35"/>
   <joint name="m16_joint" type="fixed">
     <parent link="base_link"/>
     <child link="m16_link"/>
-    <origin xyz="0.05 0 -0.35" rpy="0 0 0"/>
+    <origin xyz="${m16_position}" rpy="0 0 0"/>
   </joint>
   <xacro:link_creator_i link_name="m16_link" pose_xyz="0 0 0" pose_rpy="0 0 0" mesh_path="${m16_mesh}" scale_xyz="1 1 1" mass="1.9" center_mass_xyz="0 0 -0.025" iner_box_scale_xyz="0.75 0.055 0.14"/>
-  <!-- <gazebo>
-    <plugin name="gazebo_ros_control" filename="libgazebo_ros_control.so">
-        <robotNamespace>/robot_namespace</robotNamespace>
-        <robotParam>/robot_description</robotParam>
+  <xacro:property name="m16_position_list" value="${m16_position.split(' ')}" />
+  <xacro:property name="m16_position_x" value="${m16_position_list[0]}" />
+  <xacro:property name="m16_position_y" value="${m16_position_list[1]}" />
+  <xacro:property name="m16_position_z" value="${m16_position_list[2]}" />
+  <gazebo>
+    <plugin name="ForcePlugin" filename="libForcePlugin.so">
+      <trigger_joint>fire_trigger_servo_joint</trigger_joint>
+      <link_to_apply_force>root_link</link_to_apply_force> <!--change later to the m16_link when gimbal will be ready.-->
+      <apply_force_duration>0.03</apply_force_duration> <!--apply froce for 30ms-->
+      <trigger_angle_deg>15</trigger_angle_deg>
+      <force_x>-2000</force_x>
+      <force_y>0</force_y>
+      <force_z>0</force_z>
+      <position_x>${m16_position_x}</position_x>
+      <position_y>${m16_position_y}</position_y>
+      <position_z>${m16_position_z}</position_z>
     </plugin>
-  </gazebo> -->
+  </gazebo>
 </robot>
 <!--

File: models/iris/robot.urdf.xacro (robot description, xacro)
@@ -23,6 +23,4 @@
   <xacro:property name="arm_mesh" value="${hex_mesh}"/>
   <xacro:property name="prop_size_multiplier" value="1"/>
-  <xacro:property name="cylinder_d" value="0.25"/>
-  <xacro:property name="cylinder_l" value="0.02"/>
   <xacro:property name="a_mass" value="0.08"/>
   <xacro:property name="a_iner" value="None"/>
@@ -38,4 +36,5 @@
   <xacro:property name="ardu_cmd_max" value="2.5"/>
   <xacro:property name="ardu_cmd_min" value="-2.5"/>
+    <xacro:property name="prop_col_scale_xyz" value="0.28 0.03 0.01"/>
   <xacro:property name="number_of_blades" value="2"/>
   <xacro:property name="lift_a0" value="0.3"/>
@@ -55,6 +54,5 @@
                      dis_from_center="${dis_from_center}" length="${length}" diameter="${diameter}"
                      arm_incline_angle="${arm_incline_angle}" rotor_dis_from_arm="${rotor_dis_from_arm}" arm_mesh="${arm_mesh}" prop_size_multiplier="${prop_size_multiplier}"
-                     cylinder_d="${cylinder_d}" cylinder_l="${cylinder_l}" a_mass="${a_mass}" a_iner="${a_iner}"
-                     r_mass="${r_mass}"  r_iner="${r_iner}"
+                     prop_col_scale_xyz="${prop_col_scale_xyz}" a_mass="${a_mass}" a_iner="${a_iner}" r_mass="${r_mass}"  r_iner="${r_iner}"
                      ardu_multiplier="${ardu_multiplier}" ardu_offset="${ardu_offset}"
                      ardu_p_gain="${ardu_p_gain}" ardu_i_gain="${ardu_i_gain}" ardu_d_gain="${ardu_d_gain}"

File: xacros/arm_macro.xacro (robot description, xacro)
@@ -3,5 +3,5 @@
     <xacro:include filename="link_macros.xacro"/>
     <xacro:macro name="drone_arm" params="num parent_link dis_from_center length diameter arm_incline_angle rotor_dis_from_arm arm_mesh prop_mesh cw
-                                          prop_size_multiplier cylinder_d cylinder_l a_mass a_iner:='None' r_mass r_iner angle
+                                          prop_size_multiplier prop_col_scale_xyz a_mass a_iner:='None' r_mass r_iner angle
                                           number_of_blades lift_a0 lift_alpha_stall lift_cla lift_cda lift_cma lift_cla_stall lift_sda_stall lift_cma_stall
                                           lift_area lift_air_density lift_cp">
@@ -31,6 +31,6 @@
             </physics>
         </gazebo>
-        <xacro:link_creator_i_foundation link_name="${prop_link}" pose_xyz="0 0 0" pose_rpy="0 0 0" mesh_path="${prop_mesh}" col_mesh_path="Cylinder"
-                                         scale_xyz="${prop_size_multiplier} ${prop_size_multiplier} ${prop_size_multiplier}" col_scale_xyz="${cylinder_d} 0 ${cylinder_l}"
+        <xacro:link_creator_i_foundation link_name="${prop_link}" pose_xyz="0 0 0" pose_rpy="0 0 0" mesh_path="${prop_mesh}" col_mesh_path="Box"
+                                         scale_xyz="${prop_size_multiplier} ${prop_size_multiplier} ${prop_size_multiplier}" col_scale_xyz="${prop_col_scale_xyz}"
                                          seperate_collider_xyzrpy="None"
                                          center_mass_xyz="0 0 0" mass="${r_mass}"  iner="${r_iner}">

File: xacros/drone_maker.xacro (robot description, xacro)
@@ -7,5 +7,5 @@
                                             number_of_arms arm_angles cws prop_meshs
                                             dis_from_center length diameter arm_incline_angle:='0' rotor_dis_from_arm arm_mesh prop_size_multiplier
-                                            cylinder_d cylinder_l a_mass a_iner:='None' r_mass r_iner
+                                            prop_col_scale_xyz a_mass a_iner:='None' r_mass r_iner
                                             ardu_multiplier ardu_offset ardu_p_gain ardu_i_gain ardu_d_gain
                                             ardu_i_max ardu_i_min ardu_cmd_max ardu_cmd_min
@@ -37,5 +37,5 @@
                                 arm_incline_angle="${arm_incline_angle * deg_to_rad}" rotor_dis_from_arm="${rotor_dis_from_arm}" arm_mesh="${arm_mesh}"
                                 prop_mesh="${prop_mesh_list[counter]}" cw="${cw_list[counter]}"
-                                prop_size_multiplier="${prop_size_multiplier}" cylinder_d="${cylinder_d}" cylinder_l="${cylinder_l}"
+                                prop_size_multiplier="${prop_size_multiplier}" prop_col_scale_xyz="${prop_col_scale_xyz}"
                                 a_mass="${a_mass}" a_iner="${a_iner}" r_mass="${r_mass}" r_iner="${r_iner}" angle="${float(arm_angle_list[counter]) * deg_to_rad}"
                                 number_of_blades="${number_of_blades}"

File: xacros/link_macros.xacro (robot description, xacro)
@@ -102,4 +102,10 @@
             </extra_settings>
         </xacro:link_creator_foundation>
+        <!-- <gazebo reference="${link_name}">
+            <ode>
+                <mu1 value="1000000"/>
+                <mu2 value="1000000"/>
+            </ode>
+        </gazebo> -->
     </xacro:macro>
     <xacro:macro name="link_creator_i" params="link_name pose_xyz pose_rpy mesh_path:='Box' col_mesh_path:='None' scale_xyz col_scale_xyz:='None' seperate_collider_xyzrpy:='None' center_mass_xyz:='0 0 0' mass iner:='None' iner_box_scale_xyz:='None'">

Commit message: still working on the harmonic!

File: models/copterPIX/robot.urdf.xacro (robot description, xacro)
@@ -2,8 +2,12 @@
 <robot name="copterPIX" xmlns:xacro="http://www.ros.org/wiki/xacro">
   <xacro:include filename="$(find drone)/xacros/drone_maker.xacro"/>
-  <xacro:property name="hex_mesh" value="$(find drone)/meshes/hexagonal_prism_height_1_outer_diameter_1.stl"/>
+  <!-- <xacro:property name="hex_mesh" value="$(find drone)/meshes/hexagonal_prism_height_1_outer_diameter_1.stl"/>
   <xacro:property name="prop_cw_mesh" value="$(find drone)/meshes/iris_prop_cw.dae"/>
   <xacro:property name="prop_ccw_mesh" value="$(find drone)/meshes/iris_prop_ccw.dae"/>
-  <xacro:property name="m16_mesh" value="$(find drone)/meshes/M16.stl"/>
+  <xacro:property name="m16_mesh" value="$(find drone)/meshes/M16.stl"/> -->
+  <xacro:property name="hex_mesh" value="package://drone/meshes/hexagonal_prism_height_1_outer_diameter_1.stl"/>
+  <xacro:property name="prop_cw_mesh" value="package://drone/meshes/iris_prop_cw.dae"/>
+  <xacro:property name="prop_ccw_mesh" value="package://drone/meshes/iris_prop_ccw.dae"/>
+  <xacro:property name="m16_mesh" value="package://drone/meshes/M16.stl"/>
 <!--
   <xacro:property name="ixx" value="${373162267137.9 / g_mms_to_kg_ms}"/>  these values are not valid, they are stupid wrong
