Commit message: made the xacro compatible with both classic and harmonic and made two launch files each for different gazebo types.

File: models/copterPIX/robot.urdf.xacro (robot description, xacro)
@@ -1,13 +1,11 @@
 <?xml version="1.0" ?>
 <robot name="copterPIX" xmlns:xacro="http://www.ros.org/wiki/xacro">
+  <!--this value is changed by the launch script.-->
+  <xacro:property name="using_gazebo_classic" value="0"/>
   <xacro:include filename="$(find drone)/xacros/drone_maker.xacro"/>
-  <!-- <xacro:property name="hex_mesh" value="$(find drone)/meshes/hexagonal_prism_height_1_outer_diameter_1.stl"/>
+  <xacro:property name="hex_mesh" value="$(find drone)/meshes/hexagonal_prism_height_1_outer_diameter_1.stl"/>
   <xacro:property name="prop_cw_mesh" value="$(find drone)/meshes/iris_prop_cw.dae"/>
   <xacro:property name="prop_ccw_mesh" value="$(find drone)/meshes/iris_prop_ccw.dae"/>
-  <xacro:property name="m16_mesh" value="$(find drone)/meshes/M16.stl"/> -->
-  <xacro:property name="hex_mesh" value="package://drone/meshes/hexagonal_prism_height_1_outer_diameter_1.stl"/>
-  <xacro:property name="prop_cw_mesh" value="package://drone/meshes/iris_prop_cw.dae"/>
-  <xacro:property name="prop_ccw_mesh" value="package://drone/meshes/iris_prop_ccw.dae"/>
-  <xacro:property name="m16_mesh" value="package://drone/meshes/M16.stl"/>
+  <xacro:property name="m16_mesh" value="$(find drone)/meshes/M16.stl"/>
 <!--
   <xacro:property name="ixx" value="${373162267137.9 / g_mms_to_kg_ms}"/>  these values are not valid, they are stupid wrong
@@ -63,5 +61,5 @@
   <xacro:property name="lift_air_density" value="1.2041"/>
   <xacro:property name="lift_cp" value="0.2"/>
-  <xacro:drone_maker base_mesh="${base_mesh}" base_pose_xyz ="${base_pose_xyz}" base_pose_rpy="${base_pose_rpy}" base_scale_xyz="${base_scale_xyz}"
+  <xacro:drone_maker using_gazebo_classic="${using_gazebo_classic}" base_mesh="${base_mesh}" base_pose_xyz ="${base_pose_xyz}" base_pose_rpy="${base_pose_rpy}" base_scale_xyz="${base_scale_xyz}"
                      base_center_of_mass="${base_center_of_mass}" base_mass="${base_mass}" base_iner="${base_iner}"
                      number_of_arms="${number_of_arms}" arm_angles="${arm_angles}" cws="${cws}" prop_meshs="${prop_meshs}"
@@ -76,5 +74,5 @@
                      lift_area="${lift_area}" lift_air_density="${lift_air_density}" lift_cp="${lift_cp}">
     <extra_ardupilot_plugin_settings>
-      <xacro:extra_channel channel="6" _type="POSITION" _multiplier="-200" _jointName="fire_trigger_servo_joint"
+      <xacro:extra_channel using_gazebo_classic="${using_gazebo_classic}" channel="6" _type="POSITION" _multiplier="-200" _jointName="fire_trigger_servo_joint"
                                           _offset="0" _p_gain="1" _i_gain="0" _d_gain="0"
                                           _i_max="0" _i_min="0" _cmd_max="2.5" _cmd_min="-2.5"/>
@@ -134,16 +132,34 @@
   <xacro:property name="m16_position_z" value="${m16_position_list[2]}" />
   <gazebo>
-    <plugin name="ForcePlugin" filename="libForcePlugin.so">
-      <trigger_joint>fire_trigger_servo_joint</trigger_joint>
-      <link_to_apply_force>root_link</link_to_apply_force> <!--change later to the m16_link when gimbal will be ready.-->
-      <apply_force_duration>0.03</apply_force_duration> <!--apply froce for 30ms-->
-      <trigger_angle_deg>15</trigger_angle_deg>
-      <force_x>-2000</force_x>
-      <force_y>0</force_y>
-      <force_z>0</force_z>
-      <position_x>${m16_position_x}</position_x>
-      <position_y>${m16_position_y}</position_y>
-      <position_z>${m16_position_z}</position_z>
-    </plugin>
+    <xacro:if value="${using_gazebo_classic}">
+      <!--for gazebo classic-->
+      <plugin name="ForcePlugin" filename="libForcePlugin.so">
+        <trigger_joint>fire_trigger_servo_joint</trigger_joint>
+        <link_to_apply_force>root_link</link_to_apply_force> change later to the m16_link when gimbal will be ready.
+        <apply_force_duration>0.03</apply_force_duration> apply froce for 30ms
+        <trigger_angle_deg>15</trigger_angle_deg>
+        <force_x>-2000</force_x>
+        <force_y>0</force_y>
+        <force_z>0</force_z>
+        <position_x>${m16_position_x}</position_x>
+        <position_y>${m16_position_y}</position_y>
+        <position_z>${m16_position_z}</position_z>
+      </plugin>
+    </xacro:if>
+    <xacro:unless value="${using_gazebo_classic}">
+      <!--for gazebo harmonic-->
+      <plugin name="ForcePlugin" filename="ForcePlugin">
+        <trigger_joint>fire_trigger_servo_joint</trigger_joint>
+        <link_to_apply_force>root_link</link_to_apply_force> change later to the m16_link when gimbal will be ready.
+        <apply_force_duration>0.03</apply_force_duration> apply froce for 30ms
+        <trigger_angle_deg>15</trigger_angle_deg>
+        <force_x>-2000</force_x>
+        <force_y>0</force_y>
+        <force_z>0</force_z>
+        <position_x>${m16_position_x}</position_x>
+        <position_y>${m16_position_y}</position_y>
+        <position_z>${m16_position_z}</position_z>
+      </plugin>
+    </xacro:unless>
   </gazebo>
 </robot>

File: models/iris/robot.urdf.xacro (robot description, xacro)
@@ -1,4 +1,6 @@
 <?xml version="1.0" ?>
 <robot name="copterPIX" xmlns:xacro="http://www.ros.org/wiki/xacro">
+  <!--this value is changed by the launch script.-->
+  <xacro:property name="using_gazebo_classic" value="0"/>
   <xacro:include filename="$(find drone)/xacros/drone_maker.xacro"/>
   <xacro:property name="hex_mesh" value="$(find drone)/meshes/hexagonal_prism_height_1_outer_diameter_1.stl"/>
@@ -49,5 +51,5 @@
   <xacro:property name="lift_air_density" value="1.2041"/>
   <xacro:property name="lift_cp" value="0.084"/>
-  <xacro:drone_maker base_mesh="${base_mesh}" base_pose_xyz ="${base_pose_xyz}" base_pose_rpy="${base_pose_rpy}" base_scale_xyz="${base_scale_xyz}"
+ <xacro:drone_maker using_gazebo_classic="${using_gazebo_classic}" base_mesh="${base_mesh}" base_pose_xyz ="${base_pose_xyz}" base_pose_rpy="${base_pose_rpy}" base_scale_xyz="${base_scale_xyz}"
                      base_center_of_mass="${base_center_of_mass}" base_mass="${base_mass}" base_iner="${base_iner}"
                      number_of_arms="${number_of_arms}" arm_angles="${arm_angles}" cws="${cws}" prop_meshs="${prop_meshs}"
@@ -61,6 +63,5 @@
                      lift_cma="${lift_cma}" lift_cla_stall="${lift_cla_stall}" lift_sda_stall="${lift_sda_stall}" lift_cma_stall="${lift_cma_stall}"
                      lift_area="${lift_area}" lift_air_density="${lift_air_density}" lift_cp="${lift_cp}">
-    <extra_ardupilot_plugin_settings>
-    </extra_ardupilot_plugin_settings>
+    <extra_ardupilot_plugin_settings/>
   </xacro:drone_maker>
 </robot>

File: xacros/ardupilot_plugin.xacro (robot description, xacro)
@@ -1,61 +1,179 @@
 <?xml version="1.0" ?>
 <robot xmlns:xacro="http://www.ros.org/wiki/xacro">
-    <xacro:macro name="extra_channel" params="channel _type _multiplier _jointName _offset _p_gain _i_gain _d_gain
+    <xacro:macro name="extra_channel" params="using_gazebo_classic channel _type _multiplier _jointName _useForce_offset _servo_max='1900' _servo_min='1100' _p_gain _i_gain _d_gain
                                                           _i_max _i_min _cmd_max _cmd_min">
-        <control channel="${channel}">
-            <type>${_type}</type>
-            <multiplier>${_multiplier}</multiplier>
-            <jointName>${_jointName}</jointName>
-            <offset>${_offset}</offset>
-            <p_gain>${_p_gain}</p_gain>
-            <i_gain>${_i_gain}</i_gain>
-            <d_gain>${_d_gain}</d_gain>
-            <i_max>${_i_max}</i_max>
-            <i_min>${_i_min}</i_min>
-            <cmd_max>${_cmd_max}</cmd_max>
-            <cmd_min>${_cmd_min}</cmd_min>
-            <controlVelocitySlowdownSim>1</controlVelocitySlowdownSim>
-        </control>
+        <xacro:if value="${using_gazebo_classic}" />
+            <control channel="${channel}">
+                <type>${_type}</type>
+                <multiplier>${_multiplier}</multiplier>
+                <jointName>${_jointName}</jointName>
+                <offset>${_offset}</offset>
+                <p_gain>${_p_gain}</p_gain>
+                <i_gain>${_i_gain}</i_gain>
+                <d_gain>${_d_gain}</d_gain>
+                <i_max>${_i_max}</i_max>
+                <i_min>${_i_min}</i_min>
+                <cmd_max>${_cmd_max}</cmd_max>
+                <cmd_min>${_cmd_min}</cmd_min>
+                <controlVelocitySlowdownSim>1</controlVelocitySlowdownSim>
+            </control>
+        </xacro:if>
+        <xacro:unless value="${using_gazebo_classic}" />
+            <control channel="${channel}">
+                <!--
+                    incoming control command [0, 1]
+                    so offset it by 0 to get [0, 1]
+                    and divide max target by 1.
+                    offset = 0
+                    multiplier = 838 max rpm / 1 = 838
+                -->
+                <!--
+                    SERVO<N>_FUNCTION   ->      70 (Throttle)
+                    SERVO<N>_MAX        ->      _servo_max
+                    SERVO<N>_MIN        ->      _servo_min
+                    SERVO<N>_REVERSED   ->      absolute value of _multiplier
+                    SERVO<N>_TRIM       ->
+                -->
+                <!--
+                    The <useForce> tag determines how control commands are applied to the joint.
+                    When set to 1, the control commands are applied as forces (effort),
+                    resulting in more realistic physical interactions; when set to 0,
+                    the commands are applied directly as velocities or positions.
+                -->
+                <type>${_type}</type>
+                <multiplier>${_multiplier}</multiplier>
+                <jointName>${_jointName}</jointName>
+                <useForce>${_useForce}</useForce>
+                <offset>${_offset}</offset>
+                <servo_max>${_servo_max}</servo_max>
+                <servo_min>${_servo_min}</servo_min>
+                <p_gain>${_p_gain}</p_gain>
+                <i_gain>${_i_gain}</i_gain>
+                <d_gain>${_d_gain}</d_gain>
+                <i_max>${_i_max}</i_max>
+                <i_min>${_i_min}</i_min>
+                <cmd_max>${_cmd_max}</cmd_max>
+                <cmd_min>${_cmd_min}</cmd_min>
+                <controlVelocitySlowdownSim>1</controlVelocitySlowdownSim>
+            </control>
+        </xacro:unless>
     </xacro:macro>
-    <xacro:macro name="ardupilot_plugin" params="number_of_arms multiplier cws offset p_gain i_gain d_gain i_max i_min cmd_max cmd_min **extra_ardupilot_plugin_settings">
+    <xacro:macro name="ardupilot_plugin" params="using_gazebo_classic number_of_arms multiplier cws offset p_gain i_gain d_gain i_max i_min cmd_max cmd_min **extra_ardupilot_plugin_settings servo_max='1900' servo_min='1100'">
         <xacro:property name="cw_list" value="${cws.split(' ')}" />
         <gazebo>
-            <plugin name="arducopter_plugin" filename="libArduPilotPlugin.so">
-                <fdm_addr>127.0.0.1</fdm_addr>
-                <fdm_port_in>9002</fdm_port_in>
-                <fdm_port_out>9003</fdm_port_out>
-                <modelXYZToAirplaneXForwardZDown>0 0 0 ${pi} 0 0</modelXYZToAirplaneXForwardZDown>
-                <gazeboXYZToNED>0 0 0 ${pi} 0 0</gazeboXYZToNED>
-                <imuName>imu_link::imu_sensor</imuName>
-                <connectionTimeoutMaxCount>5</connectionTimeoutMaxCount>
-                <xacro:macro name="create_arms" params="i">
-                    <xacro:if value="${i > 0}">
-                        <!-- Here define the arm -->
-                        <xacro:property name="counter" value="${number_of_arms - i}" />
-                        <xacro:property name="jointName" value="rotor_joint_${str(counter)}" />
-                        <xacro:property name="directed_multiplier" value="${multiplier * ((int(cw_list[counter]) * (-2)) + 1)}" />
-                        <control channel="${counter}">
-                            <type>VELOCITY</type>
-                            <multiplier>${directed_multiplier}</multiplier>
-                            <jointName>${jointName}</jointName>
-                            <offset>${offset}</offset>
-                            <p_gain>${p_gain}</p_gain>
-                            <i_gain>${i_gain}</i_gain>
-                            <d_gain>${d_gain}</d_gain>
-                            <i_max>${i_max}</i_max>
-                            <i_min>${i_min}</i_min>
-                            <cmd_max>${cmd_max}</cmd_max>
-                            <cmd_min>${cmd_min}</cmd_min>
-                            <controlVelocitySlowdownSim>1</controlVelocitySlowdownSim>
-                        </control>
-                        <!-- Recursively call the macro with a decremented count -->
-                        <xacro:create_arms i="${i - 1}"/>
-                    </xacro:if>
-                </xacro:macro>
-                <!-- Initial call to the macro with the desired number of joints -->
-                <xacro:create_arms i="${int(number_of_arms)}"/>
-                <!-- end Define arms! -->
-                <xacro:insert_block name="extra_ardupilot_plugin_settings"/>
-            </plugin>
+            <xacro:if value="${using_gazebo_classic}" />
+                <plugin name="arducopter_plugin" filename="libArduPilotPlugin.so">
+                    <fdm_addr>127.0.0.1</fdm_addr>
+                    <fdm_port_in>9002</fdm_port_in>
+                    <fdm_port_out>9003</fdm_port_out>
+                    <modelXYZToAirplaneXForwardZDown>0 0 0 ${pi} 0 0</modelXYZToAirplaneXForwardZDown>
+                    <gazeboXYZToNED>0 0 0 ${pi} 0 0</gazeboXYZToNED>
+                    <imuName>imu_link::imu_sensor</imuName>
+                    <connectionTimeoutMaxCount>5</connectionTimeoutMaxCount>
+                    <xacro:macro name="create_arms" params="i">
+                        <xacro:if value="${i > 0}">
+                            <!-- Here define the arm -->
+                            <xacro:property name="counter" value="${number_of_arms - i}" />
+                            <xacro:property name="jointName" value="rotor_joint_${str(counter)}" />
+                            <xacro:property name="directed_multiplier" value="${multiplier * ((int(cw_list[counter]) * (-2)) + 1)}" />
+                            <control channel="${counter}">
+                                <type>VELOCITY</type>
+                                <multiplier>${directed_multiplier}</multiplier>
+                                <jointName>${jointName}</jointName>
+                                <offset>${offset}</offset>
+                                <p_gain>${p_gain}</p_gain>
+                                <i_gain>${i_gain}</i_gain>
+                                <d_gain>${d_gain}</d_gain>
+                                <i_max>${i_max}</i_max>
+                                <i_min>${i_min}</i_min>
+                                <cmd_max>${cmd_max}</cmd_max>
+                                <cmd_min>${cmd_min}</cmd_min>
+                                <controlVelocitySlowdownSim>1</controlVelocitySlowdownSim>
+                            </control>
+                            <!-- Recursively call the macro with a decremented count -->
+                            <xacro:create_arms i="${i - 1}"/>
+                        </xacro:if>
+                    </xacro:macro>
+                    <!-- Initial call to the macro with the desired number of joints -->
+                    <xacro:create_arms i="${int(number_of_arms)}"/>
+                    <!-- end Define arms! -->
+                    <xacro:insert_block name="extra_ardupilot_plugin_settings"/>
+                </plugin>
+            </xacro:if>
+            <xacro:unless value="${using_gazebo_classic}" />
+                <plugin name="ArduPilotPlugin" filename="ArduPilotPlugin">
+                    <fdm_addr>127.0.0.1</fdm_addr>
+                    <fdm_port_in>9002</fdm_port_in>
+                    <!-- <fdm_port_out>9003</fdm_port_out> Param <fdm_port_out> is deprecated, connection is auto detected-->
+                    <connectionTimeoutMaxCount>5</connectionTimeoutMaxCount>
+                    <!--lock_step: whether or not to wait for the ardupilot sitl's packets and stop the frame till the packet is recieved.
+                    If the sitl laggs, simulation will pause till it resumes. I do not want that so I set it to 0.-->
+                    <lock_step>0</lock_step>
+                    <!-- Frame conventions
+                        modelXYZToAirplaneXForwardZDown:
+                        - transforms body frame from orientation in Gazebo to NED
+                        gazeboXYZToNED
+                        - transforms world from Gazebo convention xyz = N -E -D
+                            to ArduPilot convention xyz = NED
+                        Zephyr is oriented x-left, y-back, z-up
+                    -->
+                    <!-- <modelXYZToAirplaneXForwardZDown degrees="true">0 0 0 180 0 -90</modelXYZToAirplaneXForwardZDown>
+                    <gazeboXYZToNED degrees="true">0 0 0 180 0 90</gazeboXYZToNED> -->
+                    <modelXYZToAirplaneXForwardZDown degrees="true">0 0 0 180 0 0</modelXYZToAirplaneXForwardZDown>
+                    <gazeboXYZToNED degrees="true">0 0 0 180 0 0</gazeboXYZToNED>
+                    <imuName>imu_link::imu_sensor</imuName>
+                    <connectionTimeoutMaxCount>5</connectionTimeoutMaxCount>
+                    <xacro:macro name="create_arms" params="i">
+                        <xacro:if value="${i > 0}">
+                            <!-- Here define the arm -->
+                            <xacro:property name="counter" value="${number_of_arms - i}" />
+                            <xacro:property name="jointName" value="rotor_joint_${str(counter)}" />
+                            <xacro:property name="directed_multiplier" value="${multiplier * ((int(cw_list[counter]) * (-2)) + 1)}" />
+                            <control channel="${counter}">
+                                <!--
+                                    incoming control command [0, 1]
+                                    so offset it by 0 to get [0, 1]
+                                    and divide max target by 1.
+                                    offset = 0
+                                    multiplier = 838 max rpm / 1 = 838
+                                -->
+                                <!--
+                                    SERVO<N>_FUNCTION   ->      70 (Throttle)
+                                    SERVO<N>_MAX        ->      servo_max
+                                    SERVO<N>_MIN        ->      servo_min
+                                    SERVO<N>_REVERSED   ->      cw_list[counter]
+                                    SERVO<N>_TRIM       ->
+                                -->
+                                <!--
+                                    The <useForce> tag determines how control commands are applied to the joint.
+                                    When set to 1, the control commands are applied as forces (effort),
+                                    resulting in more realistic physical interactions; when set to 0,
+                                    the commands are applied directly as velocities or positions.
+                                -->
+                                <type>VELOCITY</type>
+                                <multiplier>${directed_multiplier}</multiplier>
+                                <jointName>${jointName}</jointName>
+                                <useForce>1</useForce>
+                                <offset>${offset}</offset>
+                                <servo_max>${servo_max}</servo_max>deddedd
+                                <servo_min>${servo_min}</servo_min>adeeedededd
+                                <p_gain>${p_gain}</p_gain>
+                                <i_gain>${i_gain}</i_gain>
+                                <d_gain>${d_gain}</d_gain>
+                                <i_max>${i_max}</i_max>
+                                <i_min>${i_min}</i_min>
+                                <cmd_max>${cmd_max}</cmd_max>
+                                <cmd_min>${cmd_min}</cmd_min>
+                            </control>
+                            <!-- Recursively call the macro with a decremented count -->
+                            <xacro:create_arms i="${i - 1}"/>
+                        </xacro:if>
+                    </xacro:macro>
+                    <!-- Initial call to the macro with the desired number of joints -->
+                    <xacro:create_arms i="${int(number_of_arms)}"/>
+                    <!-- end Define arms! -->
+                    <xacro:insert_block name="extra_ardupilot_plugin_settings"/>
+                </plugin>
+            </xacro:unless>
         </gazebo>
     </xacro:macro>
