Commit message: made the xacro compatible with both classic and harmonic and made two launch files each for different gazebo types.

File: xacros/arm_macro.xacro (robot description, xacro)
@@ -2,5 +2,5 @@
 <robot xmlns:xacro="http://www.ros.org/wiki/xacro">
     <xacro:include filename="link_macros.xacro"/>
-    <xacro:macro name="drone_arm" params="num parent_link dis_from_center length diameter arm_incline_angle rotor_dis_from_arm arm_mesh prop_mesh cw
+    <xacro:macro name="drone_arm" params="using_gazebo_classic num parent_link dis_from_center length diameter arm_incline_angle rotor_dis_from_arm arm_mesh prop_mesh cw
                                           prop_size_multiplier prop_col_scale_xyz a_mass a_iner:='None' r_mass r_iner angle
                                           number_of_blades lift_a0 lift_alpha_stall lift_cla lift_cda lift_cma lift_cla_stall lift_sda_stall lift_cma_stall
@@ -48,4 +48,6 @@
             <extra_settings>
                 <velocity_decay/>
+                <gravity>1</gravity>
+                <self_collide>0</self_collide>
             </extra_settings>
         </xacro:link_creator_i_foundation>
@@ -59,20 +61,43 @@
                 <!-- <xacro:property name="blade_angle" value="${(num * pi) / 12}"/> -->
                 <gazebo>
-                    <plugin name="${rotor_blade}" filename="libLiftDragPlugin.so">
-                        <a0>${lift_a0}</a0>
-                        <alpha_stall>${lift_alpha_stall}</alpha_stall>
-                        <cla>${lift_cla}</cla>
-                        <cda>${lift_cda}</cda>
-                        <cma>${lift_cma}</cma>
-                        <cla_stall>${lift_cla_stall}</cla_stall>
-                        <cda_stall>${lift_sda_stall}</cda_stall>
-                        <cma_stall>${lift_cma_stall}</cma_stall>
-                        <area>${lift_area}</area>
-                        <air_density>${lift_air_density}</air_density>
-                        <cp>${cos(float(blade_angle)) * float(lift_cp)} ${sin(float(blade_angle)) * float(lift_cp)} 0</cp>
-                        <forward>${cos(float(blade_angle) - ((pi / 2) * direction))} ${sin(float(blade_angle) - ((pi / 2) * direction))} 0</forward>
-                        <upward>0 0 1</upward>
-                        <link_name>${prop_link}</link_name>
-                    </plugin>
+                    <xacro:if value="${using_gazebo_classic}">
+                        <!--for gazebo classic-->
+                        <plugin name="${rotor_blade}" filename="libLiftDragPlugin.so">
+                            <a0>${lift_a0}</a0>
+                            <alpha_stall>${lift_alpha_stall}</alpha_stall>
+                            <cla>${lift_cla}</cla>
+                            <cda>${lift_cda}</cda>
+                            <cma>${lift_cma}</cma>
+                            <cla_stall>${lift_cla_stall}</cla_stall>
+                            <cda_stall>${lift_sda_stall}</cda_stall>
+                            <cma_stall>${lift_cma_stall}</cma_stall>
+                            <area>${lift_area}</area>
+                            <air_density>${lift_air_density}</air_density>
+                            <cp>${cos(float(blade_angle)) * float(lift_cp)} ${sin(float(blade_angle)) * float(lift_cp)} 0</cp>
+                            <forward>${cos(float(blade_angle) - ((pi / 2) * direction))} ${sin(float(blade_angle) - ((pi / 2) * direction))} 0</forward>
+                            <upward>0 0 1</upward>
+                            <link_name>${prop_link}</link_name>
+                        </plugin>
+                    </xacro:if>
+                    <xacro:unless value="${using_gazebo_classic}">
+                        <!--for gazebo harmonic-->
+                        <plugin filename="gz-sim-joint-state-publisher-system" name="gz::sim::systems::JointStatePublisher"/>
+                        <plugin filename="gz-sim-lift-drag-system" name="gz::sim::systems::LiftDrag">
+                            <a0>${lift_a0}</a0>
+                            <alpha_stall>${lift_alpha_stall}</alpha_stall>
+                            <cla>${lift_cla}</cla>
+                            <cda>${lift_cda}</cda>
+                            <cma>${lift_cma}</cma>
+                            <cla_stall>${lift_cla_stall}</cla_stall>
+                            <cda_stall>${lift_sda_stall}</cda_stall>
+                            <cma_stall>${lift_cma_stall}</cma_stall>
+                            <area>${lift_area}</area>
+                            <air_density>${lift_air_density}</air_density>
+                            <cp>${cos(float(blade_angle)) * float(lift_cp)} ${sin(float(blade_angle)) * float(lift_cp)} 0</cp>
+                            <forward>${cos(float(blade_angle) - ((pi / 2) * direction))} ${sin(float(blade_angle) - ((pi / 2) * direction))} 0</forward>
+                            <upward>0 0 1</upward>
+                            <link_name>${prop_link}</link_name>
+                        </plugin>
+                    </xacro:unless>
                 </gazebo>
                 <!-- Recursively call the macro with a decremented count -->

File: xacros/drone_maker.xacro (robot description, xacro)
@@ -4,10 +4,10 @@
     <xacro:include filename="ardupilot_plugin.xacro"/>
     <xacro:property name="deg_to_rad" value="0.0174532925"/>
-    <xacro:macro name="drone_maker" params="base_mesh:='Box' base_pose_xyz:='0 0 0' base_pose_rpy:='0 0 0' base_scale_xyz:='0.4 0.4 0.04' base_center_of_mass:='0 0 0' base_mass base_iner:='None'
+    <xacro:macro name="drone_maker" params="using_gazebo_classic base_mesh:='Box' base_pose_xyz:='0 0 0' base_pose_rpy:='0 0 0' base_scale_xyz:='0.4 0.4 0.04' base_center_of_mass:='0 0 0' base_mass base_iner:='None'
                                             number_of_arms arm_angles cws prop_meshs
                                             dis_from_center length diameter arm_incline_angle:='0' rotor_dis_from_arm arm_mesh prop_size_multiplier
                                             prop_col_scale_xyz a_mass a_iner:='None' r_mass r_iner
                                             ardu_multiplier ardu_offset ardu_p_gain ardu_i_gain ardu_d_gain
-                                            ardu_i_max ardu_i_min ardu_cmd_max ardu_cmd_min
+                                            ardu_i_max ardu_i_min ardu_cmd_max ardu_cmd_min servo_max='1900' servo_min='1100'
                                             number_of_blades lift_a0 lift_alpha_stall
                                             lift_cla lift_cda lift_cma lift_cla_stall lift_sda_stall lift_cma_stall
@@ -34,13 +34,13 @@
                 <!-- Here define the arm -->
                 <xacro:property name="counter" value="${int(number_of_arms) - i}" />
-                <xacro:drone_arm num="${counter}" parent_link="base_link" dis_from_center="${dis_from_center}" length="${length}" diameter="${diameter}"
-                                arm_incline_angle="${arm_incline_angle * deg_to_rad}" rotor_dis_from_arm="${rotor_dis_from_arm}" arm_mesh="${arm_mesh}"
-                                prop_mesh="${prop_mesh_list[counter]}" cw="${cw_list[counter]}"
-                                prop_size_multiplier="${prop_size_multiplier}" prop_col_scale_xyz="${prop_col_scale_xyz}"
-                                a_mass="${a_mass}" a_iner="${a_iner}" r_mass="${r_mass}" r_iner="${r_iner}" angle="${float(arm_angle_list[counter]) * deg_to_rad}"
-                                number_of_blades="${number_of_blades}"
-                                lift_a0="${lift_a0}" lift_alpha_stall="${lift_alpha_stall}" lift_cla="${lift_cla}" lift_cda="${lift_cda}"
-                                lift_cma="${lift_cma}" lift_cla_stall="${lift_cla_stall}" lift_sda_stall="${lift_sda_stall}" lift_cma_stall="${lift_cma_stall}"
-                                lift_area="${lift_area}" lift_air_density="${lift_air_density}" lift_cp="${lift_cp}"/>
+                <xacro:drone_arm using_gazebo_classic="${using_gazebo_classic}" num="${counter}" parent_link="base_link" dis_from_center="${dis_from_center}" length="${length}" diameter="${diameter}"
+                                 arm_incline_angle="${arm_incline_angle * deg_to_rad}" rotor_dis_from_arm="${rotor_dis_from_arm}" arm_mesh="${arm_mesh}"
+                                 prop_mesh="${prop_mesh_list[counter]}" cw="${cw_list[counter]}"
+                                 prop_size_multiplier="${prop_size_multiplier}" prop_col_scale_xyz="${prop_col_scale_xyz}"
+                                 a_mass="${a_mass}" a_iner="${a_iner}" r_mass="${r_mass}" r_iner="${r_iner}" angle="${float(arm_angle_list[counter]) * deg_to_rad}"
+                                 number_of_blades="${number_of_blades}"
+                                 lift_a0="${lift_a0}" lift_alpha_stall="${lift_alpha_stall}" lift_cla="${lift_cla}" lift_cda="${lift_cda}"
+                                 lift_cma="${lift_cma}" lift_cla_stall="${lift_cla_stall}" lift_sda_stall="${lift_sda_stall}" lift_cma_stall="${lift_cma_stall}"
+                                 lift_area="${lift_area}" lift_air_density="${lift_air_density}" lift_cp="${lift_cp}"/>
                 <!-- Recursively call the macro with a decremented count -->
                 <xacro:create_arms i="${i - 1}"/>
@@ -77,5 +77,10 @@
         <gazebo reference="imu_link">
             <sensor name="imu_sensor" type="imu">
-                <pose>0 0 0 3.141593 0 0</pose>
+                <xacro:if value="${using_gazebo_classic}"/>
+                    <pose>0 0 0 3.141593 0 0</pose>
+                </xacro:if>
+                <xacro:unless value="${using_gazebo_classic}"/>
+                    <pose degrees="true">0 0 0 180 0 0</pose>
+                </xacro:unless>
                 <always_on>1</always_on>
                 <update_rate>1000.0</update_rate>
@@ -84,7 +89,7 @@
         <!-- end Define IMU! -->
         <!-- Define ardupilot_plugin! -->
-        <xacro:ardupilot_plugin number_of_arms="${number_of_arms}" multiplier="${ardu_multiplier}" cws="${cws}"
+        <xacro:ardupilot_plugin using_gazebo_classic="${using_gazebo_classic}" number_of_arms="${number_of_arms}" multiplier="${ardu_multiplier}" cws="${cws}"
                                 offset="${ardu_offset}" p_gain="${ardu_p_gain}" i_gain="${ardu_i_gain}" d_gain="${ardu_d_gain}"
-                                i_max="${ardu_i_max}" i_min="${ardu_i_min}" cmd_max="${ardu_cmd_max}" cmd_min="${ardu_cmd_min}">
+                                i_max="${ardu_i_max}" i_min="${ardu_i_min}" cmd_max="${ardu_cmd_max}" cmd_min="${ardu_cmd_min}" servo_max="${servo_max}" servo_min="${servo_min}">
             <extra_ardupilot_plugin_settings>
                 <xacro:insert_block name="extra_ardupilot_plugin_settings"/>

File: xacros/link_macros.xacro (robot description, xacro)
@@ -36,7 +36,5 @@
             <visual>
                 <material>
-                    <script>
-                        <name>Gazebo/DarkGrey</name>
-                    </script>
+                    <name>Gazebo/DarkGrey</name>
                 </material>
             </visual>

Commit message: fixed all the errors in the xacros files

File: models/copterPIX/robot.urdf.xacro (robot description, xacro)
@@ -1,7 +1,7 @@
 <?xml version="1.0" ?>
 <robot name="copterPIX" xmlns:xacro="http://www.ros.org/wiki/xacro">
-  <!--this value is changed by the launch script.-->
+  <xacro:include filename="$(find drone)/xacros/drone_maker.xacro"/>
+    <!--this value is changed by the launch script.-->
   <xacro:property name="using_gazebo_classic" value="0"/>
-  <xacro:include filename="$(find drone)/xacros/drone_maker.xacro"/>
   <xacro:property name="hex_mesh" value="$(find drone)/meshes/hexagonal_prism_height_1_outer_diameter_1.stl"/>
   <xacro:property name="prop_cw_mesh" value="$(find drone)/meshes/iris_prop_cw.dae"/>
@@ -74,6 +74,6 @@
                      lift_area="${lift_area}" lift_air_density="${lift_air_density}" lift_cp="${lift_cp}">
     <extra_ardupilot_plugin_settings>
-      <xacro:extra_channel using_gazebo_classic="${using_gazebo_classic}" channel="6" _type="POSITION" _multiplier="-200" _jointName="fire_trigger_servo_joint"
-                                          _offset="0" _p_gain="1" _i_gain="0" _d_gain="0"
+      <xacro:extra_channel using_gazebo_classic="${using_gazebo_classic}" _channel="6" _type="POSITION" _multiplier="-200" _jointName="fire_trigger_servo_joint"
+                                          _useForce="1" _offset="0" _p_gain="1" _i_gain="0" _d_gain="0"
                                           _i_max="0" _i_min="0" _cmd_max="2.5" _cmd_min="-2.5"/>
     </extra_ardupilot_plugin_settings>
@@ -132,6 +132,6 @@
   <xacro:property name="m16_position_z" value="${m16_position_list[2]}" />
   <gazebo>
+    <!--for gazebo classic-->
     <xacro:if value="${using_gazebo_classic}">
-      <!--for gazebo classic-->
       <plugin name="ForcePlugin" filename="libForcePlugin.so">
         <trigger_joint>fire_trigger_servo_joint</trigger_joint>
@@ -147,6 +147,6 @@
       </plugin>
     </xacro:if>
-    <xacro:unless value="${using_gazebo_classic}">
-      <!--for gazebo harmonic-->
+    <!--for gazebo harmonic-->
+    <!-- <xacro:unless value="${using_gazebo_classic}">
       <plugin name="ForcePlugin" filename="ForcePlugin">
         <trigger_joint>fire_trigger_servo_joint</trigger_joint>
@@ -161,5 +161,5 @@
         <position_z>${m16_position_z}</position_z>
       </plugin>
-    </xacro:unless>
+    </xacro:unless> -->
   </gazebo>
 </robot>

File: models/simple_box/robot.urdf.xacro (robot description, xacro)
@@ -2,4 +2,5 @@
 <robot name="simple_box" xmlns:xacro="http://www.ros.org/wiki/xacro">
   <origin xyz="0 0 0" rpy="0 0 0"/>
+  <xacro:include filename="$(find drone)/xacros/drone_maker.xacro"/>
   <xacro:property name="prop_cw_mesh" value="$(find drone)/meshes/iris_prop_cw.dae"/>
     <!-- Define the macro with an optional block parameter -->
@@ -66,4 +67,9 @@
   <link name="base_link">
   </link>
+  <joint name="feet_1_link_joint" type="fixed">
+    <parent link="base_link"/>
+    <child link="feet_1_link"/>
+  </joint>
+  <xacro:link_creator_i link_name="feet_1_link" pose_xyz="0 -0.29 -0.6" pose_rpy="0 1.57079633 0" mesh_path="Box" scale_xyz="0.024 0.024 0.58" mass="0.5"/>
   <joint name="base_child_joint" type="fixed">
     <parent link="base_link"/>

File: xacros/ardupilot_plugin.xacro (robot description, xacro)
@@ -1,8 +1,8 @@
 <?xml version="1.0" ?>
 <robot xmlns:xacro="http://www.ros.org/wiki/xacro">
-    <xacro:macro name="extra_channel" params="using_gazebo_classic channel _type _multiplier _jointName _useForce_offset _servo_max='1900' _servo_min='1100' _p_gain _i_gain _d_gain
+    <xacro:macro name="extra_channel" params="using_gazebo_classic _channel _type _multiplier _jointName _useForce:='1' _offset _servo_max:='1900' _servo_min:='1100' _p_gain _i_gain _d_gain
                                                           _i_max _i_min _cmd_max _cmd_min">
-        <xacro:if value="${using_gazebo_classic}" />
-            <control channel="${channel}">
+        <xacro:if value="${using_gazebo_classic}">
+            <control channel="${_channel}">
                 <type>${_type}</type>
                 <multiplier>${_multiplier}</multiplier>
@@ -16,9 +16,8 @@
                 <cmd_max>${_cmd_max}</cmd_max>
                 <cmd_min>${_cmd_min}</cmd_min>
-                <controlVelocitySlowdownSim>1</controlVelocitySlowdownSim>
             </control>
         </xacro:if>
-        <xacro:unless value="${using_gazebo_classic}" />
-            <control channel="${channel}">
+        <xacro:unless value="${using_gazebo_classic}">
+            <control channel="${_channel}">
                 <!--
                     incoming control command [0, 1]
@@ -55,12 +54,11 @@
                 <cmd_max>${_cmd_max}</cmd_max>
                 <cmd_min>${_cmd_min}</cmd_min>
-                <controlVelocitySlowdownSim>1</controlVelocitySlowdownSim>
             </control>
         </xacro:unless>
     </xacro:macro>
-    <xacro:macro name="ardupilot_plugin" params="using_gazebo_classic number_of_arms multiplier cws offset p_gain i_gain d_gain i_max i_min cmd_max cmd_min **extra_ardupilot_plugin_settings servo_max='1900' servo_min='1100'">
+    <xacro:macro name="ardupilot_plugin" params="using_gazebo_classic number_of_arms multiplier cws offset p_gain i_gain d_gain i_max i_min cmd_max cmd_min **extra_ardupilot_plugin_settings servo_max:='1900' servo_min:='1100'">
         <xacro:property name="cw_list" value="${cws.split(' ')}" />
         <gazebo>
-            <xacro:if value="${using_gazebo_classic}" />
+            <xacro:if value="${using_gazebo_classic}">
                 <plugin name="arducopter_plugin" filename="libArduPilotPlugin.so">
                     <fdm_addr>127.0.0.1</fdm_addr>
@@ -89,5 +87,4 @@
                                 <cmd_max>${cmd_max}</cmd_max>
                                 <cmd_min>${cmd_min}</cmd_min>
-                                <controlVelocitySlowdownSim>1</controlVelocitySlowdownSim>
                             </control>
                             <!-- Recursively call the macro with a decremented count -->
@@ -101,5 +98,5 @@
                 </plugin>
             </xacro:if>
-            <xacro:unless value="${using_gazebo_classic}" />
+            <xacro:unless value="${using_gazebo_classic}">
                 <plugin name="ArduPilotPlugin" filename="ArduPilotPlugin">
                     <fdm_addr>127.0.0.1</fdm_addr>

File: xacros/drone_maker.xacro (robot description, xacro)
@@ -9,5 +9,5 @@
                                             prop_col_scale_xyz a_mass a_iner:='None' r_mass r_iner
                                             ardu_multiplier ardu_offset ardu_p_gain ardu_i_gain ardu_d_gain
-                                            ardu_i_max ardu_i_min ardu_cmd_max ardu_cmd_min servo_max='1900' servo_min='1100'
+                                            ardu_i_max ardu_i_min ardu_cmd_max ardu_cmd_min servo_max:='1900' servo_min:='1100'
                                             number_of_blades lift_a0 lift_alpha_stall
                                             lift_cla lift_cda lift_cma lift_cla_stall lift_sda_stall lift_cma_stall
@@ -77,8 +77,8 @@
         <gazebo reference="imu_link">
             <sensor name="imu_sensor" type="imu">
-                <xacro:if value="${using_gazebo_classic}"/>
+                <xacro:if value="${using_gazebo_classic}">
                     <pose>0 0 0 3.141593 0 0</pose>
                 </xacro:if>
-                <xacro:unless value="${using_gazebo_classic}"/>
+                <xacro:unless value="${using_gazebo_classic}">
                     <pose degrees="true">0 0 0 180 0 0</pose>
                 </xacro:unless>

Commit message: minor edits to xacro files

File: models/copterPIX/robot.urdf.xacro (robot description, xacro)
@@ -2,5 +2,5 @@
 <robot name="copterPIX" xmlns:xacro="http://www.ros.org/wiki/xacro">
   <xacro:include filename="$(find drone)/xacros/drone_maker.xacro"/>
-    <!--this value is changed by the launch script.-->
+  <!--this value is changed by the launch script.-->
   <xacro:property name="using_gazebo_classic" value="0"/>
   <xacro:property name="hex_mesh" value="$(find drone)/meshes/hexagonal_prism_height_1_outer_diameter_1.stl"/>
@@ -17,4 +17,5 @@
   <xacro:property name="iner" value="${ixx} ${ixy} ${ixz} ${iyy} ${iyz} ${izz}" />
 -->
+  <xacro:property name="base_root_offset" value="0" />
   <xacro:property name="base_mesh" value="${hex_mesh}"/>
   <xacro:property name="base_pose_xyz" value="0 0 0"/>
@@ -61,5 +62,5 @@
   <xacro:property name="lift_air_density" value="1.2041"/>
   <xacro:property name="lift_cp" value="0.2"/>
-  <xacro:drone_maker using_gazebo_classic="${using_gazebo_classic}" base_mesh="${base_mesh}" base_pose_xyz ="${base_pose_xyz}" base_pose_rpy="${base_pose_rpy}" base_scale_xyz="${base_scale_xyz}"
+  <xacro:drone_maker using_gazebo_classic="${using_gazebo_classic}" base_root_offset="${base_root_offset}" base_mesh="${base_mesh}" base_pose_xyz ="${base_pose_xyz}" base_pose_rpy="${base_pose_rpy}" base_scale_xyz="${base_scale_xyz}"
                      base_center_of_mass="${base_center_of_mass}" base_mass="${base_mass}" base_iner="${base_iner}"
                      number_of_arms="${number_of_arms}" arm_angles="${arm_angles}" cws="${cws}" prop_meshs="${prop_meshs}"

File: models/iris/robot.urdf.xacro (robot description, xacro)
@@ -1,7 +1,7 @@
 <?xml version="1.0" ?>
 <robot name="copterPIX" xmlns:xacro="http://www.ros.org/wiki/xacro">
+  <xacro:include filename="$(find drone)/xacros/drone_maker.xacro"/>
   <!--this value is changed by the launch script.-->
   <xacro:property name="using_gazebo_classic" value="0"/>
-  <xacro:include filename="$(find drone)/xacros/drone_maker.xacro"/>
   <xacro:property name="hex_mesh" value="$(find drone)/meshes/hexagonal_prism_height_1_outer_diameter_1.stl"/>
   <xacro:property name="prop_cw_mesh" value="$(find drone)/meshes/iris_prop_cw.dae"/>
@@ -51,5 +51,5 @@
   <xacro:property name="lift_air_density" value="1.2041"/>
   <xacro:property name="lift_cp" value="0.084"/>
- <xacro:drone_maker using_gazebo_classic="${using_gazebo_classic}" base_mesh="${base_mesh}" base_pose_xyz ="${base_pose_xyz}" base_pose_rpy="${base_pose_rpy}" base_scale_xyz="${base_scale_xyz}"
+  <xacro:drone_maker using_gazebo_classic="${using_gazebo_classic}" base_mesh="${base_mesh}" base_pose_xyz ="${base_pose_xyz}" base_pose_rpy="${base_pose_rpy}" base_scale_xyz="${base_scale_xyz}"
                      base_center_of_mass="${base_center_of_mass}" base_mass="${base_mass}" base_iner="${base_iner}"
                      number_of_arms="${number_of_arms}" arm_angles="${arm_angles}" cws="${cws}" prop_meshs="${prop_meshs}"

File: xacros/drone_maker.xacro (robot description, xacro)
@@ -4,5 +4,5 @@
     <xacro:include filename="ardupilot_plugin.xacro"/>
     <xacro:property name="deg_to_rad" value="0.0174532925"/>
-    <xacro:macro name="drone_maker" params="using_gazebo_classic base_mesh:='Box' base_pose_xyz:='0 0 0' base_pose_rpy:='0 0 0' base_scale_xyz:='0.4 0.4 0.04' base_center_of_mass:='0 0 0' base_mass base_iner:='None'
+    <xacro:macro name="drone_maker" params="using_gazebo_classic base_root_offset:='0' base_mesh:='Box' base_pose_xyz:='0 0 0' base_pose_rpy:='0 0 0' base_scale_xyz:='0.4 0.4 0.04' base_center_of_mass:='0 0 0' base_mass base_iner:='None'
                                             number_of_arms arm_angles cws prop_meshs
                                             dis_from_center length diameter arm_incline_angle:='0' rotor_dis_from_arm arm_mesh prop_size_multiplier
@@ -21,5 +21,5 @@
             <parent link="root_link"/>
             <child link="base_link"/>
-            <origin xyz="0 0 0" rpy="0 0 0"/>
+            <origin xyz="0 0 ${base_root_offset}" rpy="0 0 0"/>
         </joint>
         <!-- Define base_link! -->
