Commit message: fixed gazebo_classic_sim.launch.py and link_macro.xacro

File: models/copterPIX/robot.urdf.xacro (robot description, xacro)
@@ -3,5 +3,5 @@
   <xacro:include filename="$(find drone)/xacros/drone_maker.xacro"/>
   <!--this value is changed by the launch script.-->
-  <xacro:property name="using_gazebo_classic" value="0"/>
+  <xacro:property name="using_gazebo_classic" value="1"/>
   <xacro:property name="hex_mesh" value="$(find drone)/meshes/hexagonal_prism_height_1_outer_diameter_1.stl"/>
   <xacro:property name="prop_cw_mesh" value="$(find drone)/meshes/iris_prop_cw.dae"/>

File: xacros/link_macros.xacro (robot description, xacro)
@@ -34,9 +34,10 @@
         </link>
         <gazebo reference="${link_name}">
-            <visual>
+            <material>Gazebo/DarkGrey</material><!--for classic-->
+            <!-- <visual>
                 <material>
                     <name>Gazebo/DarkGrey</name>
                 </material>
-            </visual>
+            </visual> -->
         </gazebo>
     </xacro:macro>
